Commit message: Light head tested

File: bender_common/bender_description/urdf/light_head.urdf.xacro (robot description, xacro)
@@ -165,5 +165,5 @@
         xyz="0 1 0" />
       <!-- Limits based on Dynamixel motor encoder ticks -->
-      <limit effort="0.3" velocity="1.0" upper="1.02" lower="-0.77" />
+      <limit effort="0.3" velocity="1.0" upper="1.2476" lower="-0.951" />
     </joint>
     <!-- Camera RGB and depth frames -->

Commit message: Lighthead update and gazebo interface

File: bender_common/bender_description/urdf/light_head.urdf.xacro (robot description, xacro)
@@ -5,5 +5,5 @@
     <xacro:gazebo_link link="${prefix}light_head_base_link" color="Grey" />
     <xacro:gazebo_link link="${prefix}light_head_yaw_link" color="Grey" />
-    <xacro:gazebo_link link="${prefix}light_head_pitch_link" color="Grey" />
+    <xacro:gazebo_link link="${prefix}light_head_pitch_link" color="DarkGrey" />
     <!-- Transmissions -->
     <xacro:joint_transmission joint="light_head_yaw_joint"/>
@@ -50,5 +50,5 @@
       </collision>
     </link>
-    <joint name="${prefix}light_head_base_joint" type="fixed">
+    <joint name="light_head_base_joint" type="fixed">
       <origin xyz="0 0 0" rpy="0 0 0" />
       <parent link="${parent}"/>
@@ -109,5 +109,7 @@
         xyz="0 0 1" />
       <!-- Limits based on Dynamixel motor encoder ticks -->
+      <dynamics damping="0.1" />
       <limit effort="0.3" velocity="1.0" lower="-2.62" upper="2.62" />
+      <dynamics damping="0.1" />
     </joint>
     <!-- Camera link with pitch movement -->
@@ -116,15 +118,15 @@
       <inertial>
         <origin
-          xyz="0.012803 -0.002792 0.042974"
+          xyz="-0.0085671 0.0029816 0.056743"
           rpy="0 0 0" />
         <mass
           value="0.15438" />
         <inertia
-          ixx="0.00040408"
-          ixy="-5.1443E-07"
-          ixz="1.0922E-06"
-          iyy="2.8871E-05"
-          iyz="7.7773E-08"
-          izz="0.00040656" />
+          ixx="0.00042205"
+          ixy="-2.5048E-06"
+          ixz="-1.5995E-06"
+          iyy="4.319E-05"
+          iyz="7.1E-06"
+          izz="0.00041533" />
       </inertial>
       <visual>
@@ -156,6 +158,6 @@
       type="revolute">
       <origin
-        xyz="0 0.003486 0.0525"
-        rpy="0 0 0" />
+        xyz="-0.001 -0.008 0.0525"
+        rpy="0 0.35 0" />
       <parent
         link="${prefix}light_head_yaw_link" />
@@ -165,5 +167,6 @@
         xyz="0 1 0" />
       <!-- Limits based on Dynamixel motor encoder ticks -->
-      <limit effort="0.3" velocity="1.0" upper="1.2476" lower="-0.951" />
+      <limit effort="0.3" velocity="1.0" upper="1.166" lower="-1.0328" />
+      <dynamics damping="0.1" />
     </joint>
     <!-- Camera RGB and depth frames -->
@@ -174,6 +177,6 @@
       type="fixed">
       <origin
-        xyz="0.021786 0.016 0.043893"
-        rpy="0 0 0" />
+        xyz="-0.001116 0.02305 0.062283"
+        rpy="0.0 -0.31716 0.0" />
       <parent
         link="${prefix}light_head_pitch_link" />
@@ -189,6 +192,6 @@
       type="fixed">
       <origin
-        xyz="0.021786 0.042 0.043893"
-        rpy="0 0 0" />
+        xyz="-0.001116 0.04905 0.062283"
+        rpy="0.0 -0.31716 0.0" />
       <parent
         link="${prefix}light_head_pitch_link" />
