Commit message: Add SW inertia

File: bender_common/bender_description/urdf/arm.urdf.xacro (robot description, xacro)
@@ -20,10 +20,12 @@
   <xacro:property name="shoulder_roll_joint_lower" value="-0.23776" />
   <!-- Links mass -->
-  <xacro:property name="shoulder_pitch_mass" value="${0.216}" />
-  <xacro:property name="shoulder_roll_mass"  value="${0.282}" />
-  <xacro:property name="shoulder_yaw_mass"   value="${0.256}" />
-  <xacro:property name="elbow_pitch_mass"    value="${0.243}" />
-  <xacro:property name="elbow_yaw_mass"      value="${0.222}" />
-  <xacro:property name="wrist_pitch_mass"    value="${0.430}" />
+  <xacro:property name="TO_KG" value="${0.001}" />
+  <xacro:property name="TO_KG_M2" value="${0.000000001}" />
+  <xacro:property name="shoulder_pitch_mass" value="${237.99*TO_KG}" />
+  <xacro:property name="shoulder_roll_mass"  value="${284.50*TO_KG}" />
+  <xacro:property name="shoulder_yaw_mass"   value="${261.97*TO_KG}" />
+  <xacro:property name="elbow_pitch_mass"    value="${245.92*TO_KG}" />
+  <xacro:property name="elbow_yaw_mass"      value="${199.60*TO_KG}" />
+  <xacro:property name="wrist_pitch_mass"    value="${492.01*TO_KG}" />
   <!-- Torque -->
   <xacro:property name="shoulder_pitch_torque" value="${mx106_torque}" />
@@ -53,8 +55,15 @@
       <inertial>
         <origin
-          xyz="0 ${- reflect * 0.02} 0"
+          xyz="0 0 0"
           rpy="0 0 0" />
         <mass value="${shoulder_pitch_mass}" />
-        <cuboid_inertia_def x="0.05" y="0.07" z="0.07" mass="${shoulder_pitch_mass}"/>
+        <inertia
+          ixx="${221387.60*TO_KG_M2}"
+          iyy="${113152.17*TO_KG_M2}"
+          izz="${164719.59*TO_KG_M2}"
+          ixy="${-1674.85*TO_KG_M2}"
+          iyz="${-77398.27*TO_KG_M2}"
+          ixz="${966.22*TO_KG_M2}"
+        />
       </inertial>
       <visual>
@@ -101,8 +110,15 @@
       <inertial>
         <origin
-          xyz="0.04 0 -0.075"
-          rpy="0 -0.25 0" />
+          xyz="0.0 0 0.0"
+          rpy="0 0.0 0" />
         <mass value="${shoulder_roll_mass}" />
-        <cuboid_inertia_def x="0.05" y="0.035" z="0.18" mass="${shoulder_roll_mass}"/>
+        <inertia
+          ixx="${3996527.93*TO_KG_M2}"
+          iyy="${4616215.27*TO_KG_M2}"
+          izz="${4616215.27*TO_KG_M2}"
+          ixy="${-167.80*TO_KG_M2}"
+          iyz="${428.69*TO_KG_M2}"
+          ixz="${-1563629.34*TO_KG_M2}"
+        />
       </inertial>
       <visual>
@@ -149,8 +165,15 @@
       <inertial>
         <origin
-          xyz="-0.015 0 -0.115"
+          xyz="0 0 0"
           rpy="0 0 0" />
         <mass value="${shoulder_yaw_mass}" />
-        <cuboid_inertia_def x="0.05" y="0.035" z="0.23" mass="${shoulder_yaw_mass}"/>
+        <inertia
+          ixx="${6037713.48*TO_KG_M2}"
+          iyy="${6119754.54*TO_KG_M2}"
+          izz="${86667.41*TO_KG_M2}"
+          ixy="${924.54*TO_KG_M2}"
+          iyz="${8129.28*TO_KG_M2}"
+          ixz="${685061.98*TO_KG_M2}"
+        />
       </inertial>
       <visual>
@@ -197,8 +220,15 @@
       <inertial>
         <origin
-          xyz="0.015 -0.025 -0.05"
+          xyz="0 0 0"
           rpy="0 0 0" />
         <mass value="${elbow_pitch_mass}" />
-        <cuboid_inertia_def x="0.05" y="0.07" z="0.10" mass="${elbow_pitch_mass}"/>
+        <inertia
+          ixx="${1042579.00*TO_KG_M2}"
+          iyy="${929112.85*TO_KG_M2}"
+          izz="${143277.29*TO_KG_M2}"
+          ixy="${-38569.80*TO_KG_M2}"
+          iyz="${329101.58*TO_KG_M2}"
+          ixz="${-107274.76*TO_KG_M2}"
+        />
       </inertial>
       <visual>
@@ -245,8 +275,15 @@
       <inertial>
         <origin
-          xyz="-0.015 0 -0.12"
+          xyz="0 0 0"
           rpy="0 0 0" />
         <mass value="${elbow_yaw_mass}" />
-        <cuboid_inertia_def x="0.05" y="0.035" z="0.32" mass="${elbow_yaw_mass}"/>
+        <inertia
+          ixx="${5623975.01*TO_KG_M2}"
+          iyy="${5707839.48*TO_KG_M2}"
+          izz="${125573.79*TO_KG_M2}"
+          ixy="${-106.64*TO_KG_M2}"
+          iyz="${-848.52*TO_KG_M2}"
+          ixz="${562590.78*TO_KG_M2}"
+        />
       </inertial>
       <visual>
@@ -293,8 +330,15 @@
       <inertial>
         <origin
-          xyz="0 -0.02 -0.05"
+          xyz="0 0 0"
           rpy="0 0 0" />
         <mass value="${wrist_pitch_mass}" />
-        <cuboid_inertia_def x="0.04" y="0.08" z="0.07" mass="${wrist_pitch_mass}"/>
+        <inertia
+          ixx="${6346473.13*TO_KG_M2}"
+          iyy="${6213377.71*TO_KG_M2}"
+          izz="${187625.24*TO_KG_M2}"
+          ixy="${2135.45*TO_KG_M2}"
+          iyz="${725135.57*TO_KG_M2}"
+          ixz="${19363.35*TO_KG_M2}"
+        />
       </inertial>
       <visual>

File: bender_common/bender_description/urdf/gripper.urdf.xacro (robot description, xacro)
@@ -5,6 +5,6 @@
   <xacro:property name="int_finger_joint_upper" value="0.69029" />
   <xacro:property name="int_finger_joint_lower" value="-0.02556" />
-  <xacro:property name="gripper_mass" value="1.0" />
-  <xacro:property name="gripper_effort" value="1.0" />
+  <xacro:property name="gripper_mass" value="0.160" />
+  <xacro:property name="gripper_effort" value="${rx28_torque}" />
   <xacro:macro name="gripper" params="side reflect prefix">
     <!-- Transmission -->

Commit message: Fix gazebo grippers and Arms

File: bender_common/bender_description/urdf/arm.urdf.xacro (robot description, xacro)
@@ -21,4 +21,5 @@
   <!-- Links mass -->
   <xacro:property name="TO_KG" value="${0.001}" />
+  <xacro:property name="TO_M" value="${0.001}" />
   <xacro:property name="TO_KG_M2" value="${0.000000001}" />
   <xacro:property name="shoulder_pitch_mass" value="${237.99*TO_KG}" />
@@ -45,25 +46,18 @@
     <xacro:gazebo_link link="${prefix}${side}_wrist_pitch_link" color="Grey" />
     <!-- Transmissions -->
-    <xacro:joint_pos_transmission joint="${side}_shoulder_pitch_joint"/>
-    <xacro:joint_pos_transmission joint="${side}_shoulder_roll_joint"/>
-    <xacro:joint_pos_transmission joint="${side}_shoulder_yaw_joint"/>
-    <xacro:joint_pos_transmission joint="${side}_elbow_pitch_joint"/>
-    <xacro:joint_pos_transmission joint="${side}_elbow_yaw_joint"/>
-    <xacro:joint_pos_transmission joint="${side}_wrist_pitch_joint"/>
+    <xacro:joint_transmission joint="${side}_shoulder_pitch_joint"/>
+    <xacro:joint_transmission joint="${side}_shoulder_roll_joint"/>
+    <xacro:joint_transmission joint="${side}_shoulder_yaw_joint"/>
+    <xacro:joint_transmission joint="${side}_elbow_pitch_joint"/>
+    <xacro:joint_transmission joint="${side}_elbow_yaw_joint"/>
+    <xacro:joint_transmission joint="${side}_wrist_pitch_joint"/>
     <link
       name="${prefix}${side}_shoulder_pitch_link">
       <inertial>
         <origin
-          xyz="0 0 0"
+          xyz="${-0.30*TO_M} ${-reflect*23.75*TO_M} ${-13.7*TO_M}"
           rpy="0 0 0" />
         <mass value="${shoulder_pitch_mass}" />
-        <inertia
-          ixx="${221387.60*TO_KG_M2}"
-          iyy="${113152.17*TO_KG_M2}"
-          izz="${164719.59*TO_KG_M2}"
-          ixy="${-1674.85*TO_KG_M2}"
-          iyz="${-77398.27*TO_KG_M2}"
-          ixz="${966.22*TO_KG_M2}"
-        />
+        <cuboid_inertia_def x="0.05" y="0.07" z="0.07" mass="${shoulder_pitch_mass}"/>
       </inertial>
       <visual>
@@ -110,15 +104,8 @@
       <inertial>
         <origin
-          xyz="0.0 0 0.0"
-          rpy="0 0.0 0" />
+          xyz="${46.28*TO_M} ${-0.01*TO_M} ${-118.24*TO_M}"
+          rpy="0 0 0" />
         <mass value="${shoulder_roll_mass}" />
-        <inertia
-          ixx="${3996527.93*TO_KG_M2}"
-          iyy="${4616215.27*TO_KG_M2}"
-          izz="${4616215.27*TO_KG_M2}"
-          ixy="${-167.80*TO_KG_M2}"
-          iyz="${428.69*TO_KG_M2}"
-          ixz="${-1563629.34*TO_KG_M2}"
-        />
+        <cuboid_inertia_def x="0.05" y="0.035" z="0.18" mass="${shoulder_roll_mass}"/>
       </inertial>
       <visual>
@@ -165,15 +152,8 @@
       <inertial>
         <origin
-          xyz="0 0 0"
+          xyz="${-17.25*TO_M} ${-0.20*TO_M} ${-151.64*TO_M}"
           rpy="0 0 0" />
         <mass value="${shoulder_yaw_mass}" />
-        <inertia
-          ixx="${6037713.48*TO_KG_M2}"
-          iyy="${6119754.54*TO_KG_M2}"
-          izz="${86667.41*TO_KG_M2}"
-          ixy="${924.54*TO_KG_M2}"
-          iyz="${8129.28*TO_KG_M2}"
-          ixz="${685061.98*TO_KG_M2}"
-        />
+        <cuboid_inertia_def x="0.05" y="0.035" z="0.23" mass="${shoulder_yaw_mass}"/>
       </inertial>
       <visual>
@@ -220,15 +200,8 @@
       <inertial>
         <origin
-          xyz="0 0 0"
+          xyz="${7.17*TO_M} ${-21.86*TO_M} ${-60.81*TO_M}"
           rpy="0 0 0" />
         <mass value="${elbow_pitch_mass}" />
-        <inertia
-          ixx="${1042579.00*TO_KG_M2}"
-          iyy="${929112.85*TO_KG_M2}"
-          izz="${143277.29*TO_KG_M2}"
-          ixy="${-38569.80*TO_KG_M2}"
-          iyz="${329101.58*TO_KG_M2}"
-          ixz="${-107274.76*TO_KG_M2}"
-        />
+        <cuboid_inertia_def x="0.05" y="0.07" z="0.10" mass="${elbow_pitch_mass}"/>
       </inertial>
       <visual>
@@ -275,15 +248,8 @@
       <inertial>
         <origin
-          xyz="0 0 0"
+          xyz="${-19.08*TO_M} ${0.03*TO_M} ${-152.08*TO_M}"
           rpy="0 0 0" />
         <mass value="${elbow_yaw_mass}" />
-        <inertia
-          ixx="${5623975.01*TO_KG_M2}"
-          iyy="${5707839.48*TO_KG_M2}"
-          izz="${125573.79*TO_KG_M2}"
-          ixy="${-106.64*TO_KG_M2}"
-          iyz="${-848.52*TO_KG_M2}"
-          ixz="${562590.78*TO_KG_M2}"
-        />
+        <cuboid_inertia_def x="0.05" y="0.035" z="0.32" mass="${elbow_yaw_mass}"/>
       </inertial>
       <visual>
@@ -330,15 +296,8 @@
       <inertial>
         <origin
-          xyz="0 0 0"
+          xyz="${-0.03*TO_M} ${-13.24*TO_M} ${-111.35*TO_M}"
           rpy="0 0 0" />
         <mass value="${wrist_pitch_mass}" />
-        <inertia
-          ixx="${6346473.13*TO_KG_M2}"
-          iyy="${6213377.71*TO_KG_M2}"
-          izz="${187625.24*TO_KG_M2}"
-          ixy="${2135.45*TO_KG_M2}"
-          iyz="${725135.57*TO_KG_M2}"
-          ixz="${19363.35*TO_KG_M2}"
-        />
+        <cuboid_inertia_def x="0.04" y="0.08" z="0.07" mass="${wrist_pitch_mass}"/>
       </inertial>
       <visual>

File: bender_common/bender_description/urdf/body.urdf.xacro (robot description, xacro)
@@ -23,6 +23,6 @@
           xyz="0 ${- reflect * 0.025} 0"
           rpy="${M_PI/2} 0 0" />
-        <cylinder_inertia_def length="0.05" radius="0.1" mass="10.0"/>
-        <mass value="10.0" />
+        <cylinder_inertia_def length="0.05" radius="0.1" mass="50.0"/>
+        <mass value="50.0" />
       </inertial>
       <visual>
@@ -85,8 +85,8 @@
       <inertial>
         <origin
-          xyz="0 0 0.7"
+          xyz="0 0 0.1"
           rpy="0 0 0" />
-        <mass value="100.0" />
-        <cuboid_inertia_def x="0.2" y="0.4" z="1.25" mass="100.0"/>
+        <mass value="400.0" />
+        <cuboid_inertia_def x="0.1" y="0.4" z="0.25" mass="400.0"/>
       </inertial>
       <visual>

File: bender_common/bender_description/urdf/gripper.urdf.xacro (robot description, xacro)
@@ -133,5 +133,5 @@
       <xacro:gripper_type type="${type}" />
     </link>
-    <xacro:gazebo_friction_link link="${side}_int_finger_link" color="DarkGrey" />
+    <xacro:gazebo_friction_link link="${prefix}${side}_int_finger_link" color="DarkGrey" />
     <joint
       name="${side}_int_finger_fixed_joint"
@@ -161,5 +161,5 @@
       <xacro:gripper_type type="${type}" />
     </link>
-    <xacro:gazebo_friction_link link="${side}_ext_finger_link" color="DarkGrey" />
+    <xacro:gazebo_friction_link link="${prefix}${side}_ext_finger_link" color="DarkGrey" />
     <joint
       name="${side}_ext_finger_fixed_joint"
