Commit message: New URDF

File: bender_common/bender_description/urdf/arm.urdf.xacro (robot description, xacro)
@@ -2,6 +2,5 @@
 <robot
   xmlns:xacro="http://www.ros.org/wiki/xacro"
-  name="bender_arm">
-  <xacro:include filename="$(find bender_description)/urdf/gripper.urdf.xacro" />
+  name="arm">
   <!-- Soft margin 5 deg -->
   <xacro:property name="soft_margin" value="${M_PI/36}" />
@@ -19,14 +18,4 @@
   <xacro:property name="shoulder_roll_joint_upper" value="1.51096" />
   <xacro:property name="shoulder_roll_joint_lower" value="-0.23776" />
-  <!-- Links mass -->
-  <xacro:property name="TO_KG" value="${0.001}" />
-  <xacro:property name="TO_M" value="${0.001}" />
-  <xacro:property name="TO_KG_M2" value="${0.000000001}" />
-  <xacro:property name="shoulder_pitch_mass" value="${237.99*TO_KG}" />
-  <xacro:property name="shoulder_roll_mass"  value="${284.50*TO_KG}" />
-  <xacro:property name="shoulder_yaw_mass"   value="${261.97*TO_KG}" />
-  <xacro:property name="elbow_pitch_mass"    value="${245.92*TO_KG}" />
-  <xacro:property name="elbow_yaw_mass"      value="${199.60*TO_KG}" />
-  <xacro:property name="wrist_pitch_mass"    value="${492.01*TO_KG}" />
   <!-- Torque -->
   <xacro:property name="shoulder_pitch_torque" value="${mx106_torque}" />
@@ -36,13 +25,5 @@
   <xacro:property name="elbow_yaw_torque"      value="${rx64_torque}" />
   <xacro:property name="wrist_pitch_torque"    value="${rx28_torque}" />
-  <xacro:macro name="bender_arm" params="side parent reflect prefix">
-    <!-- Gazebo elements -->
-    <!-- Gazebo Links material -->
-    <xacro:gazebo_link link="${prefix}${side}_shoulder_pitch_link" color="DarkGrey" />
-    <xacro:gazebo_link link="${prefix}${side}_shoulder_roll_link" color="Grey" />
-    <xacro:gazebo_link link="${prefix}${side}_shoulder_yaw_link" color="DarkGrey" />
-    <xacro:gazebo_link link="${prefix}${side}_elbow_pitch_link" color="Grey" />
-    <xacro:gazebo_link link="${prefix}${side}_elbow_yaw_link" color="DarkGrey" />
-    <xacro:gazebo_link link="${prefix}${side}_wrist_pitch_link" color="Grey" />
+  <xacro:macro name="arm" params="side parent reflect prefix">
     <!-- Transmissions -->
     <xacro:joint_transmission joint="${side}_shoulder_pitch_joint"/>
@@ -52,22 +33,101 @@
     <xacro:joint_transmission joint="${side}_elbow_yaw_joint"/>
     <xacro:joint_transmission joint="${side}_wrist_pitch_joint"/>
+    <!-- Base fixed joint and link -->
+    <joint
+      name="${side}_arm_base_fixed_joint"
+      type="fixed">
+      <origin
+        xyz="0 0 0"
+        rpy="0 0 0" />
+      <parent
+        link="${parent}" />
+      <child
+        link="${prefix}${side}_arm_base_link" />
+      <axis
+        xyz="0 0 0" />
+    </joint>
+    <link
+      name="${prefix}${side}_arm_base_link">
+      <inertial>
+        <origin
+          xyz="3.1697E-06 -0.017088 0.00063087"
+          rpy="0 0 0" />
+        <mass
+          value="0.17471" />
+        <inertia
+          ixx="0.00037909"
+          ixy="7.4755E-09"
+          ixz="2.8692E-09"
+          iyy="0.00040178"
+          iyz="8.0104E-07"
+          izz="9.5869E-05" />
+      </inertial>
+      <visual>
+        <xacro:if value="${(reflect+1)/2}">
+        <origin
+          xyz="0 0 0"
+          rpy="${-M_PI/2} 0 ${M_PI}" />
+        </xacro:if >
+        <xacro:unless value="${(reflect+1)/2}">
+        <origin
+          xyz="0 0 0"
+          rpy="${-M_PI/2} 0 0" />
+        </xacro:unless >
+        <geometry>
+          <mesh
+            filename="package://bender_description/meshes/visual/shoulder_base_link.dae" />
+        </geometry>
+        <material
+          name="">
+          <color
+            rgba="0.1 0.1 0.1 1" />
+        </material>
+      </visual>
+      <collision>
+        <origin
+          xyz="0 ${reflect * 0.03} 0"
+          rpy="0 0 0" />
+        <geometry>
+          <box size="0.07 0.06 0.17"/>
+        </geometry>
+      </collision>
+    </link>
+    <!-- Shoulder pitch -->
     <link
       name="${prefix}${side}_shoulder_pitch_link">
       <inertial>
         <origin
-          xyz="${-0.30*TO_M} ${-reflect*23.75*TO_M} ${-13.7*TO_M}"
-          rpy="0 0 0" />
-        <mass value="${shoulder_pitch_mass}" />
-        <cuboid_inertia_def x="0.05" y="0.07" z="0.07" mass="${shoulder_pitch_mass}"/>
-      </inertial>
-      <visual>
-        <origin
-          xyz="0 0 0"
-          rpy="0 0 0" />
-        <geometry>
-          <mesh
-            filename="package://bender_description/meshes/visual/${side}_shoulder_pitch.stl" />
-        </geometry>
-        <material name="Grey1" />
+          xyz="0.00023251 0.019812 -0.013482"
+          rpy="0 0 0" />
+        <mass
+          value="0.17152" />
+        <inertia
+          ixx="0.00010991"
+          ixy="-5.6413E-07"
+          ixz="1.0935E-06"
+          iyy="0.00010993"
+          iyz="1.8807E-06"
+          izz="8.8167E-05" />
+      </inertial>
+      <visual>
+        <xacro:if value="${(reflect+1)/2}">
+        <origin
+          xyz="0 0 0"
+          rpy="${-M_PI/2} 0 ${M_PI}" />
+        </xacro:if >
+        <xacro:unless value="${(reflect+1)/2}">
+        <origin
+          xyz="0 0 0"
+          rpy="${-M_PI/2} 0 0" />
+        </xacro:unless >
+        <geometry>
+          <mesh
+            filename="package://bender_description/meshes/visual/shoulder_pitch.dae" />
+        </geometry>
+        <material
+          name="">
+          <color
+            rgba="0.1 0.1 0.1 1" />
+        </material>
       </visual>
       <collision>
@@ -84,8 +144,8 @@
       type="revolute">
       <origin
-        xyz="0 0 0"
-        rpy="0 0 0" />
-      <parent
-        link="${parent}" />
+        xyz="0 ${- reflect * 0.0046} 0.0176"
+        rpy="0 0 0" />
+      <parent
+        link="${prefix}${side}_arm_base_link" />
       <child
         link="${prefix}${side}_shoulder_pitch_link" />
@@ -100,22 +160,34 @@
       <safety_controller soft_lower_limit="${shoulder_pitch_joint_lower-soft_margin}" soft_upper_limit="${shoulder_pitch_joint_upper+soft_margin}" k_position="30" k_velocity="30"/>
     </joint>
+    <!-- Shoulder roll -->
     <link
       name="${prefix}${side}_shoulder_roll_link">
       <inertial>
         <origin
-          xyz="${46.28*TO_M} ${-0.01*TO_M} ${-118.24*TO_M}"
-          rpy="0 0 0" />
-        <mass value="${shoulder_roll_mass}" />
-        <cuboid_inertia_def x="0.05" y="0.035" z="0.18" mass="${shoulder_roll_mass}"/>
-      </inertial>
-      <visual>
-        <origin
-          xyz="0 0 0"
-          rpy="0 0 0" />
-        <geometry>
-          <mesh
-            filename="package://bender_description/meshes/visual/shoulder_roll.stl" />
-        </geometry>
-        <material name="Grey2" />
+          xyz="0.046779 -9.3259E-06 -0.11466"
+          rpy="0 0 0" />
+        <mass
+          value="0.16104" />
+        <inertia
+          ixx="0.00050901"
+          ixy="6.2439E-09"
+          ixz="0.00010534"
+          iyy="0.00055051"
+          iyz="-6.7534E-08"
+          izz="0.00011428" />
+      </inertial>
+      <visual>
+        <origin
+          xyz="0 0 0"
+          rpy="${-M_PI/2} 0 0" />
+        <geometry>
+          <mesh
+            filename="package://bender_description/meshes/visual/shoulder_roll.dae" />
+        </geometry>
+        <material
+          name="">
+          <color
+            rgba="0.1 0.1 0.1 1" />
+        </material>
       </visual>
       <collision>
@@ -132,5 +204,5 @@
       type="revolute">
       <origin
-        xyz="-0.02178 ${- reflect * 0.0339} -0.03"
+        xyz="-0.02402 ${- reflect * 0.0339} -0.03"
         rpy="0 0 0" />
       <parent
@@ -148,22 +220,34 @@
       <safety_controller soft_lower_limit="${shoulder_roll_joint_lower-soft_margin}" soft_upper_limit="${shoulder_roll_joint_upper+soft_margin}" k_position="30" k_velocity="30"/>
     </joint>
+    <!-- Shoulder yaw -->
     <link
       name="${prefix}${side}_shoulder_yaw_link">
       <inertial>
         <origin
-          xyz="${-17.25*TO_M} ${-0.20*TO_M} ${-151.64*TO_M}"
-          rpy="0 0 0" />
-        <mass value="${shoulder_yaw_mass}" />
-        <cuboid_inertia_def x="0.05" y="0.035" z="0.23" mass="${shoulder_yaw_mass}"/>
-      </inertial>
-      <visual>
-        <origin
-          xyz="0 0 0"
-          rpy="0 0 0" />
-        <geometry>
-          <mesh
-            filename="package://bender_description/meshes/visual/shoulder_yaw.stl" />
-        </geometry>
-        <material name="Grey1" />
+          xyz="-0.017828 -0.00016574 -0.14148"
+          rpy="0 0 0" />
+        <mass
+          value="0.17312" />
+        <inertia
+          ixx="0.0008473"
+          ixy="7.9313E-08"
+          ixz="3.4804E-05"
+          iyy="0.00084882"
+          iyz="-3.1674E-06"
+          izz="6.5527E-05" />
+      </inertial>
+      <visual>
+        <origin
+          xyz="0 0 0"
+          rpy="${-M_PI/2} 0 0" />
+        <geometry>
+          <mesh
+            filename="package://bender_description/meshes/visual/shoulder_yaw.dae" />
+        </geometry>
+        <material
+          name="">
+          <color
+            rgba="0.1 0.1 0.1 1" />
+        </material>
       </visual>
       <collision>
@@ -180,5 +264,5 @@
       type="revolute">
       <origin
-        xyz="0.03218 0 -0.1366"
+        xyz="0.03392 0 -0.1361"
         rpy="0 0 0" />
       <parent
@@ -196,22 +280,34 @@
       <safety_controller soft_lower_limit="${shoulder_yaw_joint_lower-soft_margin}" soft_upper_limit="${shoulder_yaw_joint_upper+soft_margin}" k_position="30" k_velocity="30"/>
     </joint>
+    <!-- Elbow pitch -->
     <link
       name="${prefix}${side}_elbow_pitch_link">
       <inertial>
         <origin
-          xyz="${7.17*TO_M} ${-21.86*TO_M} ${-60.81*TO_M}"
-          rpy="0 0 0" />
-        <mass value="${elbow_pitch_mass}" />
-        <cuboid_inertia_def x="0.05" y="0.07" z="0.10" mass="${elbow_pitch_mass}"/>
-      </inertial>
-      <visual>
-        <origin
-          xyz="0 0 0"
-          rpy="0 0 0" />
-        <geometry>
-          <mesh
-            filename="package://bender_description/meshes/visual/elbow_pitch.stl" />
-        </geometry>
-        <material name="Grey2" />
+          xyz="0.0067447 -0.022124 -0.059507"
+          rpy="0 0 0" />
+        <mass
+          value="0.14398" />
+        <inertia
+          ixx="0.00012531"
+          ixy="1.5127E-07"
+          ixz="3.5125E-06"
+          iyy="0.00011254"
+          iyz="-1.3346E-06"
+          izz="8.6928E-05" />
+      </inertial>
+      <visual>
+        <origin
+          xyz="0 0 0"
+          rpy="${-M_PI/2} 0 0" />
+        <geometry>
+          <mesh
+            filename="package://bender_description/meshes/visual/elbow_pitch.dae" />
+        </geometry>
+        <material
+          name="">
+          <color
+            rgba="0.1 0.1 0.1 1" />
+        </material>
       </visual>
       <collision>
@@ -228,5 +324,5 @@
       type="revolute">
       <origin
-        xyz="-0.015898 0.02178 -0.21"
+        xyz="-0.015898 0.022345 -0.21"
         rpy="0 0 0" />
       <parent
@@ -244,26 +340,38 @@
       <safety_controller soft_lower_limit="${elbow_pitch_joint_lower-soft_margin}" soft_upper_limit="${elbow_pitch_joint_upper+soft_margin}" k_position="30" k_velocity="30"/>
     </joint>
+    <!-- Elbow yaw -->
     <link
       name="${prefix}${side}_elbow_yaw_link">
       <inertial>
         <origin
-          xyz="${-19.08*TO_M} ${0.03*TO_M} ${-152.08*TO_M}"
-          rpy="0 0 0" />
-        <mass value="${elbow_yaw_mass}" />
-        <cuboid_inertia_def x="0.05" y="0.035" z="0.32" mass="${elbow_yaw_mass}"/>
-      </inertial>
-      <visual>
-        <origin
-          xyz="0 0 0"
-          rpy="0 0 0" />
-        <geometry>
-          <mesh
-            filename="package://bender_description/meshes/visual/elbow_yaw.stl" />
-        </geometry>
-        <material name="Grey1"/>
-      </visual>
-      <collision>
-        <origin
-          xyz="-0.015 0 -0.12"
+          xyz="-0.0196 8.4626E-05 -0.17771"
+          rpy="0 0 0" />
+        <mass
+          value="0.1675" />
+        <inertia
+          ixx="0.0017359"
+          ixy="-4.8507E-09"
+          ixz="3.1814E-05"
+          iyy="0.0017441"
+          iyz="2.1946E-07"
+          izz="5.881E-05" />
+      </inertial>
+      <visual>
+        <origin
+          xyz="0 0 0"
+          rpy="${-M_PI/2} 0 0" />
+        <geometry>
+          <mesh
+            filename="package://bender_description/meshes/visual/elbow_yaw.dae" />
+        </geometry>
+        <material
+          name="">
+          <color
+            rgba="0.1 0.1 0.1 1" />
+        </material>
+      </visual>
+      <collision>
+        <origin
+          xyz="-0.015 0 -0.15"
           rpy="0 0 0" />
         <geometry>
@@ -276,5 +384,5 @@
       type="revolute">
       <origin
-        xyz="-0.0136 -0.02228 -0.09218"
+        xyz="-0.0136 -0.022345 -0.0519"
         rpy="0 0 0" />
       <parent
@@ -292,22 +400,34 @@
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
File: bender_common/bender_description/urdf/gazebo.urdf.xacro (robot description, xacro)
@@ -47,5 +47,4 @@
   <xacro:macro name="gazebo_link" params="link color">
     <gazebo reference="${link}">
-      <material>Gazebo/${color}</material>
       <mu1>0.2</mu1>
       <mu2>0.2</mu2>
@@ -53,7 +52,6 @@
   </xacro:macro>
   <!-- Wheel links -->
-  <xacro:macro name="gazebo_wheel_link" params="link color reflect">
+  <xacro:macro name="gazebo_wheel_link" params="link reflect">
     <gazebo reference="${link}">
-      <material>Gazebo/${color}</material>
       <kp>1000000.0</kp>
       <!-- kp and kd for rubber -->
@@ -75,4 +73,5 @@
   <xacro:macro name="gazebo_friction_link" params="link color">
     <gazebo reference="${link}">
+      <selfCollide>true</selfCollide>
       <material>Gazebo/${color}</material>
       <minDepth>0.005</minDepth>

File: bender_common/bender_description/urdf/gripper.urdf.xacro (robot description, xacro)
@@ -11,6 +11,4 @@
     <xacro:joint_transmission joint="${side}_int_finger_joint"/>
     <xacro:joint_transmission joint="${side}_ext_finger_joint"/>
-    <link
-      name="${prefix}${side}_base_int_finger_link" />
     <joint
       name="${side}_int_finger_joint"
@@ -18,18 +16,18 @@
       <xacro:if value="${(reflect+1)/2}">
         <origin
-          xyz="0.01775 0.00085 -0.0794"
-          rpy="${reflect * M_PI / 6} 0 0" />
+          xyz="0 0 0"
+          rpy="${M_PI/6} 0 0" />
       </xacro:if>
       <xacro:unless value="${(reflect+1)/2}">
         <origin
-          xyz="0.01775 -0.03555 -0.0794"
-          rpy="${reflect * M_PI / 6} 0 0" />
+          xyz="-0.0275 0 0"
+          rpy="${M_PI/6} 0 ${M_PI}" />
       </xacro:unless>
       <parent
-        link="${prefix}${side}_wrist_pitch_link" />
+        link="${prefix}${side}_int_finger_mount_link" />
       <child
-        link="${prefix}${side}_base_int_finger_link" />
+        link="${prefix}${side}_int_finger_link" />
       <axis
-        xyz="${reflect} 0 0" />
+        xyz="1 0 0" />
       <limit
         upper="${int_finger_joint_upper}"
@@ -39,6 +37,4 @@
       <dynamics damping="${damping}" friction="${friccion}" />
     </joint>
-    <link
-      name="${prefix}${side}_base_ext_finger_link" />
     <joint
       name="${side}_ext_finger_joint"
@@ -46,18 +42,18 @@
       <xacro:if value="${(reflect+1)/2}">
         <origin
-          xyz="0.01775 -0.03555 -0.0794"
-          rpy="${- reflect * M_PI / 6} 0 0" />
+          xyz="-0.0275 0 0"
+          rpy="${M_PI/6} 0 ${M_PI}" />
       </xacro:if>
       <xacro:unless value="${(reflect+1)/2}">
         <origin
-          xyz="0.01775 0.00085 -0.0794"
-          rpy="${- reflect * M_PI / 6} 0 0" />
+          xyz="0 0 0"
+          rpy="${M_PI/6} 0 0" />
       </xacro:unless>
       <parent
-        link="${prefix}${side}_wrist_pitch_link" />
+        link="${prefix}${side}_ext_finger_mount_link" />
       <child
-        link="${prefix}${side}_base_ext_finger_link" />
+        link="${prefix}${side}_ext_finger_link" />
       <axis
-        xyz="${-reflect} 0 0" />
+        xyz="1 0 0" />
       <limit
         upper="${ext_finger_joint_upper}"
@@ -69,5 +65,5 @@
   </xacro:macro>
   <!-- Gripper type -->
-  <xacro:macro name="gripper_type" params="type">
+  <xacro:macro name="gripper_type" params="type ext">
     <xacro:if value="${type}">
       <inertial>
@@ -79,7 +75,14 @@
       </inertial>
       <visual>
+        <xacro:if value="${ext}">
         <origin
           xyz="0 0 0"
           rpy="0 0 0" />
+        </xacro:if>
+        <xacro:unless value="${ext}">
+        <origin
+          xyz="0.008 0 0"
+          rpy="0 0 0" />
+        </xacro:unless>
         <geometry>
           <mesh
@@ -89,7 +92,14 @@
       </visual>
       <collision>
+        <xacro:if value="${ext}">
         <origin
           xyz="0 0 0.011"
           rpy="0 0 0" />
+        </xacro:if>
+        <xacro:unless value="${ext}">
+        <origin
+          xyz="0.005 0 0.011"
+          rpy="0 0 0" />
+        </xacro:unless>
         <geometry>
           <mesh
@@ -107,7 +117,14 @@
       </inertial>
       <visual>
+        <xacro:if value="${ext}">
+        <origin
+          xyz="0.008 0 0"
+          rpy="0 0 0" />
+        </xacro:if>
+        <xacro:unless value="${ext}">
         <origin
           xyz="0 0 0"
           rpy="0 0 0" />
+        </xacro:unless>
         <geometry>
           <mesh
@@ -117,7 +134,14 @@
       </visual>
       <collision>
+        <xacro:if value="${ext}">
+        <origin
+          xyz="0.0355 0 0.011"
+          rpy="0 0 0" />
+        </xacro:if>
+        <xacro:unless value="${ext}">
         <origin
           xyz="0.0275 0 0.011"
           rpy="0 0 0" />
+        </xacro:unless>
         <geometry>
           <mesh
@@ -131,27 +155,7 @@
     <link
     name="${prefix}${side}_int_finger_link">
-      <xacro:gripper_type type="${type}" />
+      <xacro:gripper_type type="${type}" ext="0"/>
     </link>
     <xacro:gazebo_friction_link link="${prefix}${side}_int_finger_link" color="DarkGrey" />
-    <joint
-      name="${side}_int_finger_fixed_joint"
-      type="fixed">
-      <xacro:if value="${(reflect+1)/2}">
-        <origin
-          xyz="0 0 0"
-          rpy="0 0 0" />
-      </xacro:if >
-      <xacro:unless value="${(reflect+1)/2}">
-        <origin
-          xyz="-0.035 0 0"
-          rpy="0 0 ${-M_PI}" />
-      </xacro:unless >
-      <parent
-        link="${prefix}${side}_base_int_finger_link" />
-      <child
-        link="${prefix}${side}_int_finger_link" />
-      <axis
-        xyz="0 0 0" />
-    </joint>
   </xacro:macro>
   <!-- Gripper exterior, type 1 - 2 finger, type 0 - 1 finger -->
@@ -159,27 +163,7 @@
     <link
     name="${prefix}${side}_ext_finger_link">
-      <xacro:gripper_type type="${type}" />
+      <xacro:gripper_type type="${type}" ext="1"/>
     </link>
     <xacro:gazebo_friction_link link="${prefix}${side}_ext_finger_link" color="DarkGrey" />
-    <joint
-      name="${side}_ext_finger_fixed_joint"
-      type="fixed">
-      <xacro:unless value="${(reflect+1)/2}">
-        <origin
-          xyz="0 0 0"
-          rpy="0 0 0" />
-      </xacro:unless >
-      <xacro:if value="${(reflect+1)/2}">
-        <origin
-          xyz="-0.035 0 0"
-          rpy="0 0 ${-M_PI}" />
-      </xacro:if >
-      <parent
-        link="${prefix}${side}_base_ext_finger_link" />
-      <child
-        link="${prefix}${side}_ext_finger_link" />
-      <axis
-        xyz="0 0 0" />
-    </joint>
   </xacro:macro>
 </robot>
