Commit message: New URDF

File: bender_common/bender_description/urdf/head.urdf.xacro (robot description, xacro)
@@ -1,83 +1,59 @@
 <?xml version="1.0"?>
-<robot
-  xmlns:xacro="http://www.ros.org/wiki/xacro"
-  name="bender_head">
-  <xacro:macro name="head" params="parent prefix" >
-    <!-- Gazebo Links material -->
+<robot name="mask_head" xmlns:xacro="http://ros.org/wiki/xacro">
+    <xacro:property name="head_pitch_joint_lower" value="-0.39372" />
+    <xacro:property name="head_pitch_joint_upper" value="0.88459" />
+    <xacro:property name="head_yaw_joint_upper"   value="1.89190" />
+    <xacro:property name="head_yaw_joint_lower"   value="-1.89190" />
+    <!-- Torque -->
+    <xacro:property name="head_yaw_torque"   value="${rx64_torque}" />
+    <xacro:property name="head_pitch_torque" value="${rx64_torque}" />
+  <xacro:macro name="head" params="parent prefix ns">
+    <!-- Gazebo Links material
     <xacro:gazebo_link link="${prefix}neck_link" color="Grey" />
-    <xacro:gazebo_link link="${prefix}head_link" color="Grey" />
+    <xacro:gazebo_link link="${prefix}face_link" color="Grey" />
+    <xacro:gazebo_link link="${prefix}head_link" color="DarkGrey" />
+    -->
     <!-- Transmissions -->
-    <xacro:joint_transmission joint="neck_yaw_joint"/>
+    <xacro:joint_transmission joint="head_yaw_joint"/>
+    <xacro:joint_transmission joint="head_pitch_joint"/>
     <link
       name="${prefix}neck_link">
       <inertial>
         <origin
-          xyz="0 0 0.04"
-          rpy="0 0 0" />
-        <mass value="0.05" />
-        <cuboid_inertia_def x="0.06" y="0.06" z="0.08" mass="0.05"/>
+          xyz="-0.027227 -1.1356E-07 0.017004"
+          rpy="0 0 0" />
+        <mass
+          value="0.092467" />
+        <inertia
+          ixx="0.00013489"
+          ixy="-3.52E-09"
+          ixz="-6.6205E-07"
+          iyy="7.5254E-05"
+          iyz="1.356E-10"
+          izz="0.00012174" />
       </inertial>
       <visual>
         <origin
           xyz="0 0 0"
-          rpy="0 0 0" />
+          rpy="${-M_PI/2} 0 0" />
         <geometry>
           <mesh
-            filename="package://bender_description/meshes/visual/neck.stl" />
-        </geometry>
-        <material name="Head" />
+            filename="package://bender_description/meshes/visual/neck.dae" />
+        </geometry>
+        <material name="Grey3" />
       </visual>
       <collision>
         <origin
-          xyz="0 0 0.04"
-          rpy="0 0 0" />
-        <geometry>
-          <box size="0.06 0.06 0.08"/>
+          xyz="-0.03 0 0.02"
+          rpy="0 0 0" />
+        <geometry>
+          <box size="0.08 0.1 0.08"/>
         </geometry>
       </collision>
     </link>
-    <joint
-      name="right_eye_joint"
-      type="fixed">
-      <origin
-        xyz="0.1 0.04 0.18"
-        rpy="0 0 0" />
-      <child
-        link="${prefix}sensors/camera_right_eye_link" />
-      <parent
-        link="${prefix}neck_link" />
-    </joint>
-    <joint
-      name="left_eye_joint"
-      type="fixed">
-      <origin
-        xyz="0.1 -0.04 0.18"
-        rpy="0 0 0" />
-      <child
-        link="${prefix}sensors/camera_left_eye_link" />
-      <parent
-        link="${prefix}neck_link" />
-    </joint>
-    <link
-      name="${prefix}sensors/camera_right_eye_link"  >
-       <xacro:dummy_inertial/>
-    </link>
-    <link
-      name="${prefix}sensors/camera_left_eye_link"  >
-       <xacro:dummy_inertial/>
-    </link>
-    <joint
-      name="neck_yaw_joint"
-      type="revolute">
-      <origin
-        xyz="0 0 0"
-        rpy="0 0 0" />
-      <parent
-        link="${parent}" />
-      <child
-        link="${prefix}neck_link" />
-      <axis xyz="0 0 1" />
-      <limit effort="${effort_head}" lower="${- M_PI / 4}" upper="${M_PI / 4}" velocity="${vel_head}"/>
-      <dynamics damping="${damping}" friction="${friccion}" />
+    <joint name="neck_mount_fixed_joint" type="fixed">
+      <origin xyz="0 0 0" rpy="0 0 0" />
+      <parent link="${parent}"/>
+      <child link="${prefix}neck_link" />
     </joint>
     <link
@@ -85,56 +61,154 @@
       <inertial>
         <origin
-          xyz="0.02 0.06 0.1"
-          rpy="0 0 0" />
-        <mass value="1.0" />
-        <cuboid_inertia_def x="0.18" y="0.18" z="0.2" mass="1.0"/>
+          xyz="-0.012141 -1.7505E-05 0.041401"
+          rpy="0 0 0" />
+        <mass
+          value="0.17983" />
+        <inertia
+          ixx="0.00015925"
+          ixy="4.0867E-07"
+          ixz="-7.9102E-06"
+          iyy="0.0001892"
+          iyz="-6.1427E-08"
+          izz="8.7881E-05" />
       </inertial>
       <visual>
         <origin
           xyz="0 0 0"
-          rpy="0 0 0" />
+          rpy="${-M_PI/2} 0 0" />
         <geometry>
           <mesh
-            filename="package://bender_description/meshes/visual/head.stl" />
-        </geometry>
-        <material name="Head" />
+            filename="package://bender_description/meshes/visual/head.dae" />
+        </geometry>
+        <material name="Grey3" />
       </visual>
       <collision>
         <origin
-          xyz="0.02 0.06 0.1"
-          rpy="0 0 0" />
-        <geometry>
-          <box size="0.18 0.18 0.2"/>
+          xyz="-0.01 0 0.05"
+          rpy="0 0 0" />
+        <geometry>
+          <box size="0.08 0.06 0.10"/>
         </geometry>
       </collision>
     </link>
     <joint
+      name="head_yaw_joint"
+      type="revolute">
+      <origin
+        xyz="-0.027 0 0.0529"
+        rpy="0 0 0" />
+      <parent
+        link="${prefix}neck_link" />
+      <child
+        link="${prefix}head_link" />
+      <axis
+        xyz="0 0 1" />
+      <limit
+        effort="${head_yaw_torque}"
+        velocity="1.0"
+        upper="${head_yaw_joint_upper}"
+        lower="${head_yaw_joint_lower}" />
+        <dynamics damping="${dxl_damping}"/>
+    </joint>
+    <link
+      name="${prefix}face_link">
+      <inertial>
+        <origin
+          xyz="0.046115 -0.026111 0.10189"
+          rpy="0 0 0" />
+        <mass
+          value="0.33187" />
+        <inertia
+          ixx="0.0013461"
+          ixy="-2.8029E-07"
+          ixz="-9.224E-05"
+          iyy="0.00080978"
+          iyz="-6.6351E-07"
+          izz="0.00074443" />
+      </inertial>
+      <visual>
+        <origin
+          xyz="0 0 0"
+          rpy="${-M_PI/2} 0 0" />
+        <geometry>
+          <mesh
+            filename="package://bender_description/meshes/visual/face.dae" />
+        </geometry>
+        <material name="Grey3" />
+      </visual>
+      <collision>
+        <origin
+          xyz="0.05 -0.03 0.08"
+          rpy="0 0 0" />
+        <geometry>
+          <box size="0.05 0.18 0.18"/>
+        </geometry>
+      </collision>
+    </link>
+    <joint
       name="head_pitch_joint"
+      type="revolute">
+      <origin
+        xyz="0 0.02598 0.0679"
+        rpy="0 0 0" />
+      <parent
+        link="${prefix}head_link" />
+      <child
+        link="${prefix}face_link" />
+      <axis
+        xyz="0 1 0" />
+      <limit
+        effort="${head_pitch_torque}"
+        velocity="1.0"
+        upper="${head_pitch_joint_upper}"
+        lower="${head_pitch_joint_lower}"/>
+      <dynamics damping="${dxl_damping}"/>
+    </joint>
+    <!-- Camera RGB and depth frames -->
+    <link
+      name="${prefix}sensors/rgbd_head_rgb_frame" />
+    <joint
+      name="rgbd_head_rgb_joint"
       type="fixed">
       <origin
-        xyz="0 -0.0585 0.067"
-        rpy="0 0 0" />
-      <parent
-        link="${prefix}neck_link" />
-      <child
-        link="${prefix}head_link" />
-    </joint>
-    <link
-      name="${prefix}head_up_link"  >
-       <xacro:dummy_inertial/>
-    </link>
-    <joint
-      name="head_up_joint"
+        xyz="0.05332 -0.0042 0.14105"
+        rpy="0 0.031904 0" />
+      <parent
+        link="${prefix}face_link" />
+      <child
+        link="${prefix}sensors/rgbd_head_rgb_frame" />
+      <axis
+        xyz="0 0 0" />
+    </joint>
+    <link
+      name="${prefix}sensors/rgbd_head_depth_frame" />
+    <joint
+      name="rgbd_head_depth_joint"
       type="fixed">
       <origin
-        xyz="0.017 0.0585 0.17"
-        rpy="0 0 0" />
-      <parent
-        link="${prefix}head_link" />
-      <child
-        link="${prefix}head_up_link" />
-      <axis
-        xyz="1 0 0" />
-    </joint>
+        xyz="0.05332 0.0208 0.14105"
+        rpy="0 0.031904 0" />
+      <parent
+        link="${prefix}face_link" />
+      <child
+        link="${prefix}sensors/rgbd_head_depth_frame" />
+      <axis
+        xyz="0 0 0" />
+    </joint>
+    <!-- Optical frames -->
+    <joint name="rgbd_head_rgb_optical_joint" type="fixed">
+      <origin xyz="0 0 0" rpy="${-M_PI/2} 0 ${-M_PI/2}" />
+      <parent link="${prefix}sensors/rgbd_head_rgb_frame" />
+      <child link="${prefix}sensors/rgbd_head_rgb_optical_frame" />
+    </joint>
+    <link name="${prefix}sensors/rgbd_head_rgb_optical_frame"/>
+    <joint name="rgbd_head_depth_optical_joint" type="fixed">
+      <origin xyz="0 0 0" rpy="${-M_PI/2} 0 ${-M_PI/2}" />
+      <parent link="${prefix}sensors/rgbd_head_depth_frame" />
+      <child link="${prefix}sensors/rgbd_head_depth_optical_frame" />
+    </joint>
+    <link name="${prefix}sensors/rgbd_head_depth_optical_frame"/>
+    <!-- Camera depth Gazebo -->
+    <xacro:sim_depth_camera name="rgbd_head" frame="${prefix}sensors/rgbd_head_depth" ns="${ns}"/>
   </xacro:macro>
 </robot>

File: bender_common/bender_description/urdf/laser_sensor.xacro (robot description, xacro)
@@ -21,4 +21,9 @@
           <mesh filename="package://bender_description/meshes/sensors/hokuyo.dae"/>
         </geometry>
+        <material
+          name="">
+          <color
+            rgba="0.1 0.1 0.1 1" />
+        </material>
       </visual>
       <xacro:cuboid_inertia_def x="0.05" y="0.05" z="0.05" mass="0.3"/>

Commit message: fix urdf

File: bender_common/bender_description/urdf/arm.urdf.xacro (robot description, xacro)
@@ -133,8 +133,8 @@
       <collision>
         <origin
-          xyz="0 ${- reflect * 0.02} 0"
-          rpy="0 0 0" />
-        <geometry>
-          <box size="0.05 0.07 0.07"/>
+          xyz="0 ${- reflect * 0.025} -0.01"
+          rpy="0 0 0" />
+        <geometry>
+          <box size="0.05 0.05 0.07"/>
         </geometry>
       </collision>
