Commit message: merging develop to feat-calibration

File: bender_common/bender_description/urdf/arm.urdf.xacro (robot description, xacro)
@@ -2,6 +2,5 @@
 <robot
   xmlns:xacro="http://www.ros.org/wiki/xacro"
-  name="bender_arm">
-  <xacro:include filename="$(find bender_description)/urdf/gripper.urdf.xacro" />
+  name="arm">
   <!-- Soft margin 5 deg -->
   <xacro:property name="soft_margin" value="${M_PI/36}" />
@@ -19,25 +18,12 @@
   <xacro:property name="shoulder_roll_joint_upper" value="1.51096" />
   <xacro:property name="shoulder_roll_joint_lower" value="-0.23776" />
-  <!-- Links mass -->
-  <xacro:property name="link_mass" value="1.0" />
-  <xacro:property name="elbow_yaw_mass" value="${link_mass}" />
-  <xacro:property name="elbow_pitch_mass" value="${link_mass}" />
-  <xacro:property name="shoulder_yaw_mass" value="${link_mass}" />
-  <xacro:property name="shoulder_pitch_mass" value="${link_mass}" />
-  <xacro:property name="wrist_pitch_mass" value="${link_mass}" />
-  <xacro:property name="shoulder_roll_mass" value="${link_mass}" />
-  <!-- Effort -->
-  <xacro:property name="effort_shoulder" value="80" />
-  <xacro:property name="effort_elbow" value="30" />
-  <xacro:property name="effort_wrisp" value="15" />
-  <xacro:macro name="bender_arm" params="side parent reflect prefix">
-    <!-- Gazebo elements -->
-    <!-- Gazebo Links material -->
-    <xacro:gazebo_link link="${prefix}${side}_shoulder_pitch_link" color="DarkGrey" />
-    <xacro:gazebo_link link="${prefix}${side}_shoulder_roll_link" color="Grey" />
-    <xacro:gazebo_link link="${prefix}${side}_shoulder_yaw_link" color="DarkGrey" />
-    <xacro:gazebo_link link="${prefix}${side}_elbow_pitch_link" color="Grey" />
-    <xacro:gazebo_link link="${prefix}${side}_elbow_yaw_link" color="DarkGrey" />
-    <xacro:gazebo_link link="${prefix}${side}_wrist_pitch_link" color="Grey" />
+  <!-- Torque -->
+  <xacro:property name="shoulder_pitch_torque" value="${mx106_torque}" />
+  <xacro:property name="shoulder_roll_torque"  value="${mx106_torque}" />
+  <xacro:property name="shoulder_yaw_torque"   value="${rx64_torque}" />
+  <xacro:property name="elbow_pitch_torque"    value="${mx106_torque}" />
+  <xacro:property name="elbow_yaw_torque"      value="${rx64_torque}" />
+  <xacro:property name="wrist_pitch_torque"    value="${rx28_torque}" />
+  <xacro:macro name="arm" params="side parent reflect prefix">
     <!-- Transmissions -->
     <xacro:joint_transmission joint="${side}_shoulder_pitch_joint"/>
@@ -47,29 +33,108 @@
     <xacro:joint_transmission joint="${side}_elbow_yaw_joint"/>
     <xacro:joint_transmission joint="${side}_wrist_pitch_joint"/>
+    <!-- Base fixed joint and link -->
+    <joint
+      name="${side}_arm_base_fixed_joint"
+      type="fixed">
+      <origin
+        xyz="0 0 0"
+        rpy="0 0 0" />
+      <parent
+        link="${parent}" />
+      <child
+        link="${prefix}${side}_arm_base_link" />
+      <axis
+        xyz="0 0 0" />
+    </joint>
+    <link
+      name="${prefix}${side}_arm_base_link">
+      <inertial>
+        <origin
+          xyz="3.1697E-06 -0.017088 0.00063087"
+          rpy="0 0 0" />
+        <mass
+          value="0.17471" />
+        <inertia
+          ixx="0.00037909"
+          ixy="7.4755E-09"
+          ixz="2.8692E-09"
+          iyy="0.00040178"
+          iyz="8.0104E-07"
+          izz="9.5869E-05" />
+      </inertial>
+      <visual>
+        <xacro:if value="${(reflect+1)/2}">
+        <origin
+          xyz="0 0 0"
+          rpy="${-M_PI/2} 0 ${M_PI}" />
+        </xacro:if >
+        <xacro:unless value="${(reflect+1)/2}">
+        <origin
+          xyz="0 0 0"
+          rpy="${-M_PI/2} 0 0" />
+        </xacro:unless >
+        <geometry>
+          <mesh
+            filename="package://bender_description/meshes/visual/shoulder_base_link.dae" />
+        </geometry>
+        <material
+          name="">
+          <color
+            rgba="0.1 0.1 0.1 1" />
+        </material>
+      </visual>
+      <collision>
+        <origin
+          xyz="0 ${reflect * 0.03} 0"
+          rpy="0 0 0" />
+        <geometry>
+          <box size="0.07 0.06 0.17"/>
+        </geometry>
+      </collision>
+    </link>
+    <!-- Shoulder pitch -->
     <link
       name="${prefix}${side}_shoulder_pitch_link">
       <inertial>
         <origin
-          xyz="0 ${- reflect * 0.02} 0"
-          rpy="0 0 0" />
-        <mass value="${shoulder_pitch_mass}" />
-        <cuboid_inertia_def x="0.05" y="0.07" z="0.07" mass="${shoulder_pitch_mass}"/>
-      </inertial>
-      <visual>
-        <origin
-          xyz="0 0 0"
-          rpy="0 0 0" />
-        <geometry>
-          <mesh
-            filename="package://bender_description/meshes/visual/${side}_shoulder_pitch.stl" />
-        </geometry>
-        <material name="Grey1" />
-      </visual>
-      <collision>
-        <origin
-          xyz="0 ${- reflect * 0.02} 0"
-          rpy="0 0 0" />
-        <geometry>
-          <box size="0.05 0.07 0.07"/>
+          xyz="0.00023251 0.019812 -0.013482"
+          rpy="0 0 0" />
+        <mass
+          value="0.17152" />
+        <inertia
+          ixx="0.00010991"
+          ixy="-5.6413E-07"
+          ixz="1.0935E-06"
+          iyy="0.00010993"
+          iyz="1.8807E-06"
+          izz="8.8167E-05" />
+      </inertial>
+      <visual>
+        <xacro:if value="${(reflect+1)/2}">
+        <origin
+          xyz="0 0 0"
+          rpy="${-M_PI/2} 0 ${M_PI}" />
+        </xacro:if >
+        <xacro:unless value="${(reflect+1)/2}">
+        <origin
+          xyz="0 0 0"
+          rpy="${-M_PI/2} 0 0" />
+        </xacro:unless >
+        <geometry>
+          <mesh
+            filename="package://bender_description/meshes/visual/shoulder_pitch.dae" />
+        </geometry>
+        <material
+          name="">
+          <color
+            rgba="0.1 0.1 0.1 1" />
+        </material>
+      </visual>
+      <collision>
+        <origin
+          xyz="0 ${- reflect * 0.025} -0.01"
+          rpy="0 0 0" />
+        <geometry>
+          <box size="0.05 0.05 0.07"/>
         </geometry>
       </collision>
@@ -79,8 +144,8 @@
       type="revolute">
       <origin
-        xyz="0 0 0"
-        rpy="0 0 0" />
-      <parent
-        link="${parent}" />
+        xyz="0 ${- reflect * 0.0046} 0.0176"
+        rpy="0 0 0" />
+      <parent
+        link="${prefix}${side}_arm_base_link" />
       <child
         link="${prefix}${side}_shoulder_pitch_link" />
@@ -88,34 +153,46 @@
         xyz="0 -1 0" />
       <limit
-        effort="${effort_shoulder}"
+        effort="${shoulder_pitch_torque}"
         lower="${shoulder_pitch_joint_lower}"
         upper="${shoulder_pitch_joint_upper}"
         velocity="${vel_arm * M_PI / 180}"/>
-      <dynamics damping="${damping}" friction="${friccion}" />
+      <dynamics damping="${dxl_damping}" friction="${dxl_friction}" />
       <safety_controller soft_lower_limit="${shoulder_pitch_joint_lower-soft_margin}" soft_upper_limit="${shoulder_pitch_joint_upper+soft_margin}" k_position="30" k_velocity="30"/>
     </joint>
+    <!-- Shoulder roll -->
     <link
       name="${prefix}${side}_shoulder_roll_link">
       <inertial>
+        <origin
+          xyz="0.046779 -9.3259E-06 -0.11466"
+          rpy="0 0 0" />
+        <mass
+          value="0.16104" />
+        <inertia
+          ixx="0.00050901"
+          ixy="6.2439E-09"
+          ixz="0.00010534"
+          iyy="0.00055051"
+          iyz="-6.7534E-08"
+          izz="0.00011428" />
+      </inertial>
+      <visual>
+        <origin
+          xyz="0 0 0"
+          rpy="${-M_PI/2} 0 0" />
+        <geometry>
+          <mesh
+            filename="package://bender_description/meshes/visual/shoulder_roll.dae" />
+        </geometry>
+        <material
+          name="">
+          <color
+            rgba="0.1 0.1 0.1 1" />
+        </material>
+      </visual>
+      <collision>
         <origin
           xyz="0.04 0 -0.075"
           rpy="0 -0.25 0" />
-        <mass value="${shoulder_roll_mass}" />
-        <cuboid_inertia_def x="0.05" y="0.035" z="0.18" mass="${shoulder_roll_mass}"/>
-      </inertial>
-      <visual>
-        <origin
-          xyz="0 0 0"
-          rpy="0 0 0" />
-        <geometry>
-          <mesh
-            filename="package://bender_description/meshes/visual/shoulder_roll.stl" />
-        </geometry>
-        <material name="Grey2" />
-      </visual>
-      <collision>
-        <origin
-          xyz="0.04 0 -0.075"
-          rpy="0 -0.25 0" />
         <geometry>
           <box size="0.05 0.035 0.18"/>
@@ -127,5 +204,5 @@
       type="revolute">
       <origin
-        xyz="-0.02178 ${- reflect * 0.0339} -0.03"
+        xyz="-0.02402 ${- reflect * 0.0339} -0.03"
         rpy="0 0 0" />
       <parent
@@ -138,27 +215,39 @@
         lower="${shoulder_roll_joint_lower}"
         upper="${shoulder_roll_joint_upper}"
-        effort="${effort_shoulder}"
+        effort="${shoulder_roll_torque}"
         velocity="${vel_arm * M_PI / 180}" />
-      <dynamics damping="${damping}" friction="${friccion}" />
+      <dynamics damping="${dxl_damping}" friction="${dxl_friction}" />
       <safety_controller soft_lower_limit="${shoulder_roll_joint_lower-soft_margin}" soft_upper_limit="${shoulder_roll_joint_upper+soft_margin}" k_position="30" k_velocity="30"/>
     </joint>
+    <!-- Shoulder yaw -->
     <link
       name="${prefix}${side}_shoulder_yaw_link">
       <inertial>
         <origin
-          xyz="-0.015 0 -0.115"
-          rpy="0 0 0" />
-        <mass value="${shoulder_yaw_mass}" />
-        <cuboid_inertia_def x="0.05" y="0.035" z="0.23" mass="${shoulder_yaw_mass}"/>
-      </inertial>
-      <visual>
-        <origin
-          xyz="0 0 0"
-          rpy="0 0 0" />
-        <geometry>
-          <mesh
-            filename="package://bender_description/meshes/visual/shoulder_yaw.stl" />
-        </geometry>
-        <material name="Grey1" />
+          xyz="-0.017828 -0.00016574 -0.14148"
+          rpy="0 0 0" />
+        <mass
+          value="0.17312" />
+        <inertia
+          ixx="0.0008473"
+          ixy="7.9313E-08"
+          ixz="3.4804E-05"
+          iyy="0.00084882"
+          iyz="-3.1674E-06"
+          izz="6.5527E-05" />
+      </inertial>
+      <visual>
+        <origin
+          xyz="0 0 0"
+          rpy="${-M_PI/2} 0 0" />
+        <geometry>
+          <mesh
+            filename="package://bender_description/meshes/visual/shoulder_yaw.dae" />
+        </geometry>
+        <material
+          name="">
+          <color
+            rgba="0.1 0.1 0.1 1" />
+        </material>
       </visual>
       <collision>
@@ -175,5 +264,5 @@
       type="revolute">
       <origin
-        xyz="0.03218 0 -0.1366"
+        xyz="0.03392 0 -0.1361"
         rpy="0 0 0" />
       <parent
@@ -186,27 +275,39 @@
         lower="${shoulder_yaw_joint_lower}"
         upper="${shoulder_yaw_joint_upper}"
-        effort="${effort_shoulder}"
+        effort="${shoulder_yaw_torque}"
         velocity="${vel_arm * M_PI / 180}" />
-      <dynamics damping="${damping}" friction="${friccion}" />
+      <dynamics damping="${dxl_damping}" friction="${dxl_friction}" />
       <safety_controller soft_lower_limit="${shoulder_yaw_joint_lower-soft_margin}" soft_upper_limit="${shoulder_yaw_joint_upper+soft_margin}" k_position="30" k_velocity="30"/>
     </joint>
+    <!-- Elbow pitch -->
     <link
       name="${prefix}${side}_elbow_pitch_link">
       <inertial>
         <origin
-          xyz="0.015 -0.025 -0.05"
-          rpy="0 0 0" />
-        <mass value="${elbow_pitch_mass}" />
-        <cuboid_inertia_def x="0.05" y="0.07" z="0.10" mass="${elbow_pitch_mass}"/>
-      </inertial>
-      <visual>
-        <origin
-          xyz="0 0 0"
-          rpy="0 0 0" />
-        <geometry>
-          <mesh
-            filename="package://bender_description/meshes/visual/elbow_pitch.stl" />
-        </geometry>
-        <material name="Grey2" />
+          xyz="0.0067447 -0.022124 -0.059507"
+          rpy="0 0 0" />
+        <mass
+          value="0.14398" />
+        <inertia
+          ixx="0.00012531"
+          ixy="1.5127E-07"
+          ixz="3.5125E-06"
+          iyy="0.00011254"
+          iyz="-1.3346E-06"
+          izz="8.6928E-05" />
+      </inertial>
+      <visual>
+        <origin
+          xyz="0 0 0"
+          rpy="${-M_PI/2} 0 0" />
+        <geometry>
+          <mesh
+            filename="package://bender_description/meshes/visual/elbow_pitch.dae" />
+        </geometry>
+        <material
+          name="">
+          <color
+            rgba="0.1 0.1 0.1 1" />
+        </material>
       </visual>
       <collision>
@@ -223,5 +324,5 @@
       type="revolute">
       <origin
-        xyz="-0.015898 0.02178 -0.21"
+        xyz="-0.015898 0.022345 -0.21"
         rpy="0 0 0" />
       <parent
@@ -234,31 +335,43 @@
         lower="${elbow_pitch_joint_lower}"
         upper="${elbow_pitch_joint_upper}"
-        effort="${effort_elbow}"
+        effort="${elbow_pitch_torque}"
         velocity="${vel_arm * M_PI / 180}" />
-      <dynamics damping="${damping}" friction="${friccion}" />
+      <dynamics damping="${dxl_damping}" friction="${dxl_friction}" />
       <safety_controller soft_lower_limit="${elbow_pitch_joint_lower-soft_margin}" soft_upper_limit="${elbow_pitch_joint_upper+soft_margin}" k_position="30" k_velocity="30"/>
     </joint>
+    <!-- Elbow yaw -->
     <link
       name="${prefix}${side}_elbow_yaw_link">
       <inertial>
         <origin
-          xyz="-0.015 0 -0.12"
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
File: bender_common/bender_description/urdf/gazebo.urdf.xacro (robot description, xacro)
@@ -47,5 +47,4 @@
   <xacro:macro name="gazebo_link" params="link color">
     <gazebo reference="${link}">
-      <material>Gazebo/${color}</material>
       <mu1>0.2</mu1>
       <mu2>0.2</mu2>
@@ -53,7 +52,6 @@
   </xacro:macro>
   <!-- Wheel links -->
-  <xacro:macro name="gazebo_wheel_link" params="link color reflect">
-    <gazebo reference="${link}">
-      <material>Gazebo/${color}</material>
+  <xacro:macro name="gazebo_wheel_link" params="link reflect">
+    <gazebo reference="${link}">
       <kp>1000000.0</kp>
       <!-- kp and kd for rubber -->
@@ -75,4 +73,5 @@
   <xacro:macro name="gazebo_friction_link" params="link color">
     <gazebo reference="${link}">
+      <selfCollide>true</selfCollide>
       <material>Gazebo/${color}</material>
       <minDepth>0.005</minDepth>
@@ -105,6 +104,6 @@
           <updateRate>5.0</updateRate>
           <cameraName>${name}</cameraName>
-          <imageTopicName>${ns}/ir/image_raw</imageTopicName>
-          <cameraInfoTopicName>${ns}/ir/camera_info</cameraInfoTopicName>
+          <imageTopicName>${ns}/rgb/image_raw</imageTopicName>
+          <cameraInfoTopicName>${ns}/rgb/camera_info</cameraInfoTopicName>
           <depthImageTopicName>${ns}/depth/image_raw</depthImageTopicName>
           <depthImageCameraInfoTopicName>${ns}/depth/camera_info</depthImageCameraInfoTopicName>
@@ -136,6 +135,6 @@
         <wheelDiameter>0.215</wheelDiameter>
         <robotBaseFrame>${prefix}base_link</robotBaseFrame>
-        <torque>200</torque>
-        <MaxForce>5.0</MaxForce>
+        <torque>400</torque>
+        <MaxForce>10.0</MaxForce>
         <commandTopic>base/cmd_vel</commandTopic>
         <odometryTopic>odom</odometryTopic>
@@ -146,5 +145,5 @@
   </xacro:macro>
   <!-- Laser sensor plugin -->
-  <xacro:macro name="laser_sensor_sim" params="name frame ns">
+  <xacro:macro name="laser_sim_urg_04lx" params="name frame ns">
     <gazebo reference="${frame}">
       <sensor type="ray" name="${name}">
@@ -155,13 +154,13 @@
           <scan>
             <horizontal>
-              <samples>720</samples>
+              <samples>445</samples>
               <resolution>1</resolution>
-              <min_angle>-1.570796</min_angle>
-              <max_angle>1.570796</max_angle>
+              <min_angle>-1.40</min_angle>
+              <max_angle>1.40</max_angle>
             </horizontal>
           </scan>
           <range>
-            <min>0.10</min>
-            <max>6.0</max>
+            <min>0.1</min>
+            <max>4.0</max>
             <resolution>0.01</resolution>
           </range>
@@ -179,3 +178,37 @@
     </gazebo>
   </xacro:macro>
+  <!-- Laser sensor plugin -->
+  <xacro:macro name="laser_sim_utm_30lx" params="name frame ns">
+    <gazebo reference="${frame}">
+      <sensor type="ray" name="${name}">
+        <pose>0 0 0 0 0 0</pose>
+        <visualize>false</visualize>
+        <update_rate>40</update_rate>
+        <ray>
+          <scan>
+            <horizontal>
+              <samples>1080</samples>
+              <resolution>1</resolution>
+              <min_angle>-2.01</min_angle>
+              <max_angle>2.01</max_angle>
+            </horizontal>
+          </scan>
+          <range>
+            <min>0.1</min>
+            <max>30.0</max>
+            <resolution>0.01</resolution>
+          </range>
+          <noise>
+            <type>gaussian</type>
+            <mean>0.0</mean>
+            <stddev>0.01</stddev>
+          </noise>
+        </ray>
+        <plugin name="gazebo_ros_${name}_hokuyo_controller" filename="libgazebo_ros_laser.so">
+          <topicName>${ns}/scan</topicName>
+          <frameName>${frame}</frameName>
+        </plugin>
+      </sensor>
+    </gazebo>
+  </xacro:macro>
 </robot>
