Commit message: Link mass and damping

File: bender_common/bender_description/robots/bender_asus.urdf.xacro (robot description, xacro)
@@ -13,4 +13,6 @@
   <!-- Calibration parameters, used for arms in body.urdf.xacro -->
   <xacro:include filename="$(find bender_description)/urdf/calibration.xacro" />
+  <!-- Dynamixel parameters -->
+  <xacro:include filename="$(find bender_description)/urdf/dynamixel.xacro" />
   <!-- ******** Bender Parts ******** -->
   <!-- Bender Body -->

File: bender_common/bender_description/urdf/arm.urdf.xacro (robot description, xacro)
@@ -20,15 +20,17 @@
   <xacro:property name="shoulder_roll_joint_lower" value="-0.23776" />
   <!-- Links mass -->
-  <xacro:property name="link_mass" value="1.0" />
-  <xacro:property name="elbow_yaw_mass" value="${link_mass}" />
-  <xacro:property name="elbow_pitch_mass" value="${link_mass}" />
-  <xacro:property name="shoulder_yaw_mass" value="${link_mass}" />
-  <xacro:property name="shoulder_pitch_mass" value="${link_mass}" />
-  <xacro:property name="wrist_pitch_mass" value="${link_mass}" />
-  <xacro:property name="shoulder_roll_mass" value="${link_mass}" />
-  <!-- Effort -->
-  <xacro:property name="effort_shoulder" value="80" />
-  <xacro:property name="effort_elbow" value="30" />
-  <xacro:property name="effort_wrisp" value="15" />
+  <xacro:property name="shoulder_pitch_mass" value="${0.216}" />
+  <xacro:property name="shoulder_roll_mass"  value="${0.282}" />
+  <xacro:property name="shoulder_yaw_mass"   value="${0.256}" />
+  <xacro:property name="elbow_pitch_mass"    value="${0.243}" />
+  <xacro:property name="elbow_yaw_mass"      value="${0.222}" />
+  <xacro:property name="wrist_pitch_mass"    value="${0.430}" />
+  <!-- Torque -->
+  <xacro:property name="shoulder_pitch_torque" value="${mx106_torque}" />
+  <xacro:property name="shoulder_roll_torque"  value="${mx106_torque}" />
+  <xacro:property name="shoulder_yaw_torque"   value="${rx64_torque}" />
+  <xacro:property name="elbow_pitch_torque"    value="${mx106_torque}" />
+  <xacro:property name="elbow_yaw_torque"      value="${rx64_torque}" />
+  <xacro:property name="wrist_pitch_torque"    value="${rx28_torque}" />
   <xacro:macro name="bender_arm" params="side parent reflect prefix">
     <!-- Gazebo elements -->
@@ -88,9 +90,9 @@
         xyz="0 -1 0" />
       <limit
-        effort="${effort_shoulder}"
+        effort="${shoulder_pitch_torque}"
         lower="${shoulder_pitch_joint_lower}"
         upper="${shoulder_pitch_joint_upper}"
         velocity="${vel_arm * M_PI / 180}"/>
-      <dynamics damping="${damping}" friction="${friccion}" />
+      <dynamics damping="${dxl_damping}" friction="${dxl_friction}" />
       <safety_controller soft_lower_limit="${shoulder_pitch_joint_lower-soft_margin}" soft_upper_limit="${shoulder_pitch_joint_upper+soft_margin}" k_position="30" k_velocity="30"/>
     </joint>
@@ -138,7 +140,7 @@
         lower="${shoulder_roll_joint_lower}"
         upper="${shoulder_roll_joint_upper}"
-        effort="${effort_shoulder}"
-        velocity="${vel_arm * M_PI / 180}" />
-      <dynamics damping="${damping}" friction="${friccion}" />
+        effort="${shoulder_roll_torque}"
+        velocity="${vel_arm * M_PI / 180}" />
+      <dynamics damping="${dxl_damping}" friction="${dxl_friction}" />
       <safety_controller soft_lower_limit="${shoulder_roll_joint_lower-soft_margin}" soft_upper_limit="${shoulder_roll_joint_upper+soft_margin}" k_position="30" k_velocity="30"/>
     </joint>
@@ -186,7 +188,7 @@
         lower="${shoulder_yaw_joint_lower}"
         upper="${shoulder_yaw_joint_upper}"
-        effort="${effort_shoulder}"
-        velocity="${vel_arm * M_PI / 180}" />
-      <dynamics damping="${damping}" friction="${friccion}" />
+        effort="${shoulder_yaw_torque}"
+        velocity="${vel_arm * M_PI / 180}" />
+      <dynamics damping="${dxl_damping}" friction="${dxl_friction}" />
       <safety_controller soft_lower_limit="${shoulder_yaw_joint_lower-soft_margin}" soft_upper_limit="${shoulder_yaw_joint_upper+soft_margin}" k_position="30" k_velocity="30"/>
     </joint>
@@ -234,7 +236,7 @@
         lower="${elbow_pitch_joint_lower}"
         upper="${elbow_pitch_joint_upper}"
-        effort="${effort_elbow}"
-        velocity="${vel_arm * M_PI / 180}" />
-      <dynamics damping="${damping}" friction="${friccion}" />
+        effort="${elbow_pitch_torque}"
+        velocity="${vel_arm * M_PI / 180}" />
+      <dynamics damping="${dxl_damping}" friction="${dxl_friction}" />
       <safety_controller soft_lower_limit="${elbow_pitch_joint_lower-soft_margin}" soft_upper_limit="${elbow_pitch_joint_upper+soft_margin}" k_position="30" k_velocity="30"/>
     </joint>
@@ -282,7 +284,7 @@
         lower="${elbow_yaw_joint_lower}"
         upper="${elbow_yaw_joint_upper}"
-        effort="${effort_elbow}"
-        velocity="${vel_arm * M_PI / 180}" />
-      <dynamics damping="${damping}" friction="${friccion}" />
+        effort="${elbow_yaw_torque}"
+        velocity="${vel_arm * M_PI / 180}" />
+      <dynamics damping="${dxl_damping}" friction="${dxl_friction}" />
       <safety_controller soft_lower_limit="${elbow_yaw_joint_lower-soft_margin}" soft_upper_limit="${elbow_yaw_joint_upper+soft_margin}" k_position="30" k_velocity="30"/>
     </joint>
@@ -330,7 +332,7 @@
         lower="${wrist_pitch_joint_lower}"
         upper="${wrist_pitch_joint_upper}"
-        effort="${effort_wrisp}"
-        velocity="${vel_arm * M_PI / 180}" />
-      <dynamics damping="${damping}" friction="${friccion}" />
+        effort="${wrist_pitch_torque}"
+        velocity="${vel_arm * M_PI / 180}" />
+      <dynamics damping="${dxl_damping}" friction="${dxl_friction}" />
       <safety_controller soft_lower_limit="${wrist_pitch_joint_lower-soft_margin}" soft_upper_limit="${wrist_pitch_joint_upper+soft_margin}" k_position="30" k_velocity="30"/>
     </joint>

File: bender_common/bender_description/urdf/common.xacro (robot description, xacro)
@@ -6,5 +6,5 @@
   <xacro:property name="M_PI" value="3.1415926535897931" />
   <!-- Dynamics -->
-  <xacro:property name="damping" value="0.8" />
+  <xacro:property name="damping" value="0.2" />
   <!-- Friccion -->
   <xacro:property name="friccion" value="1.0" />
