Commit message: Update laser models

File: bender_common/bender_description/robots/bender_base.urdf.xacro (robot description, xacro)
@@ -21,6 +21,6 @@
   <!-- Hokuyo sensors -->
   <xacro:include filename="$(find bender_description)/urdf/laser_sensor.xacro" />
-  <xacro:laser_sensor parent="${prefix}base_link" name="laser_front" prefix="${prefix}sensors/" xyz="0.22 0.0 0.22"  rpy="0.0 0.0 0.0" ns="${prefix}sensors/laser_front"/>
-  <xacro:laser_sensor parent="${prefix}base_link" name="laser_rear"  prefix="${prefix}sensors/" xyz="-0.22 0.0 0.09" rpy="0.0 ${M_PI} 0.0" ns="${prefix}sensors/laser_rear" />
+  <xacro:laser_utm_30lx parent="${prefix}base_link" name="laser_front" prefix="${prefix}sensors/" xyz="0.22 0.0 0.22"  rpy="0.0 0.0 0.0" ns="${prefix}sensors/laser_front"/>
+  <xacro:laser_urg_04lx parent="${prefix}base_link" name="laser_rear"  prefix="${prefix}sensors/" xyz="-0.22 0.0 0.09" rpy="0.0 ${M_PI} 0.0" ns="${prefix}sensors/laser_rear" />
   <!-- ROS Controllers -->
   <xacro:ros_control prefix="${prefix}" />

File: bender_common/bender_description/robots/bender_calibration.urdf.xacro (robot description, xacro)
@@ -43,6 +43,6 @@
   <!-- Hokuyo sensors -->
   <xacro:include filename="$(find bender_description)/urdf/laser_sensor.xacro" />
-  <xacro:laser_sensor parent="${prefix}base_link" name="laser_front" prefix="${prefix}sensors/" xyz="0.22 0.0 0.22"  rpy="0.0 0.0 0.0" ns="${prefix}sensors/laser_front"/>
-  <xacro:laser_sensor parent="${prefix}base_link" name="laser_rear"  prefix="${prefix}sensors/" xyz="-0.22 0.0 0.09" rpy="0.0 ${M_PI} 0.0" ns="${prefix}sensors/laser_rear" />
+  <xacro:laser_utm_30lx parent="${prefix}base_link" name="laser_front" prefix="${prefix}sensors/" xyz="0.22 0.0 0.22"  rpy="0.0 0.0 0.0" ns="${prefix}sensors/laser_front"/>
+  <xacro:laser_urg_04lx parent="${prefix}base_link" name="laser_rear"  prefix="${prefix}sensors/" xyz="-0.22 0.0 0.09" rpy="0.0 ${M_PI} 0.0" ns="${prefix}sensors/laser_rear" />
   <!-- ROS Controllers -->
   <xacro:ros_control prefix="${prefix}" />

File: bender_common/bender_description/robots/bender_standard.urdf.xacro (robot description, xacro)
@@ -43,6 +43,6 @@
   <!-- Hokuyo sensors -->
   <xacro:include filename="$(find bender_description)/urdf/laser_sensor.xacro" />
-  <xacro:laser_sensor parent="${prefix}base_link" name="laser_front" prefix="${prefix}sensors/" xyz="0.22 0.0 0.22"  rpy="0.0 0.0 0.0" ns="${prefix}sensors/laser_front"/>
-  <xacro:laser_sensor parent="${prefix}base_link" name="laser_rear"  prefix="${prefix}sensors/" xyz="-0.22 0.0 0.09" rpy="0.0 ${M_PI} 0.0" ns="${prefix}sensors/laser_rear" />
+  <xacro:laser_utm_30lx parent="${prefix}base_link" name="laser_front" prefix="${prefix}sensors/" xyz="0.22 0.0 0.22"  rpy="0.0 0.0 0.0" ns="${prefix}sensors/laser_front"/>
+  <xacro:laser_urg_04lx parent="${prefix}base_link" name="laser_rear"  prefix="${prefix}sensors/" xyz="-0.22 0.0 0.09" rpy="0.0 ${M_PI} 0.0" ns="${prefix}sensors/laser_rear" />
   <!-- ROS Controllers -->
   <xacro:ros_control prefix="${prefix}" />

File: bender_common/bender_description/urdf/base.urdf.xacro (robot description, xacro)
@@ -109,8 +109,16 @@
       <collision>
         <origin
-          xyz="0 0 0.1"
+          xyz="0 0 0.075"
           rpy="0 0 0" />
         <geometry>
-          <box size="0.54 0.38 0.2"/>
+          <box size="0.4 0.3 0.15"/>
+        </geometry>
+      </collision>
+      <collision>
+        <origin
+          xyz="0 0 0.17"
+          rpy="0 0 0" />
+        <geometry>
+          <box size="0.54 0.38 0.05"/>
         </geometry>
       </collision>

File: bender_common/bender_description/urdf/gazebo.urdf.xacro (robot description, xacro)
@@ -145,5 +145,5 @@
   </xacro:macro>
   <!-- Laser sensor plugin -->
-  <xacro:macro name="laser_sensor_sim" params="name frame ns">
+  <xacro:macro name="laser_sim_urg_04lx" params="name frame ns">
     <gazebo reference="${frame}">
       <sensor type="ray" name="${name}">
@@ -154,13 +154,13 @@
           <scan>
             <horizontal>
-              <samples>720</samples>
+              <samples>445</samples>
               <resolution>1</resolution>
-              <min_angle>-1.570796</min_angle>
-              <max_angle>1.570796</max_angle>
+              <min_angle>-1.40</min_angle>
+              <max_angle>1.40</max_angle>
             </horizontal>
           </scan>
           <range>
-            <min>0.10</min>
-            <max>6.0</max>
+            <min>0.1</min>
+            <max>4.0</max>
             <resolution>0.01</resolution>
           </range>
@@ -178,3 +178,37 @@
     </gazebo>
   </xacro:macro>
+  <!-- Laser sensor plugin -->
+  <xacro:macro name="laser_sim_utm_30lx" params="name frame ns">
+    <gazebo reference="${frame}">
+      <sensor type="ray" name="${name}">
+        <pose>0 0 0 0 0 0</pose>
+        <visualize>false</visualize>
+        <update_rate>40</update_rate>
+        <ray>
+          <scan>
+            <horizontal>
+              <samples>1080</samples>
+              <resolution>1</resolution>
+              <min_angle>-2.01</min_angle>
+              <max_angle>2.01</max_angle>
+            </horizontal>
+          </scan>
+          <range>
+            <min>0.1</min>
+            <max>30.0</max>
+            <resolution>0.01</resolution>
+          </range>
+          <noise>
+            <type>gaussian</type>
+            <mean>0.0</mean>
+            <stddev>0.01</stddev>
+          </noise>
+        </ray>
+        <plugin name="gazebo_ros_${name}_hokuyo_controller" filename="libgazebo_ros_laser.so">
+          <topicName>${ns}/scan</topicName>
+          <frameName>${frame}</frameName>
+        </plugin>
+      </sensor>
+    </gazebo>
+  </xacro:macro>
 </robot>

File: bender_common/bender_description/urdf/laser_sensor.xacro (robot description, xacro)
@@ -1,5 +1,5 @@
 <?xml version="1.0"?>
 <robot name="laser_sensor" xmlns:xacro="http://ros.org/wiki/xacro">
-  <xacro:macro name="laser_sensor" params="parent name xyz rpy ns prefix">
+  <xacro:macro name="laser_urg_04lx" params="parent name xyz rpy ns prefix">
     <joint name="${name}_joint" type="fixed">
       <axis xyz="0 1 0" />
@@ -13,5 +13,5 @@
         <origin xyz="0 0 0" rpy="0 0 0"/>
         <geometry>
-          <box size="0.1 0.1 0.1"/>
+          <box size="0.05 0.05 0.08"/>
         </geometry>
       </collision>
@@ -30,5 +30,36 @@
     </link>
     <!-- Gazebo Sim -->
-    <xacro:laser_sensor_sim frame="${prefix}${name}_link" name="${name}" ns="${ns}" />
+    <xacro:laser_sim_urg_04lx frame="${prefix}${name}_link" name="${name}" ns="${ns}" />
+  </xacro:macro>
+  <xacro:macro name="laser_utm_30lx" params="parent name xyz rpy ns prefix">
+    <joint name="${name}_joint" type="fixed">
+      <axis xyz="0 1 0" />
+      <origin xyz="${xyz}" rpy="${rpy}"/>
+      <parent link="${parent}"/>
+      <child link="${prefix}${name}_link"/>
+    </joint>
+    <!-- Hokuyo Laser -->
+    <link name="${prefix}${name}_link">
+      <collision>
+        <origin xyz="0 0 0" rpy="0 0 0"/>
+        <geometry>
+          <box size="0.05 0.05 0.08"/>
+        </geometry>
+      </collision>
+      <visual>
+        <origin xyz="0 0 0" rpy="0 0 0"/>
+        <geometry>
+          <mesh filename="package://bender_description/meshes/sensors/hokuyo.dae"/>
+        </geometry>
+        <material
+          name="">
+          <color
+            rgba="0.1 0.1 0.1 1" />
+        </material>
+      </visual>
+      <xacro:cuboid_inertia_def x="0.05" y="0.05" z="0.05" mass="0.3"/>
+    </link>
+    <!-- Gazebo Sim -->
+    <xacro:laser_sim_utm_30lx frame="${prefix}${name}_link" name="${name}" ns="${ns}" />
   </xacro:macro>
 </robot>
