Commit message: Change grippers and put elbow motor to max angle

File: bender_description/robots/bender_calibration.urdf.xacro (robot description, xacro)
@@ -34,8 +34,8 @@
   <xacro:gripper side="l" reflect="-1" prefix="${prefix}" />
   <!-- Grippers Links -->
-  <xacro:gripper_int side="r" reflect="1" type="0" prefix="${prefix}"/>
-  <xacro:gripper_ext side="r" reflect="1" type="0" prefix="${prefix}"/>
-  <xacro:gripper_int side="l" reflect="-1" type="1" prefix="${prefix}"/>
-  <xacro:gripper_ext side="l" reflect="-1" type="1" prefix="${prefix}"/>
+  <xacro:gripper_int side="r" reflect="-1" type="1" prefix="${prefix}"/>
+  <xacro:gripper_ext side="r" reflect="-1" type="1" prefix="${prefix}"/>
+  <xacro:gripper_int side="l" reflect="1" type="0" prefix="${prefix}"/>
+  <xacro:gripper_ext side="l" reflect="1" type="0" prefix="${prefix}"/>
   <!-- Head with Asus depth camera -->
   <xacro:include filename="$(find bender_description)/urdf/head.urdf.xacro" />

File: bender_description/robots/bender_standard.urdf.xacro (robot description, xacro)
@@ -34,8 +34,8 @@
   <xacro:gripper side="l" reflect="-1" prefix="${prefix}" />
   <!-- Grippers Links -->
-  <xacro:gripper_int side="r" reflect="1" type="1" prefix="${prefix}"/>
-  <xacro:gripper_ext side="r" reflect="1" type="1" prefix="${prefix}"/>
-  <xacro:gripper_int side="l" reflect="-1" type="0" prefix="${prefix}"/>
-  <xacro:gripper_ext side="l" reflect="-1" type="0" prefix="${prefix}"/>
+  <xacro:gripper_int side="r" reflect="-1" type="0" prefix="${prefix}"/>
+  <xacro:gripper_ext side="r" reflect="-1" type="0" prefix="${prefix}"/>
+  <xacro:gripper_int side="l" reflect="1" type="1" prefix="${prefix}"/>
+  <xacro:gripper_ext side="l" reflect="1" type="1" prefix="${prefix}"/>
   <!-- Head with Asus depth camera -->
   <xacro:include filename="$(find bender_description)/urdf/head.urdf.xacro" />

File: bender_description/urdf/arm.urdf.xacro (robot description, xacro)
@@ -14,6 +14,6 @@
   <xacro:property name="wrist_pitch_joint_upper" value="1.22717" />
   <xacro:property name="wrist_pitch_joint_lower" value="-1.07378" />
-  <xacro:property name="elbow_pitch_joint_upper" value="1.86378" />
-  <xacro:property name="elbow_pitch_joint_lower" value="-1.03543" />
+  <xacro:property name="elbow_pitch_joint_upper" value="1.90213" />
+  <xacro:property name="elbow_pitch_joint_lower" value="-1.04310" />
   <xacro:property name="shoulder_roll_joint_upper" value="1.51096" />
   <xacro:property name="shoulder_roll_joint_lower" value="-0.23776" />

Commit message: Add power supply box on URDF

File: bender_description/robots/bender_calibration.urdf.xacro (robot description, xacro)
@@ -21,5 +21,5 @@
   <!-- Torso -->
   <xacro:include filename="$(find bender_description)/urdf/torso.urdf.xacro" />
-  <xacro:torso prefix="${prefix}" parent="${prefix}torso_base_link"/>
+  <xacro:torso prefix="${prefix}" parent="${prefix}torso_base_link" psu="0"/>
   <!-- Arm -->
   <xacro:include filename="$(find bender_description)/urdf/arm.urdf.xacro" />

File: bender_description/robots/bender_standard.urdf.xacro (robot description, xacro)
@@ -21,5 +21,5 @@
   <!-- Torso -->
   <xacro:include filename="$(find bender_description)/urdf/torso.urdf.xacro" />
-  <xacro:torso prefix="${prefix}" parent="${prefix}torso_base_link"/>
+  <xacro:torso prefix="${prefix}" parent="${prefix}torso_base_link" psu="1"/>
   <!-- Arm -->
   <xacro:include filename="$(find bender_description)/urdf/arm.urdf.xacro" />

File: bender_description/urdf/gazebo.urdf.xacro (robot description, xacro)
@@ -47,4 +47,5 @@
   <xacro:macro name="gazebo_link" params="link color">
     <gazebo reference="${link}">
+      <material>Gazebo/${color}</material>
       <mu1>0.2</mu1>
       <mu2>0.2</mu2>

File: bender_description/urdf/torso.urdf.xacro (robot description, xacro)
@@ -3,5 +3,5 @@
   xmlns:xacro="http://www.ros.org/wiki/xacro"
   name="torso">
-  <xacro:macro name="torso" params="prefix parent">
+  <xacro:macro name="torso" params="prefix parent psu">
     <!-- Lower torso  -->
     <link
@@ -76,4 +76,47 @@
         xyz="0 0 0" />
     </joint>
+    <!-- Power supply unit -->
+    <xacro:if value="${psu}">
+    <joint
+      name="psu_mount_fixed_joint"
+      type="fixed">
+      <origin
+        xyz="0 0 0"
+        rpy="0 0 0" />
+      <parent
+        link="${prefix}lower_torso_base" />
+      <child
+        link="${prefix}psu_base" />
+    </joint>
+    <link
+      name="${prefix}psu_base">
+      <inertial>
+        <origin
+          xyz="0.175 0 0.33"
+          rpy="0 0 0" />
+        <mass
+          value="1.5" />
+        <cuboid_inertia_def x="0.12" y="0.20" z="0.27" mass="1.5"/>
+      </inertial>
+      <visual>
+        <origin
+          xyz="0.175 0 0.33"
+          rpy="0 0 0" />
+        <geometry>
+          <box size="0.12 0.20 0.27"/>
+        </geometry>
+        <material name="Grey3" />
+      </visual>
+      <collision>
+        <origin
+          xyz="0.175 0 0.33"
+          rpy="0 0 0" />
+        <geometry>
+          <box size="0.12 0.20 0.27"/>
+        </geometry>
+      </collision>
+    </link>
+    <xacro:gazebo_link link="${prefix}psu_base" color="Grey" />
+    </xacro:if>
     <!-- Upper torso -->
     <link
