Commit message: working on pick and place

File: bender_description/robots/bender.urdf.xacro (robot description, xacro)
@@ -18,32 +18,32 @@
   <!-- Base -->
   <xacro:include filename="$(find bender_description)/urdf/base.urdf.xacro" />
-  <xacro:base prefix="${prefix}" />
+  <xacro:base prefix="bender/" />
   <!-- Torso -->
   <xacro:include filename="$(find bender_description)/urdf/bender_torso.xacro" />
-  <xacro:Torso prefix="${prefix}" parent="${prefix}mobile_base_link"/>
+  <xacro:Torso prefix="bender/" parent="bender/mobile_base_link"/>
   <!-- Arm -->
   <xacro:include filename="$(find bender_description)/urdf/right_arm.urdf.xacro" />
   <xacro:include filename="$(find bender_description)/urdf/left_arm.urdf.xacro" />
   <!-- Left Arm -->
-  <xacro:left_arm side="r" parent="${prefix}left_shoulder" reflect="-1" prefix="${prefix}"/>
+  <xacro:left_arm side="r" parent="bender/left_shoulder" reflect="-1" prefix="bender/"/>
   <!-- Right Arm -->
-  <xacro:right_arm side="l" parent="${prefix}right_shoulder" reflect="1" prefix="${prefix}"/>
+  <xacro:right_arm side="l" parent="bender/right_shoulder" reflect="1" prefix="bender/"/>
   <!-- Gripper -->
   <xacro:include filename="$(find bender_description)/urdf/gripper.urdf.xacro" />
   <!-- Gripper Joints -->
-  <xacro:gripper side="l" reflect="-1" prefix="${prefix}" />
-  <xacro:gripper side="r" reflect="1" prefix="${prefix}" />
+  <xacro:gripper side="l" reflect="-1" prefix="bender/" />
+  <xacro:gripper side="r" reflect="1" prefix="bender/" />
   <!-- Grippers Links -->
-  <xacro:gripper_int side="l" reflect="-1" type="1" prefix="${prefix}"/>
-  <xacro:gripper_ext side="l" reflect="-1" type="1" prefix="${prefix}"/>
-  <xacro:gripper_int side="r" reflect="1" type="1" prefix="${prefix}"/>
-  <xacro:gripper_ext side="r" reflect="1" type="1" prefix="${prefix}"/>
+  <xacro:gripper_int side="l" reflect="-1" type="1" prefix="bender/"/>
+  <xacro:gripper_ext side="l" reflect="-1" type="1" prefix="bender/"/>
+  <xacro:gripper_int side="r" reflect="1" type="1" prefix="bender/"/>
+  <xacro:gripper_ext side="r" reflect="1" type="1" prefix="bender/"/>
   <!-- Head with Asus depth camera -->
   <xacro:include filename="$(find bender_description)/urdf/head.urdf.xacro" />
-  <xacro:head parent="${prefix}neck_base" prefix="${prefix}" ns="/${prefix}sensors/rgbd_head" />
+  <xacro:head parent="bender/neck_base" prefix="bender/" ns="/bender/sensors/rgbd_head" />
   <!-- Hokuyo sensors -->
   <xacro:include filename="$(find bender_description)/urdf/laser_sensor.xacro" />
-  <xacro:laser_utm_30lx parent="${prefix}base_link" name="laser_front" prefix="${prefix}sensors/" xyz="0.22 0.0 0.22"  rpy="0.0 0.0 0.0" ns="${prefix}sensors/laser_front"/>
-  <xacro:laser_urg_04lx parent="${prefix}base_link" name="laser_rear"  prefix="${prefix}sensors/" xyz="-0.22 0.0 0.09" rpy="0.0 ${M_PI} 0.0" ns="${prefix}sensors/laser_rear" />
+  <xacro:laser_utm_30lx parent="bender/base_link" name="laser_front" prefix="bender/sensors/" xyz="0.22 0.0 0.22"  rpy="0.0 0.0 0.0" ns="bender/sensors/laser_front"/>
+  <xacro:laser_urg_04lx parent="bender/base_link" name="laser_rear"  prefix="bender/sensors/" xyz="-0.22 0.0 0.09" rpy="0.0 ${M_PI} 0.0" ns="bender/sensors/laser_rear" />
   <!-- ROS Controllers -->
   <xacro:ros_control prefix="/bender" />

File: bender_description/urdf/left_arm.urdf.xacro (robot description, xacro)
@@ -100,6 +100,6 @@
       xyz="-0.024808 0.99969 -4.5542E-05" />
     <limit
-      lower="-1.57"
-      upper="1.57"
+      lower="-3"
+      upper="3"
       effort="5"
       velocity="5" />
@@ -183,8 +183,8 @@
       <origin
         xyz="0 0 0"
-        rpy="0 0 0" />
-      <geometry>
-        <mesh
-          filename="package://bender_description/meshes/visual/l_shoulder_yaw_link.STL" />
+        rpy="0 0 ${-M_PI/2}" />
+      <geometry>
+        <mesh
+          filename="package://bender_description/meshes/visual/bicep_reoriented.stl" scale="0.001 0.001 0.001" />
       </geometry>
       <material
@@ -208,5 +208,5 @@
     <origin
       xyz="-0.030926 0.0014463 -0.061069"
-      rpy="0 0 0" />
+      rpy="0 0 ${M_PI/2}" />
     <parent
       link="${prefix}${side}_shoulder_roll_link" />
@@ -357,8 +357,8 @@
       <origin
         xyz="0 0 0"
-        rpy="0 0 0" />
-      <geometry>
-        <mesh
-          filename="package://bender_description/meshes/visual/l_wrist_pitch_link.STL" />
+        rpy="0 0 ${M_PI}" />
+      <geometry>
+        <mesh
+          filename="package://bender_description/meshes/visual/wrist_reoriented.stl" scale="0.001 0.001 0.001"/>
       </geometry>
       <material
@@ -412,11 +412,11 @@
       <xacro:if value="${(reflect+1)/2}">
         <origin
-          xyz="0.009625 0.03555 -0.0794"
-          rpy="0 0 0" />
+          xyz="${0.03555-0.017} 0.007 -0.0794"
+          rpy="0 0 ${-M_PI/2}" />
       </xacro:if >
       <xacro:unless value="${(reflect+1)/2}">
         <origin
-          xyz="0.009625 -0.00085 -0.0794"
-          rpy="0 0 0" />
+          xyz="${-0.00085-0.017} 0.007 -0.0794"
+          rpy="0 0 ${-M_PI/2}" />
       </xacro:unless >
       <parent
@@ -436,11 +436,11 @@
       <xacro:if value="${(reflect+1)/2}">
         <origin
-          xyz="0.009625 -0.00085 -0.0794"
-          rpy="0 0 0" />
+          xyz="${0.00085-0.017} 0.007 -0.0794"
+          rpy="0 0 ${-M_PI/2}" />
       </xacro:if >
       <xacro:unless value="${(reflect+1)/2}">
         <origin
-          xyz="0.009625 0.03555 -0.0794"
-          rpy="0 0 0" />
+          xyz="${0.03555-0.017} 0.007 -0.0794"
+          rpy="0 0 ${-M_PI/2}" />
       </xacro:unless >
       <parent
@@ -451,4 +451,27 @@
         xyz="0 0 0" />
     </joint>
+    <!-- Gripper Grasp -->
+    <link
+        name="${prefix}${side}_grasp_link">
+        <xacro:dummy_inertial/>
+      </link>
+    <joint
+        name="${side}_grasp_joint"
+        type="fixed">
+        <xacro:if value="${(reflect+1)/2}">
+          <origin
+            xyz="0.0 -0.02 -0.18"
+            rpy="0 ${M_PI/2} ${-M_PI/2}" />
+        </xacro:if>
+        <xacro:unless value="${(reflect+1)/2}">
+          <origin
+            xyz="0.0 0.02 -0.18"
+            rpy="0 ${M_PI/2} ${-M_PI/2}" />
+        </xacro:unless>
+        <parent
+          link="${prefix}${side}_wrist_pitch_link" />
+        <child
+          link="${prefix}${side}_grasp_link" />
+      </joint>
 	</xacro:macro>
 </robot>

File: bender_description/urdf/right_arm.urdf.xacro (robot description, xacro)
@@ -101,6 +101,6 @@
       xyz="-0.024808 0.99969 -4.5542E-05" />
     <limit
-      lower="-1.57"
-      upper="1.57"
+      lower="-3"
+      upper="3"
       effort="5"
       velocity="5" />
@@ -184,8 +184,8 @@
       <origin
         xyz="0 0 0"
-        rpy="0 0 0" />
-      <geometry>
-        <mesh
-          filename="package://bender_description/meshes/visual/l_shoulder_yaw_link.STL" />
+        rpy="0 0 ${M_PI/2}" />
+      <geometry>
+        <mesh
+          filename="package://bender_description/meshes/visual/bicep_reoriented.stl" scale="0.001 0.001 0.001" />
       </geometry>
       <material
@@ -209,5 +209,5 @@
     <origin
       xyz="-0.030926 -0.0014463 -0.061069"
-      rpy="0 0 0" />
+      rpy="0 0 ${-M_PI/2}" />
     <parent
       link="${prefix}${side}_shoulder_roll_link" />
@@ -361,5 +361,5 @@
       <geometry>
         <mesh
-          filename="package://bender_description/meshes/visual/l_wrist_pitch_link.STL" />
+          filename="package://bender_description/meshes/visual/wrist_reoriented.stl" scale="0.001 0.001 0.001"/>
       </geometry>
       <material
@@ -383,5 +383,5 @@
     <origin
       xyz="0.00020829 -0.019843 -0.29049"
-      rpy="0 0 0" />
+      rpy="0 0 ${M_PI}" />
     <parent
       link="${prefix}${side}_elbow_yaw_link" />
@@ -413,6 +413,6 @@
       <xacro:if value="${(reflect+1)/2}">
         <origin
-          xyz="0.01925 0.04 -0.0794"
-          rpy="0 0 0" />
+          xyz="${0.03555-0.017} -0.0365 -0.0794"
+          rpy="0 0 ${-M_PI/2}" />
       </xacro:if >
       <xacro:unless value="${(reflect+1)/2}">
@@ -437,6 +437,6 @@
       <xacro:if value="${(reflect+1)/2}">
         <origin
-          xyz="0.01925 -0.0008 -0.0794"
-          rpy="0 0 0" />
+          xyz="${-0.00085-0.017} -0.0365 -0.0794"
+          rpy="0 0 ${-M_PI/2}" />
       </xacro:if >
       <xacro:unless value="${(reflect+1)/2}">
@@ -452,4 +452,27 @@
         xyz="0 0 0" />
     </joint>
+    <!-- Gripper Grasp -->
+    <link
+        name="${prefix}${side}_grasp_link">
+        <xacro:dummy_inertial/>
+      </link>
+    <joint
+        name="${side}_grasp_joint"
+        type="fixed">
+        <xacro:if value="${(reflect+1)/2}">
+          <origin
+            xyz="0.0 -0.02 -0.18"
+            rpy="0 ${M_PI/2} ${-M_PI/2}" />
+        </xacro:if>
+        <xacro:unless value="${(reflect+1)/2}">
+          <origin
+            xyz="0.0 0.02 -0.18"
+            rpy="0 ${M_PI/2} ${-M_PI/2}" />
+        </xacro:unless>
+        <parent
+          link="${prefix}${side}_wrist_pitch_link" />
+        <child
+          link="${prefix}${side}_grasp_link" />
+      </joint>
 	</xacro:macro>
 </robot>

File: bender_description/urdf/torso.urdf.xacro (robot description, xacro)
@@ -218,5 +218,5 @@
       <!-- CALIBRATION Z 0.619 => 0.610 -->
       <origin
-        xyz="-0.005 0.23 0.610"
+        xyz="0 0 0"
         rpy="0 0 0" />
       <parent
