Commit message: new updates (to lazy too list them all)

File: bender_description/robots/bender_standard.urdf.xacro (robot description, xacro)
@@ -26,17 +26,17 @@
   <xacro:include filename="$(find bender_description)/urdf/left_arm.urdf.xacro" />
   <!-- Left Arm -->
-  <xacro:left_arm side="l" parent="${prefix}left_shoulder" reflect="-1" prefix="${prefix}"/>
+  <xacro:left_arm side="r" parent="${prefix}left_shoulder" reflect="-1" prefix="${prefix}"/>
   <!-- Right Arm -->
-  <xacro:right_arm side="r" parent="${prefix}right_shoulder" reflect="1" prefix="${prefix}"/>
+  <xacro:right_arm side="l" parent="${prefix}right_shoulder" reflect="1" prefix="${prefix}"/>
   <!-- Gripper -->
   <xacro:include filename="$(find bender_description)/urdf/gripper.urdf.xacro" />
   <!-- Gripper Joints -->
-  <xacro:gripper side="r" reflect="-1" prefix="${prefix}" />
-  <xacro:gripper side="l" reflect="1" prefix="${prefix}" />
+  <xacro:gripper side="l" reflect="-1" prefix="${prefix}" />
+  <xacro:gripper side="r" reflect="1" prefix="${prefix}" />
   <!-- Grippers Links -->
-  <xacro:gripper_int side="r" reflect="-1" type="1" prefix="${prefix}"/>
-  <xacro:gripper_ext side="r" reflect="-1" type="1" prefix="${prefix}"/>
-  <xacro:gripper_int side="l" reflect="1" type="1" prefix="${prefix}"/>
-  <xacro:gripper_ext side="l" reflect="1" type="1" prefix="${prefix}"/>
+  <xacro:gripper_int side="l" reflect="-1" type="1" prefix="${prefix}"/>
+  <xacro:gripper_ext side="l" reflect="-1" type="1" prefix="${prefix}"/>
+  <xacro:gripper_int side="r" reflect="1" type="1" prefix="${prefix}"/>
+  <xacro:gripper_ext side="r" reflect="1" type="1" prefix="${prefix}"/>
   <!-- Head with Asus depth camera -->
   <xacro:include filename="$(find bender_description)/urdf/head.urdf.xacro" />

File: bender_description/urdf/bender_torso.xacro (robot description, xacro)
@@ -2,5 +2,5 @@
 <robot xmlns:xacro="http://www.ros.org/wiki/xacro" name="Torso">
 	<xacro:property name="prefix" value="$(arg prefix)" />
-	<xacro:property name="altura" value="0.2" />
+	<xacro:property name="altura" value="0.19" />
 	<xacro:macro name="Torso" params="prefix parent">
 		<!-- Body Base link (Parent of all future links)-->
@@ -69,14 +69,13 @@
 		        name="">
 		        <color
-		          rgba="0.79216 0.81961 0.93333 1" />
-		      </material>
-		    </visual>
-		    <collision>
-		      <origin
-        		xyz="0 0 0"
-        		rpy="0 0 1.57" />
-		      <geometry>
-		        <mesh
-		          filename="package://bender_description/meshes/visual/PC_Base.STL" />
+		          rgba="0.650980392156863 0.619607843137255 0.588235294117647 1" />
+		      </material>
+		    </visual>
+		    <collision>
+		      <origin
+        		xyz="-0.08 0 0.25"
+        		rpy="0 0.15 0" />
+		      <geometry>
+		        <box size="0.09 0.4 0.28" />
 		      </geometry>
 		    </collision>
@@ -121,14 +120,13 @@
 		        name="">
 		        <color
-		          rgba="0.75294 0.75294 0.75294 1" />
-		      </material>
-		    </visual>
-		    <collision>
-		      <origin
-        		xyz="0 -0.1305 0"
-        		rpy="3.14 0 1.57" />
-		      <geometry>
-		        <mesh
-		          filename="package://bender_description/meshes/visual/router.STL" />
+		          rgba="0.650980392156863 0.619607843137255 0.588235294117647 1" />
+		      </material>
+		    </visual>
+		    <collision>
+		      <origin
+        		xyz="0.02 0 0.12"
+        		rpy="0 0 0" />
+		      <geometry>
+		        <box size="0.05 0.27 0.22" />
 		      </geometry>
 		    </collision>
@@ -147,5 +145,5 @@
 		  </joint>
 		  <!--Bender Left shoulder, here we will later fixe the left arm-->
-		  <link name="${prefix}left_shoulder">
+		  <link name="${prefix}right_shoulder">
 		    <inertial>
 		      <origin
@@ -164,9 +162,9 @@
 		    <visual>
 		     <origin
-        		xyz="0 0 0"
+        		xyz="0 0 -0.12"
         		rpy="1.57 1.57 0" />
 		      <geometry>
 		        <mesh
-		          filename="package://bender_description/meshes/visual/left_shoulder.STL" />
+		          filename="package://bender_description/meshes/visual/right_shoulder.STL" />
 		      </geometry>
 		      <material
@@ -187,5 +185,5 @@
 		 <!-- Here we join the left shoulder with the Body with the-->
 		  <joint
-		    name="left_shoulder_to_torso_joint"
+		    name="right_shoulder_to_torso_joint"
 		    type="fixed">
 		    <origin
@@ -195,9 +193,9 @@
 		      link="${prefix}torso" />
 		    <child
-		      link="${prefix}left_shoulder" />
+		      link="${prefix}right_shoulder" />
 		  </joint>
 		  <!--Bender right shoulder, here we will later fixe the right arm-->
 		  <link
-		    name="${prefix}right_shoulder">
+		    name="${prefix}left_shoulder">
 		    <inertial>
 		      <origin
@@ -216,9 +214,9 @@
 		    <visual>
 		       <origin
-        			xyz="0 0 0"
+        			xyz="0 0 -0.12"
         			rpy="-1.57 -1.57 0" />
 		      <geometry>
 		        <mesh
-		          filename="package://bender_description/meshes/visual/right_shoulder.STL" />
+		          filename="package://bender_description/meshes/visual/left_shoulder.STL" />
 		      </geometry>
 		      <material
@@ -239,5 +237,5 @@
 		  <!-- Here we join the left shoulder with the Body with the-->
 		  <joint
-		    name="right_shoulder_to_torso_joint"
+		    name="left_shoulder_to_torso_joint"
 		    type="fixed">
 		    <origin
@@ -247,5 +245,5 @@
 		      link="${prefix}torso" />
 		    <child
-		      link="${prefix}right_shoulder" />
+		      link="${prefix}left_shoulder" />
 		  </joint>
 		  <!-- here we have already created the Torso of Bender, so now we will create the joint with the other bender base-->
@@ -263,5 +261,5 @@
 		 <link name="${prefix}neck_base"/>
 		 <joint name="neck_base_to_body" type="fixed">
-		 	<origin xyz="0.03 0 1.1" rpy="0 0 0"/>
+		 	<origin xyz="0.03 0 1.085" rpy="0 0 0"/>
 		 	<parent link="${prefix}torso" />
 		 	<child link="${prefix}neck_base" />

File: bender_description/urdf/left_arm.urdf.xacro (robot description, xacro)
@@ -37,5 +37,5 @@
         name="">
         <color
-          rgba="0.792156862745098 0.819607843137255 0.933333333333333 1" />
+          rgba="0.05 0.05 0.05 1" />
       </material>
     </visual>
@@ -76,5 +76,5 @@
         name="">
         <color
-          rgba="0.792156862745098 0.819607843137255 0.933333333333333 1" />
+          rgba="0.05 0.05 0.05 1" />
       </material>
     </visual>
@@ -133,5 +133,5 @@
         name="">
         <color
-          rgba="0.792156862745098 0.819607843137255 0.933333333333333 1" />
+          rgba="0.05 0.05 0.05 1" />
       </material>
     </visual>
@@ -191,5 +191,5 @@
         name="">
         <color
-          rgba="0.792156862745098 0.819607843137255 0.933333333333333 1" />
+          rgba="0.05 0.05 0.05 1" />
       </material>
     </visual>
@@ -249,5 +249,5 @@
         name="">
         <color
-          rgba="0.792156862745098 0.819607843137255 0.933333333333333 1" />
+          rgba="0.05 0.05 0.05 1" />
       </material>
     </visual>
@@ -307,5 +307,5 @@
         name="">
         <color
-          rgba="0.792156862745098 0.819607843137255 0.933333333333333 1" />
+          rgba="0.05 0.05 0.05 1" />
       </material>
     </visual>
@@ -365,5 +365,5 @@
         name="">
         <color
-          rgba="0.792156862745098 0.819607843137255 0.933333333333333 1" />
+          rgba="0.05 0.05 0.05 1" />
       </material>
     </visual>

File: bender_description/urdf/right_arm.urdf.xacro (robot description, xacro)
@@ -37,5 +37,5 @@
         name="">
         <color
-          rgba="0.792156862745098 0.819607843137255 0.933333333333333 1" />
+          rgba="0.05 0.05 0.05 1" />
       </material>
     </visual>
@@ -76,5 +76,5 @@
         name="">
         <color
-          rgba="0.792156862745098 0.819607843137255 0.933333333333333 1" />
+          rgba="0.05 0.05 0.05 1" />
       </material>
     </visual>
@@ -134,5 +134,5 @@
         name="">
         <color
-          rgba="0.792156862745098 0.819607843137255 0.933333333333333 1" />
+          rgba="0.05 0.05 0.05 1" />
       </material>
     </visual>
@@ -192,5 +192,5 @@
         name="">
         <color
-          rgba="0.792156862745098 0.819607843137255 0.933333333333333 1" />
+          rgba="0.05 0.05 0.05 1" />
       </material>
     </visual>
@@ -250,5 +250,5 @@
         name="">
         <color
-          rgba="0.792156862745098 0.819607843137255 0.933333333333333 1" />
+          rgba="0.05 0.05 0.05 1" />
       </material>
     </visual>
@@ -308,5 +308,5 @@
         name="">
         <color
-          rgba="0.792156862745098 0.819607843137255 0.933333333333333 1" />
+          rgba="0.05 0.05 0.05 1" />
       </material>
     </visual>
@@ -366,5 +366,5 @@
         name="">
         <color
-          rgba="0.792156862745098 0.819607843137255 0.933333333333333 1" />
+          rgba="0.05 0.05 0.05 1" />
       </material>
     </visual>

Commit message: add realsense d435 camera urdf and gazebo functionality

File: bender_description/robots/bender_standard.urdf.xacro (robot description, xacro)
@@ -22,4 +22,9 @@
   <xacro:include filename="$(find bender_description)/urdf/bender_torso.xacro" />
   <xacro:Torso prefix="${prefix}" parent="${prefix}mobile_base_link"/>
+  <!-- Realsense D435 -->
+  <xacro:include filename="$(find bender_description)/urdf/d435.urdf.xacro" />
+  <xacro:realsense_d435 prefix="${prefix}" name="d435_camera" parent="bender/torso" ns="bender/d435_camera/" />
+  <!-- Realsense D435 Gazebo -->
+  <xacro:d435_sim_camera prefix="${prefix}" name="d435_camera" />
   <!-- Arm -->
   <xacro:include filename="$(find bender_description)/urdf/right_arm.urdf.xacro" />

File: bender_description/urdf/gazebo.urdf.xacro (robot description, xacro)
@@ -1,4 +1,5 @@
 <?xml version="1.0"?>
 <robot xmlns:xacro="http://www.ros.org/wiki/xacro">
+  <xacro:property name="deg_to_rad" value="0.01745329251994329577"/>
   <!-- ROS Control -->
   <xacro:macro name="ros_control" params="prefix">
@@ -121,4 +122,131 @@
         </plugin>
       </sensor>
+    </gazebo>
+  </xacro:macro>
+  <!-- Realsense D435 plugin -->
+  <xacro:macro name="d435_sim_camera" params="prefix name">
+    <gazebo reference="${name}_color_frame">
+      <sensor name="color" type="camera">
+        <pose frame="">0 0 0 0 0 0</pose>
+        <camera name="__default__">
+          <horizontal_fov>1.5009831567151233</horizontal_fov>
+          <image>
+            <width>640</width>
+            <height>480</height>
+            <format>RGB_INT8</format>
+          </image>
+          <clip>
+            <near>0.1</near>
+            <far>100</far>
+          </clip>
+          <noise>
+            <type>gaussian</type>
+            <mean>0.0</mean>
+            <stddev>0.007</stddev>
+          </noise>
+        </camera>
+        <always_on>1</always_on>
+        <update_rate>30</update_rate>
+        <visualize>1</visualize>
+      </sensor>
+    </gazebo>
+    <gazebo reference="${name}_left_ir_frame">
+      <sensor name="ired1" type="camera">
+        <pose frame="">0 0 0 0 0 0</pose>
+        <camera name="__default__">
+          <horizontal_fov>1.5009831567151233</horizontal_fov>
+          <image>
+            <width>640</width>
+            <height>480</height>
+            <format>L_INT8</format>
+          </image>
+          <clip>
+            <near>0.1</near>
+            <far>100</far>
+          </clip>
+          <noise>
+            <type>gaussian</type>
+            <mean>0.0</mean>
+            <stddev>0.007</stddev>
+          </noise>
+        </camera>
+        <always_on>1</always_on>
+        <update_rate>30</update_rate>
+        <visualize>0</visualize>
+      </sensor>
+    </gazebo>
+    <gazebo reference="${name}_right_ir_frame">
+      <sensor name="ired2" type="camera">
+        <pose frame="">0 0 0 0 0 0</pose>
+        <camera name="__default__">
+          <horizontal_fov>1.5009831567151233</horizontal_fov>
+          <image>
+            <width>640</width>
+            <height>480</height>
+            <format>L_INT8</format>
+          </image>
+          <clip>
+            <near>0.1</near>
+            <far>100</far>
+          </clip>
+          <noise>
+            <type>gaussian</type>
+            <mean>0.0</mean>
+            <stddev>0.007</stddev>
+          </noise>
+        </camera>
+        <always_on>1</always_on>
+        <update_rate>30</update_rate>
+        <visualize>0</visualize>
+      </sensor>
+    </gazebo>
+    <gazebo reference="${name}_depth_frame">
+      <sensor name="depth" type="depth">
+        <pose frame="">0 0 0 0 0 0</pose>
+        <camera name="__default__">
+          <horizontal_fov>1.5009831567151233</horizontal_fov>
+          <image>
+            <width>640</width>
+            <height>480</height>
+          </image>
+          <clip>
+            <near>0.1</near>
+            <far>100</far>
+          </clip>
+          <noise>
+            <type>gaussian</type>
+            <mean>0.0</mean>
+            <stddev>0.007</stddev>
+          </noise>
+        </camera>
+        <always_on>1</always_on>
+        <update_rate>30</update_rate>
+        <visualize>0</visualize>
+      </sensor>
+    </gazebo>
+    <gazebo>
+      <plugin name="${prefix}sensors/${name}" filename="librealsense_gazebo_plugin.so">
+        <depthUpdateRate>30</depthUpdateRate>
+        <colorUpdateRate>30</colorUpdateRate>
+        <infraredUpdateRate>30</infraredUpdateRate>
+        <depthTopicName>depth/image_raw</depthTopicName>
+        <depthCameraInfoTopicName>depth/camera_info</depthCameraInfoTopicName>
+        <colorTopicName>color/image_raw</colorTopicName>
+        <colorCameraInfoTopicName>color/camera_info</colorCameraInfoTopicName>
+        <infrared1TopicName>infrared/image_raw</infrared1TopicName>
+        <infrared1CameraInfoTopicName>infrared/camera_info</infrared1CameraInfoTopicName>
+        <infrared2TopicName>infrared2/image_raw</infrared2TopicName>
+        <infrared2CameraInfoTopicName>infrared2/camera_info</infrared2CameraInfoTopicName>
+        <colorOpticalframeName>camera_color_optical_frame</colorOpticalframeName>
+        <depthOpticalframeName>camera_depth_optical_frame</depthOpticalframeName>
+        <infrared1OpticalframeName>camera_left_ir_optical_frame</infrared1OpticalframeName>
+        <infrared2OpticalframeName>camera_right_ir_optical_frame</infrared2OpticalframeName>
+        <rangeMinDepth>0.1</rangeMinDepth>
+        <rangeMaxDepth>10</rangeMaxDepth>
+        <pointCloud>1</pointCloud>
+        <pointCloudTopicName>depth/color/points</pointCloudTopicName>
+        <pointCloudCutoff>0.15</pointCloudCutoff>
+        <pointCloudCutoffMax>10</pointCloudCutoffMax>
+      </plugin>
     </gazebo>
   </xacro:macro>

Commit message: gazebo.launch updated to noetic

File: bender_description/robots/bender_standard.urdf.xacro (robot description, xacro)
@@ -3,4 +3,6 @@
   xmlns:xacro="http://www.ros.org/wiki/xacro"
   name="bender">
+  <!-- Macros -->
+  <xacro:include filename="$(find bender_description)/urdf/inertia_macros.xacro" />
   <!-- Prefix for Bender links -->
   <xacro:property name="prefix" value="bender/" />
@@ -34,14 +36,14 @@
   <!-- Right Arm -->
   <xacro:right_arm side="l" parent="${prefix}right_shoulder" reflect="1" prefix="${prefix}"/>
-  <!-- Gripper -->
+  <!-- Gripper
   <xacro:include filename="$(find bender_description)/urdf/gripper.urdf.xacro" />
-  <!-- Gripper Joints -->
+  Gripper Joints
   <xacro:gripper side="l" reflect="-1" prefix="${prefix}" />
   <xacro:gripper side="r" reflect="1" prefix="${prefix}" />
-  <!-- Grippers Links -->
+  Grippers Links
   <xacro:gripper_int side="l" reflect="-1" type="1" prefix="${prefix}"/>
   <xacro:gripper_ext side="l" reflect="-1" type="1" prefix="${prefix}"/>
   <xacro:gripper_int side="r" reflect="1" type="1" prefix="${prefix}"/>
-  <xacro:gripper_ext side="r" reflect="1" type="1" prefix="${prefix}"/>
+  <xacro:gripper_ext side="r" reflect="1" type="1" prefix="${prefix}"/> -->
   <!-- Head with Asus depth camera -->
   <xacro:include filename="$(find bender_description)/urdf/head.urdf.xacro" />

File: bender_description/urdf/base.urdf.xacro (robot description, xacro)
@@ -32,5 +32,5 @@
           xyz="0 ${- reflect * 0.025} 0"
           rpy="${M_PI/2} 0 0" />
-        <cylinder_inertia_def length="0.05" radius="0.1" mass="50.0"/>
+        <xacro:cylinder_inertia_def length="0.05" radius="0.1" mass="50.0"/>
         <mass value="50.0" />
       </inertial>
@@ -91,5 +91,5 @@
           rpy="0 0 0" />
         <mass value="12.0" />
-        <cuboid_inertia_def x="0.54" y="0.38" z="0.2" mass="12.0"/>
+        <xacro:cuboid_inertia_def x="0.54" y="0.38" z="0.2" mass="12.0"/>
       </inertial>
       <visual>

File: bender_description/urdf/gripper.urdf.xacro (robot description, xacro)
@@ -73,5 +73,5 @@
           rpy="${-M_PI/6} 0 0" />
         <mass value="${gripper_mass}" />
-        <cuboid_inertia_def x="0.05" y="0.035" z="0.16" mass="${gripper_mass}"/>
+        <xacro:cuboid_inertia_def x="0.05" y="0.035" z="0.16" mass="${gripper_mass}"/>
       </inertial>
       <visual>
@@ -87,6 +87,6 @@
         </xacro:unless>
         <geometry>
-          <mesh
-            filename="package://bender_description/meshes/visual/one_finger.stl" />
+          <!-- <mesh
+            filename="package://bender_description/meshes/visual/one_finger.stl" /> -->
         </geometry>
         <material name="Grey1" />
@@ -104,6 +104,8 @@
         </xacro:unless>
         <geometry>
+        <!-- Ignorado
           <mesh
             filename="package://bender_description/meshes/collision/finger.stl" scale="0.35 1.0 1.0"/>
+        -->
         </geometry>
       </collision>
@@ -115,5 +117,5 @@
           rpy="${-M_PI/6} 0 0" />
         <mass value="${gripper_mass}" />
-        <cuboid_inertia_def x="0.05" y="0.035" z="0.16" mass="${gripper_mass}"/>
+        <xacro:cuboid_inertia_def x="0.05" y="0.035" z="0.16" mass="${gripper_mass}"/>
       </inertial>
       <visual>
@@ -129,6 +131,6 @@
         </xacro:unless>
         <geometry>
-          <mesh
-            filename="package://bender_description/meshes/visual/two_finger.stl" />
+          <!-- <mesh
+            filename="package://bender_description/meshes/visual/two_finger.stl" /> -->
         </geometry>
         <material name="Grey1" />
@@ -146,6 +148,6 @@
         </xacro:unless>
         <geometry>
-          <mesh
-            filename="package://bender_description/meshes/collision/finger.stl"/>
+          <!-- <mesh
+            filename="package://bender_description/meshes/collision/finger.stl"/> -->
         </geometry>
       </collision>
