Commit message: backup felipe

File: bender2_description/urdf/bender_standart.urdf.xacro (robot description, xacro)
@@ -32,5 +32,5 @@
   <xacro:head parent="${prefix}neck_base" prefix="${prefix}" ns="/${prefix}sensors/rgbd_head" />
 <gazebo>
-      <plugin filename="libgazebo_ros_control.so" name="ros_control">
+      <plugin filename="libgazebo_ros_control.so" name="gazebo_ros_control">
         <robotNamespace>${prefix}</robotNamespace>
       </plugin>

File: bender2_description/urdf/left_arm.urdf.xacro (robot description, xacro)
@@ -1,5 +1,5 @@
 <?xml version="1.0"?>
 <robot xmlns:xacro="http://www.ros.org/wiki/xacro" name="arm">
-  <xacro:property name="prefix" value="bender" />
+  <xacro:property name="prefix" value="bender/" />
 	<xacro:macro name="left_arm" params="side prefix parent reflect">
 		<link

File: bender2_description/urdf/right_arm.urdf.xacro (robot description, xacro)
@@ -1,5 +1,5 @@
 <?xml version="1.0"?>
 <robot xmlns:xacro="http://www.ros.org/wiki/xacro" name="arm">
-  <xacro:property name="prefix" value="bender" />
+  <xacro:property name="prefix" value="bender/" />
 	<xacro:macro name="right_arm" params=" side prefix parent reflect">
 		<link
