Commit message: 2022 manipulation

File: bender_description/urdf/right_arm.urdf.xacro (robot description, xacro)
@@ -371,8 +371,8 @@
     <collision>
       <origin
-        xyz="0 0.01525 -0.06"
-        rpy="0 0 0" />
-      <geometry>
-        <box size="0.04 0.08 0.0625" />
+        xyz="0 -0.01525 -0.06"
+        rpy="0 0 0" />
+      <geometry>
+        <box size="0.08 0.04 0.0625" />
       </geometry>
     </collision>
