Commit message: lenovo update push

File: bender_description/urdf/gripper.urdf.xacro (robot description, xacro)
@@ -7,4 +7,5 @@
   <xacro:property name="gripper_mass" value="0.160" />
   <xacro:property name="gripper_effort" value="${rx28_torque}" />
+  <!-- <xacro:property name="gripper_effort" value="${rx28_torque}" /> -->
   <xacro:macro name="gripper" params="side reflect prefix">
     <!-- Transmission -->

File: bender_description/urdf/left_arm.urdf.xacro (robot description, xacro)
@@ -102,5 +102,5 @@
       lower="-3"
       upper="3"
-      effort="5"
+      effort="40"
       velocity="5" />
       <dynamics damping="${dxl_damping}" friction="${dxl_friction}" />
@@ -160,5 +160,5 @@
       lower="-1.57"
       upper="0.1"
-      effort="5"
+      effort="40"
       velocity="5" />
       <dynamics damping="${dxl_damping}" friction="${dxl_friction}" />
@@ -218,5 +218,5 @@
       lower="-1.37"
       upper="1.37"
-      effort="5"
+      effort="40"
       velocity="5" />
       <dynamics damping="${dxl_damping}" friction="${dxl_friction}" />
@@ -276,5 +276,5 @@
       lower="-1.97"
       upper="0"
-      effort="5"
+      effort="40"
       velocity="5" />
       <dynamics damping="${dxl_damping}" friction="${dxl_friction}" />
@@ -334,5 +334,5 @@
       lower="-1.2"
       upper="1.2"
-      effort="5"
+      effort="40"
       velocity="5" />
         <dynamics damping="${dxl_damping}" friction="${dxl_friction}" />
@@ -392,5 +392,5 @@
       lower="-1.57"
       upper="1.57"
-      effort="5"
+      effort="40"
       velocity="5" />
       <dynamics damping="${dxl_damping}" friction="${dxl_friction}" />

File: bender_description/urdf/right_arm.urdf.xacro (robot description, xacro)
@@ -103,5 +103,5 @@
       lower="-3"
       upper="3"
-      effort="5"
+      effort="40"
       velocity="5" />
       <dynamics damping="${dxl_damping}" friction="${dxl_friction}" />
@@ -161,5 +161,5 @@
       lower="-0.1"
       upper="1.57"
-      effort="5"
+      effort="40"
       velocity="5" />
       <dynamics damping="${dxl_damping}" friction="${dxl_friction}" />
@@ -219,5 +219,5 @@
       lower="-1.37"
       upper="1.37"
-      effort="5"
+      effort="40"
       velocity="5" />
       <dynamics damping="${dxl_damping}" friction="${dxl_friction}" />
@@ -277,5 +277,5 @@
       lower="-1.97"
       upper="0"
-      effort="5"
+      effort="40"
       velocity="5" />
       <dynamics damping="${dxl_damping}" friction="${dxl_friction}" />
@@ -335,5 +335,5 @@
       lower="-1.2"
       upper="1.2"
-      effort="5"
+      effort="40"
       velocity="5" />
       <dynamics damping="${dxl_damping}" friction="${dxl_friction}" />
@@ -393,5 +393,5 @@
       lower="-1.57"
       upper="1.57"
-      effort="5"
+      effort="40"
       velocity="5" />
       <dynamics damping="${dxl_damping}" friction="${dxl_friction}" />
