Commit message: (FG): added laser filter

File: bender_description/urdf/bender.xacro (robot description, xacro)
@@ -722,5 +722,5 @@
 </joint>
 <joint name="laser_to_base_link" type="fixed">
-  <origin xyz="0.188322 -0.007366 0.25882" rpy="0 0 0"/>
+  <origin xyz="0.188322 -0.007366 0.25882" rpy="0 0 ${pi}"/>
   <parent link="base_link"/>
   <child link="laser"/>

Commit message: (FG): updating changes (and adding filter node)

File: bender_description/urdf/bender.xacro (robot description, xacro)
@@ -722,5 +722,5 @@
 </joint>
 <joint name="laser_to_base_link" type="fixed">
-  <origin xyz="0.188322 -0.007366 0.25882" rpy="0 0 ${pi}"/>
+	<origin xyz="0.188322 -0.007366 0.25882" rpy="0 0 ${pi}"/>
   <parent link="base_link"/>
   <child link="laser"/>

Commit message: (FG): add new files made by Luis Cuevas

File: bender_description/urdf/bender.xacro (robot description, xacro)
@@ -1,812 +1,725 @@
 <?xml version="1.0" ?>
 <robot name="bender" xmlns:xacro="http://www.ros.org/wiki/xacro">
-<link name="base_link">
-  <!--
-  <inertial>
-    <origin xyz="0.007788124759933493 -0.007355769738403454 0.7107401090172263" rpy="0 0 0"/>
-    <mass value="8.572188299348024"/>
-    <inertia ixx="1.515422" iyy="1.498033" izz="0.132123" ixy="-0.0" iyz="5.1e-05" ixz="-0.001283"/>
-  </inertial>
-  -->
-  <visual>
+  <xacro:include filename="$(find bender_description)/urdf/materials.xacro" />
+  <xacro:include filename="$(find bender_description)/urdf/rgbd_camera.xacro"/>
+  <xacro:include filename="$(find bender_description)/urdf/ros2_control.xacro" />
+  <xacro:property name="epsilon" value="1e-4"/>
+  <xacro:rgbd_camera
+      prefix=""
+      camera_name="camera"
+      parent='l2h_1'
+      xyz_offset="0.0435 0.03 0.160"
+      rpy_offset="0 0 0"/>
+  <link name="base_link">
+    <visual>
+      <origin xyz="0 0 0" rpy="0 0 0"/>
+      <geometry>
+        <mesh filename="file://$(find bender_description)/meshes/base_link.stl" scale="0.001 0.001 0.001"/>
+      </geometry>
+      <material name="silver"/>
+    </visual>
+    <collision>
+      <origin xyz="0 0 0" rpy="0 0 0"/>
+      <geometry>
+        <mesh filename="file://$(find bender_description)/meshes/base_link.stl" scale="0.001 0.001 0.001"/>
+      </geometry>
+    </collision>
+  </link>
+  <link name="l2l_1">
+    <inertial>
+      <origin xyz="-0.008469138038562633 4.816697341814002e-07 -0.07819087904751898" rpy="0 0 0"/>
+      <mass value="0.14071836856258027"/>
+      <inertia ixx="9.8e-05" iyy="0.000118" izz="8.7e-05" ixy="-0.0" iyz="-0.0" ixz="1.7e-05"/>
+    </inertial>
+    <visual>
+      <origin xyz="-0.035737 -0.247634 -1.04582" rpy="0 0 0"/>
+      <geometry>
+        <mesh filename="file://$(find bender_description)/meshes/l2l_1.stl" scale="0.001 0.001 0.001"/>
+      </geometry>
+      <material name="black"/>
+    </visual>
+    <collision>
+      <origin xyz="-0.035737 -0.247634 -1.04582" rpy="0 0 0"/>
+      <geometry>
+        <mesh filename="file://$(find bender_description)/meshes/l2l_1.stl" scale="0.001 0.001 0.001"/>
+      </geometry>
+    </collision>
+  </link>
+  <link name="l3l_1">
+    <inertial>
+      <origin xyz="-0.004049240589701097 -0.00011662761889197348 -0.1333626785766504" rpy="0 0 0"/>
+      <mass value="0.13433192894969845"/>
+      <inertia ixx="0.000296" iyy="0.000299" izz="4.9e-05" ixy="0.0" iyz="-0.0" ixz="4e-05"/>
+    </inertial>
+    <visual>
+      <origin xyz="-0.007987 -0.247634 -0.985406" rpy="0 0 0"/>
+      <geometry>
+        <mesh filename="file://$(find bender_description)/meshes/l3l_1.stl" scale="0.001 0.001 0.001"/>
+      </geometry>
+      <material name="grey"/>
+    </visual>
+    <collision>
+      <origin xyz="-0.007987 -0.247634 -0.985406" rpy="0 0 0"/>
+      <geometry>
+        <mesh filename="file://$(find bender_description)/meshes/l3l_1.stl" scale="0.001 0.001 0.001"/>
+      </geometry>
+    </collision>
+  </link>
+  <link name="l4l_1">
+    <inertial>
+      <origin xyz="-0.022033052289373113 -0.027751420924878867 -0.07009451131427447" rpy="0 0 0"/>
+      <mass value="0.1319735958452518"/>
+      <inertia ixx="6.8e-05" iyy="8e-05" izz="7.4e-05" ixy="-0.0" iyz="0.0" ixz="-2e-06"/>
+    </inertial>
+    <visual>
+      <origin xyz="-0.006819 -0.275388 -0.815556" rpy="0 0 0"/>
+      <geometry>
+        <mesh filename="file://$(find bender_description)/meshes/l4l_1.stl" scale="0.001 0.001 0.001"/>
+      </geometry>
+      <material name="black"/>
+    </visual>
+    <collision>
+      <origin xyz="-0.006819 -0.275388 -0.815556" rpy="0 0 0"/>
+      <geometry>
+        <mesh filename="file://$(find bender_description)/meshes/l4l_1.stl" scale="0.001 0.001 0.001"/>
+      </geometry>
+    </collision>
+  </link>
+  <link name="l5l_1">
+    <inertial>
+      <origin xyz="0.0039138191304953236 -6.519106588914747e-05 -0.1904912654580233" rpy="0 0 0"/>
+      <mass value="0.09538513786529154"/>
+      <inertia ixx="0.000748" iyy="0.000753" izz="3e-05" ixy="-0.0" iyz="-0.0" ixz="-5.3e-05"/>
+    </inertial>
+    <visual>
+      <origin xyz="-0.006819 -0.247637 -0.767806" rpy="0 0 0"/>
+      <geometry>
+        <mesh filename="file://$(find bender_description)/meshes/l5l_1.stl" scale="0.001 0.001 0.001"/>
+      </geometry>
+      <material name="grey"/>
+    </visual>
+    <collision>
+      <origin xyz="-0.006819 -0.247637 -0.767806" rpy="0 0 0"/>
+      <geometry>
+        <mesh filename="file://$(find bender_description)/meshes/l5l_1.stl" scale="0.001 0.001 0.001"/>
+      </geometry>
+    </collision>
+  </link>
+  <link name="l6l_1">
+    <inertial>
+      <origin xyz="1.1454305421428751e-07 -0.02225042100756011 -0.015076116417847174" rpy="0 0 0"/>
+      <mass value="0.004187419664904639"/>
+      <inertia ixx="2e-06" iyy="1e-06" izz="2e-06" ixy="-0.0" iyz="0.0" ixz="-0.0"/>
+    </inertial>
+    <visual>
+      <origin xyz="-0.007275 -0.269887 -0.504262" rpy="0 0 0"/>
+      <geometry>
+        <mesh filename="file://$(find bender_description)/meshes/l6l_1.stl" scale="0.001 0.001 0.001"/>
+      </geometry>
+      <material name="black"/>
+    </visual>
+    <collision>
+      <origin xyz="-0.007275 -0.269887 -0.504262" rpy="0 0 0"/>
+      <geometry>
+        <mesh filename="file://$(find bender_description)/meshes/l6l_1.stl" scale="0.001 0.001 0.001"/>
+      </geometry>
+    </collision>
+  </link>
+  <link name="l2r_1">
+    <inertial>
+      <origin xyz="-0.008469138038563282 4.816697872778164e-07 -0.07819087904754218" rpy="0 0 0"/>
+      <mass value="0.14071836856258027"/>
+      <inertia ixx="9.8e-05" iyy="0.000118" izz="8.7e-05" ixy="-0.0" iyz="-0.0" ixz="1.7e-05"/>
+    </inertial>
+    <visual>
+      <origin xyz="-0.035737 0.262366 -1.04582" rpy="0 0 0"/>
+      <geometry>
+        <mesh filename="file://$(find bender_description)/meshes/l2r_1.stl" scale="0.001 0.001 0.001"/>
+      </geometry>
+      <material name="black"/>
+    </visual>
+    <collision>
+      <origin xyz="-0.035737 0.262366 -1.04582" rpy="0 0 0"/>
+      <geometry>
+        <mesh filename="file://$(find bender_description)/meshes/l2r_1.stl" scale="0.001 0.001 0.001"/>
+      </geometry>
+    </collision>
+  </link>
+  <link name="l3r_1">
+    <inertial>
+      <origin xyz="-0.004049240589694631 -0.00011662761884700945 -0.1333626785766734" rpy="0 0 0"/>
+      <mass value="0.13433192894969845"/>
+      <inertia ixx="0.000296" iyy="0.000299" izz="4.9e-05" ixy="0.0" iyz="-0.0" ixz="4e-05"/>
+    </inertial>
+    <visual>
+      <origin xyz="-0.007987 0.262366 -0.985406" rpy="0 0 0"/>
+      <geometry>
+        <mesh filename="file://$(find bender_description)/meshes/l3r_1.stl" scale="0.001 0.001 0.001"/>
+      </geometry>
+      <material name="grey"/>
+    </visual>
+    <collision>
+      <origin xyz="-0.007987 0.262366 -0.985406" rpy="0 0 0"/>
+      <geometry>
+        <mesh filename="file://$(find bender_description)/meshes/l3r_1.stl" scale="0.001 0.001 0.001"/>
+      </geometry>
+    </collision>
+  </link>
+  <link name="l4r_1">
+    <inertial>
+      <origin xyz="-0.022033052289359936 0.02775238458496604 -0.070094511314298" rpy="0 0 0"/>
+      <mass value="0.1319735958452518"/>
+      <inertia ixx="6.8e-05" iyy="8e-05" izz="7.4e-05" ixy="-0.0" iyz="0.0" ixz="-2e-06"/>
+    </inertial>
+    <visual>
+      <origin xyz="-0.006819 0.290116 -0.815556" rpy="0 0 0"/>
+      <geometry>
+        <mesh filename="file://$(find bender_description)/meshes/l4r_1.stl" scale="0.001 0.001 0.001"/>
+      </geometry>
+      <material name="black"/>
+    </visual>
+    <collision>
+      <origin xyz="-0.006819 0.290116 -0.815556" rpy="0 0 0"/>
+      <geometry>
+        <mesh filename="file://$(find bender_description)/meshes/l4r_1.stl" scale="0.001 0.001 0.001"/>
+      </geometry>
+    </collision>
+  </link>
+  <link name="l5r_1">
+    <inertial>
+      <origin xyz="0.003913819130518236 -6.438555604931784e-05 -0.1904912654580455" rpy="0 0 0"/>
+      <mass value="0.09538513786529154"/>
+      <inertia ixx="0.000748" iyy="0.000753" izz="3e-05" ixy="-0.0" iyz="-0.0" ixz="-5.3e-05"/>
+    </inertial>
+    <visual>
+      <origin xyz="-0.006819 0.262364 -0.767806" rpy="0 0 0"/>
+      <geometry>
+        <mesh filename="file://$(find bender_description)/meshes/l5r_1.stl" scale="0.001 0.001 0.001"/>
+      </geometry>
+      <material name="grey"/>
+    </visual>
+    <collision>
+      <origin xyz="-0.006819 0.262364 -0.767806" rpy="0 0 0"/>
+      <geometry>
+        <mesh filename="file://$(find bender_description)/meshes/l5r_1.stl" scale="0.001 0.001 0.001"/>
+      </geometry>
+    </collision>
+  </link>
+  <link name="l6r_1">
+    <inertial>
+      <origin xyz="1.1454308115020628e-07 0.022250384502269127 -0.015076116417858498" rpy="0 0 0"/>
+      <mass value="0.004187419664904639"/>
+      <inertia ixx="2e-06" iyy="1e-06" izz="2e-06" ixy="-0.0" iyz="-0.0" ixz="0.0"/>
+    </inertial>
+    <visual>
+      <origin xyz="-0.007275 0.284614 -0.504262" rpy="0 0 0"/>
+      <geometry>
+        <mesh filename="file://$(find bender_description)/meshes/l6r_1.stl" scale="0.001 0.001 0.001"/>
+      </geometry>
+      <material name="black"/>
+    </visual>
+    <collision>
+      <origin xyz="-0.007275 0.284614 -0.504262" rpy="0 0 0"/>
+      <geometry>
+        <mesh filename="file://$(find bender_description)/meshes/l6r_1.stl" scale="0.001 0.001 0.001"/>
+      </geometry>
+    </collision>
+  </link>
+  <link name="l2h_1">
+    <inertial>
+      <origin xyz="-0.01404344492546073 0.030000481747364617 0.06449858090998739" rpy="0 0 0"/>
+      <mass value="3.4435410806483597"/>
+      <inertia ixx="0.011996" iyy="0.015757" izz="0.017434" ixy="0.0" iyz="-0.0" ixz="-0.000256"/>
+    </inertial>
+    <visual>
+      <origin xyz="-0.007987 0.037366 -1.28382" rpy="0 0 0"/>
+      <geometry>
+        <mesh filename="file://$(find bender_description)/meshes/l2h_1.stl" scale="0.001 0.001 0.001"/>
+      </geometry>
+      <material name="head"/>
+    </visual>
+    <!-- Ojo izquierdo -->
+    <visual>
+      <origin xyz="0.07 -0.00 0.055" rpy="1.5708 1.5708 1.5708"/> <!-- rotado para que sea un disco plano -->
+      <geometry>
+        <cylinder radius="0.045" length="0.001"/> <!-- radio 4mm, grosor 1mm -->
+      </geometry>
+      <material name="light_blue"/>
+    </visual>
+    <!-- Ojo derecho -->
+    <visual>
+      <origin xyz="0.07 0.06 0.055" rpy="1.5708 1.5708 1.5708"/> <!-- rotado para que sea un disco plano -->
+      <geometry>
+        <cylinder radius="0.045" length="0.001"/>
+      </geometry>
+      <material name="light_blue"/>
+    </visual>
+    <!-- Boca -->
+    <visual>
+      <origin xyz="0.07 0.03 0" rpy="0 0 0"/> <!-- rotado para que sea un disco plano -->
+      <geometry>
+        <box size="0.01 0.08 0.02"/>
+      </geometry>
+      <material name="casi_blue"/>
+    </visual>
+    <collision>
+      <origin xyz="-0.007987 0.037366 -1.28382" rpy="0 0 0"/>
+      <geometry>
+        <mesh filename="file://$(find bender_description)/meshes/l2h_1.stl" scale="0.001 0.001 0.001"/>
+      </geometry>
+    </collision>
+  </link>
+  <link name="g1r_1">
+    <inertial>
+      <origin xyz="6.478948623842799e-05 3.840721814474257e-07 -0.026736939315767316" rpy="0 0 0"/>
+      <mass value="0.12876405832743776"/>
+      <inertia ixx="8.6e-05" iyy="4.3e-05" izz="7e-05" ixy="-0.0" iyz="-0.0" ixz="0.0"/>
+    </inertial>
+    <visual>
+      <origin xyz="-0.007275 0.262364 -0.480247" rpy="0 0 0"/>
+      <geometry>
+        <mesh filename="file://$(find bender_description)/meshes/g1r_1.stl" scale="0.001 0.001 0.001"/>
+      </geometry>
+      <material name="grey"/>
+    </visual>
+    <collision>
+      <origin xyz="-0.007275 0.262364 -0.480247" rpy="0 0 0"/>
+      <geometry>
+        <mesh filename="file://$(find bender_description)/meshes/g1r_1.stl" scale="0.001 0.001 0.001"/>
+      </geometry>
+    </collision>
+  </link>
+  <link name="g2ra_1">
+    <inertial>
+      <origin xyz="-0.0220993118378398 0.01442646877260062 -0.05721188075257794" rpy="0 0 0"/>
+      <mass value="0.05474843522698835"/>
+      <inertia ixx="3.9e-05" iyy="3.7e-05" izz="2e-05" ixy="-0.0" iyz="-1e-05" ixz="0.0"/>
+    </inertial>
+    <visual>
+      <origin xyz="-0.029225 0.243864 -0.438647" rpy="0 0 0"/>
+      <geometry>
+        <mesh filename="file://$(find bender_description)/meshes/g2ra_1.stl" scale="0.001 0.001 0.001"/>
+      </geometry>
+      <material name="blue"/>
+    </visual>
+    <collision>
+      <origin xyz="-0.029225 0.243864 -0.438647" rpy="0 0 0"/>
+      <geometry>
+        <mesh filename="file://$(find bender_description)/meshes/g2ra_1.stl" scale="0.001 0.001 0.001"/>
+      </geometry>
+    </collision>
+  </link>
+  <link name="g2rb_1">
+    <inertial>
+      <origin xyz="-0.02210045907599773 -0.014425699768063904 -0.05721188075257849" rpy="0 0 0"/>
+      <mass value="0.05474843522698835"/>
+      <inertia ixx="3.9e-05" iyy="3.7e-05" izz="2e-05" ixy="-0.0" iyz="1e-05" ixz="-0.0"/>
+    </inertial>
+    <visual>
+      <origin xyz="-0.029225 0.280864 -0.438647" rpy="0 0 0"/>
+      <geometry>
+        <mesh filename="file://$(find bender_description)/meshes/g2rb_1.stl" scale="0.001 0.001 0.001"/>
+      </geometry>
+      <material name="blue"/>
+    </visual>
+    <collision>
+      <origin xyz="-0.029225 0.280864 -0.438647" rpy="0 0 0"/>
+      <geometry>
+        <mesh filename="file://$(find bender_description)/meshes/g2rb_1.stl" scale="0.001 0.001 0.001"/>
+      </geometry>
+    </collision>
+  </link>
+  <link name="g1l_1">
+    <inertial>
+      <origin xyz="6.478948621099247e-05 -4.2143764839019937e-07 -0.026736939315755603" rpy="0 0 0"/>
+      <mass value="0.12876405832743776"/>
+      <inertia ixx="8.6e-05" iyy="4.3e-05" izz="7e-05" ixy="-0.0" iyz="-0.0" ixz="0.0"/>
+    </inertial>
+    <visual>
+      <origin xyz="-0.007275 -0.247637 -0.480247" rpy="0 0 0"/>
+      <geometry>
+        <mesh filename="file://$(find bender_description)/meshes/g1l_1.stl" scale="0.001 0.001 0.001"/>
+      </geometry>
+      <material name="grey"/>
+    </visual>
+    <collision>
+      <origin xyz="-0.007275 -0.247637 -0.480247" rpy="0 0 0"/>
+      <geometry>
+        <mesh filename="file://$(find bender_description)/meshes/g1l_1.stl" scale="0.001 0.001 0.001"/>
+      </geometry>
+    </collision>
+  </link>
+  <link name="g2lb_1">
+    <inertial>
+      <origin xyz="-0.022099311837869458 0.014425663262769728 -0.057211880752566724" rpy="0 0 0"/>
+      <mass value="0.05474843522698835"/>
+      <inertia ixx="3.9e-05" iyy="3.7e-05" izz="2e-05" ixy="-0.0" iyz="-1e-05" ixz="0.0"/>
+    </inertial>
+    <visual>
+      <origin xyz="-0.029225 -0.266137 -0.438647" rpy="0 0 0"/>
+      <geometry>
+        <mesh filename="file://$(find bender_description)/meshes/g2lb_1.stl" scale="0.001 0.001 0.001"/>
+      </geometry>
+      <material name="red"/>
+    </visual>
+    <collision>
+      <origin xyz="-0.029225 -0.266137 -0.438647" rpy="0 0 0"/>
+      <geometry>
+        <mesh filename="file://$(find bender_description)/meshes/g2lb_1.stl" scale="0.001 0.001 0.001"/>
+      </geometry>
+    </collision>
+  </link>
+  <link name="g2la_1">
+    <inertial>
+      <origin xyz="-0.022100459076024488 -0.01442650527789352 -0.057211880752566335" rpy="0 0 0"/>
+      <mass value="0.05474843522698835"/>
+      <inertia ixx="3.9e-05" iyy="3.7e-05" izz="2e-05" ixy="-0.0" iyz="1e-05" ixz="-0.0"/>
+    </inertial>
+    <visual>
+      <origin xyz="-0.029225 -0.229137 -0.438647" rpy="0 0 0"/>
+      <geometry>
+        <mesh filename="file://$(find bender_description)/meshes/g2la_1.stl" scale="0.001 0.001 0.001"/>
+      </geometry>
+      <material name="red"/>
+    </visual>
+    <collision>
+      <origin xyz="-0.029225 -0.229137 -0.438647" rpy="0 0 0"/>
+      <geometry>
+        <mesh filename="file://$(find bender_description)/meshes/g2la_1.stl" scale="0.001 0.001 0.001"/>
+      </geometry>
+    </collision>
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
File: bender_description/urdf/materials.xacro (robot description, xacro)
@@ -1,6 +1,30 @@
-<?xml version="1.0" ?>
-<robot name="bender" xmlns:xacro="http://www.ros.org/wiki/xacro" >
-<material name="silver">
-  <color rgba="0.700 0.700 0.700 1.000"/>
-</material>
+<?xml version="1.0"?>
+<robot>
+  <material name="black">
+    <color rgba="0.0 0.0 0.0 1.0"/>
+  </material>
+  <material name="grey">
+    <color rgba="0.3 0.3 0.3 1.0"/>
+  </material>
+  <material name="white">
+    <color rgba="1.0 1.0 1.0 1.0"/>
+  </material>
+  <material name="silver">
+    <color rgba="0.55 0.55 0.55 1.0"/>
+  </material>
+  <material name="head">
+    <color rgba="0.65 0.65 0.65 1.0"/>
+  </material>
+  <material name="blue">
+    <color rgba="0 0 1 0.5"/>
+  </material>
+  <material name="red">
+    <color rgba="1 0 0 0.5"/>
+  </material>
+  <material name="light_blue">
+    <color rgba="0.6 0.8 1 1"/>
+  </material>
+  <material name="casi_blue">
+    <color rgba="0.2 0.3 1 1"/>
+  </material>
 </robot>
