Commit message: FG: add limits and motor recentering

File: bender_description/urdf/bender.xacro (robot description, xacro)
@@ -646,5 +646,5 @@
     <child link="l4r_1"/>
     <axis xyz="-0.0 -1.0 0.0"/>
-    <limit upper="${2.356194 + epsilon}" lower="${-epsilon}" effort="100" velocity="100"/>
+    <limit upper="${2.356194 + epsilon}" lower="-3.14" effort="100" velocity="100"/>
   </joint>
   <joint name="l5r_to_l4r" type="revolute">
@@ -662,4 +662,5 @@
     <limit upper="${1.570796 + epsilon}" lower="${-1.570796 - epsilon}" effort="100" velocity="100"/>
   </joint>
+  <!-- head pitch joint -->
   <joint name="l2h_to_l1h" type="revolute">
     <origin rpy="0 0 0" xyz="0.0 -0.03 0.07"/>
@@ -669,4 +670,12 @@
     <limit effort="50" lower="${-0.706858 - epsilon}" upper="${0.706858 + epsilon}" velocity="50"/>
   </joint>
+  <!-- head roll joint -->
+  <!-- <joint name="l3h_to_l2h" type="revolute">
+    <origin rpy="0 0 0" xyz="0.0 -0.03 0.07"/>
+    <parent link="l2h_1"/>
+    <child link="l3h_1"/>
+    <axis xyz="-0.0 -1.0 0.0"/>
+    <limit effort="50" lower="${-0.706858 - epsilon}" upper="${0.706858 + epsilon}" velocity="50"/>
+  </joint> -->
   <joint name="g1r_to_l6r" type="fixed">
     <origin xyz="0.0 0.02225 -0.024015" rpy="0 0 0"/>

File: bender_description/urdf/ros2_control.xacro (robot description, xacro)
@@ -1,5 +1,5 @@
 <?xml version="1.0" ?>
 <robot xmlns:xacro="http://www.ros.org/wiki/xacro">
-<xacro:macro name="odrive_ros2_control" params="name serial_number joint_name axis:=0">
+<!-- <xacro:macro name="odrive_ros2_control" params="name serial_number joint_name axis:=0">
     <ros2_control name="${name}" type="system">
       <hardware>
@@ -37,5 +37,5 @@
     <actuator name="motor_l1l_to_base_link" role="actuator1"/>
     <joint name="l1l_to_base_link" role="joint1">
-      <mechanicalReduction>10.0</mechanicalReduction> <!-- Cambiar reducción-->
+      <mechanicalReduction>10.0</mechanicalReduction>
     </joint>
   </transmission>
@@ -44,5 +44,5 @@
     <actuator name="motor_l1r_to_base_link" role="actuator1"/>
     <joint name="l1r_to_base_link" role="joint1">
-      <mechanicalReduction>10.0</mechanicalReduction><!-- Cambiar reducción-->
+      <mechanicalReduction>10.0</mechanicalReduction>
     </joint>
   </transmission>
@@ -61,5 +61,5 @@
              <state_interface name="velocity" />
            </sensor>
-         </ros2_control>
+         </ros2_control> -->
          <ros2_control name="DynamixelChainMain" type="system">
              <hardware>
@@ -148,4 +148,6 @@
                 <state_interface name="Present Velocity" />
                 <state_interface name="Present Load" />
+                <!-- software re-center -->
+                <param name="[unit info]">Present Position, 0.001533981, rad, unsigned, -3.1001879291; Goal Position, 0.001533981, rad, unsigned, -3.1001879291</param>
                 <param name="P Gain">8</param>
                 <param name="I Gain">2</param>
@@ -160,4 +162,5 @@
                 <state_interface name="Present Velocity" />
                 <state_interface name="Present Load" />
+                <!-- doesn't need recentering -->
                 <param name="CW Compliance Margin">1</param>
                 <param name="CCW Compliance Margin">1</param>
@@ -173,4 +176,5 @@
                 <state_interface name="Present Velocity" />
                 <state_interface name="Present Load" />
+                <param name="[unit info]">Present Position, 0.001533981, rad, unsigned, -3.471399003; Goal Position, 0.001533981, rad, unsigned, -3.471399003</param>
                 <param name="P Gain">8</param>
                 <param name="I Gain">2</param>
@@ -211,4 +215,5 @@
                 <state_interface name="Present Velocity" />
                 <state_interface name="Present Load" />
+                <param name="[unit info]">Present Position, 0.001047198, rad, unsigned, -1.6221098; Goal Position, 0.001047198, rad, unsigned, -1.6221098</param>
                 <param name="CW Compliance Margin">1</param>
                 <param name="CCW Compliance Margin">1</param>
@@ -224,4 +229,5 @@
                 <state_interface name="Present Velocity" />
                 <state_interface name="Present Load" />
+                <param name="[unit info]">Present Position, 0.005061455, rad, unsigned, -2.070135026; Goal Position, 0.005061455, rad, unsigned, -2.070135026</param>
                 <param name="CW Compliance Margin">1</param>
                 <param name="CCW Compliance Margin">1</param>
@@ -320,4 +326,5 @@
                <state_interface name="Present Velocity" />
                <state_interface name="Present Load" />
+               <param name="[unit info]">Present Position, 0.001533981, rad, unsigned, -2.963651292; Goal Position, 0.001533981, rad, unsigned, -2.963651292</param>
                <param name="P Gain">8</param>
                <param name="I Gain">2</param>
@@ -325,5 +332,5 @@
                <param name="Return Delay Time">25</param>
              </gpio>
-             <!-- <gpio name="motor_l2h_master">
+             <!-- <gpio name="motor_l2h_1">
                 <param name="type">dxl</param>
                 <param name="ID">20</param>
@@ -338,5 +345,5 @@
                 <param name="Return Delay Time">25</param>
              </gpio>
-             <gpio name="motor_l2h_slave">
+             <gpio name="motor_l2h_2">
                 <param name="type">dxl</param>
                 <param name="ID">21</param>
@@ -352,17 +359,3 @@
              </gpio> -->
            </ros2_control>
-<!--
-           <ros2_control name="DynamixelChainSlow" type="system">
-             <hardware>
-               <plugin>dynamixel_hardware_interface/DynamixelHardware</plugin>
-               <param name="port_name">/dev/dynamixel</param>
-               <param name="baud_rate">57600</param>
-               <param name="protocol_version">1.0</param>
-               <param name="number_of_joints">1</param>
-               <param name="number_of_transmissions">1</param>
-               <param name="dynamixel_model_folder">/param/dxl_model</param>
-               <param name="disable_torque_at_init">true</param>
-               <param name="torque_enable">0</param>
-             </hardware>
-           </ros2_control> -->
 </robot>

Commit message: (FG): add left gripper

File: bender_description/urdf/bender.xacro (robot description, xacro)
@@ -330,67 +330,6 @@
     </collision>
   </link>
-  <!-- <link name="g1l_1">
-    <inertial>
-      <origin xyz="6.478948621099247e-05 -4.2143764839019937e-07 -0.026736939315755603" rpy="0 0 0"/>
-      <mass value="0.12876405832743776"/>
-      <inertia ixx="8.6e-05" iyy="4.3e-05" izz="7e-05" ixy="-0.0" iyz="-0.0" ixz="0.0"/>
-    </inertial>
-    <visual>
-      <origin xyz="-0.007275 -0.247637 -0.480247" rpy="0 0 0"/>
-      <geometry>
-        <mesh filename="file://$(find bender_description)/meshes/g1l_1.stl" scale="0.001 0.001 0.001"/>
-      </geometry>
-      <material name="grey"/>
-    </visual>
-    <collision>
-      <origin xyz="-0.007275 -0.247637 -0.480247" rpy="0 0 0"/>
-      <geometry>
-        <mesh filename="file://$(find bender_description)/meshes/g1l_1.stl" scale="0.001 0.001 0.001"/>
-      </geometry>
-    </collision>
-  </link>
- -->
-  <!-- <link name="g2lb_1">
-    <inertial>
-      <origin xyz="-0.022099311837869458 0.014425663262769728 -0.057211880752566724" rpy="0 0 0"/>
-      <mass value="0.05474843522698835"/>
-      <inertia ixx="3.9e-05" iyy="3.7e-05" izz="2e-05" ixy="-0.0" iyz="-1e-05" ixz="0.0"/>
-    </inertial>
-    <visual>
-      <origin xyz="-0.029225 -0.266137 -0.438647" rpy="0 0 0"/>
-      <geometry>
-        <mesh filename="file://$(find bender_description)/meshes/g2lb_1.stl" scale="0.001 0.001 0.001"/>
-      </geometry>
-      <material name="red"/>
-    </visual>
-    <collision>
-      <origin xyz="-0.029225 -0.266137 -0.438647" rpy="0 0 0"/>
-      <geometry>
-        <mesh filename="file://$(find bender_description)/meshes/g2lb_1.stl" scale="0.001 0.001 0.001"/>
-      </geometry>
-    </collision>
-  </link> -->
-  <!-- <link name="g2la_1">
-    <inertial>
-      <origin xyz="-0.022100459076024488 -0.01442650527789352 -0.057211880752566335" rpy="0 0 0"/>
-      <mass value="0.05474843522698835"/>
-      <inertia ixx="3.9e-05" iyy="3.7e-05" izz="2e-05" ixy="-0.0" iyz="1e-05" ixz="-0.0"/>
-    </inertial>
-    <visual>
-      <origin xyz="-0.029225 -0.229137 -0.438647" rpy="0 0 0"/>
-      <geometry>
-        <mesh filename="file://$(find bender_description)/meshes/g2la_1.stl" scale="0.001 0.001 0.001"/>
-      </geometry>
-      <material name="red"/>
-    </visual>
-    <collision>
-      <origin xyz="-0.029225 -0.229137 -0.438647" rpy="0 0 0"/>
-      <geometry>
-        <mesh filename="file://$(find bender_description)/meshes/g2la_1.stl" scale="0.001 0.001 0.001"/>
-      </geometry>
-    </collision>
-  </link> -->
   <joint name="l6l_to_gripper" type="fixed">
-      <origin xyz="0.0 -0.02225 -0.024015" rpy="0 0 0"/>
+      <origin xyz="0.0 -0.02225 -0.091" rpy="0 3.14159 0"/>
       <parent link="l6l_1"/>
       <child link="gripper_l_base"/>
@@ -400,5 +339,5 @@
         <origin rpy="0 0 0" xyz="0 0 0"/>
         <geometry>
-          <mesh filename="package://robot_gripper/meshes/base.stl"/>
+          <mesh filename="file://$(find bender_description)/meshes/base.stl" scale="0.001 0.001 0.001"/>
         </geometry>
       </visual>
@@ -413,5 +352,5 @@
         <origin rpy="0 0 0" xyz="0 0 0"/>
         <geometry>
-          <mesh filename="package://robot_gripper/meshes/fijo_v2.stl"/>
+          <mesh filename="file://$(find bender_description)/meshes/fijo_v2.stl" scale="0.001 0.001 0.001"/>
         </geometry>
       </visual>
@@ -419,5 +358,5 @@
     <joint name="gripper_base_to_movil" type="revolute">
       <axis xyz="0 1 0"/>
-      <origin rpy="0 0 0" xyz="-18.69 0 -19.45"/>
+      <origin rpy="0 0 0" xyz="-0.01869 0 -0.01945"/>
       <parent link="gripper_l_base"/>
       <child link="movil"/>
@@ -428,5 +367,5 @@
         <origin rpy="0 0 0" xyz="0 0 0"/>
         <geometry>
-          <mesh filename="package://robot_gripper/meshes/movil2.stl"/>
+          <mesh filename="file://$(find bender_description)/meshes/movil2.stl" scale="0.001 0.001 0.001"/>
         </geometry>
       </visual>
