Commit message: (FG): new joint origins in ros2 control

File: bender_description/urdf/bender.xacro (robot description, xacro)
@@ -536,5 +536,5 @@
     <child link="l2l_1"/>
     <axis xyz="-1.0 0.0 -0.0"/>
-    <limit upper="${epsilon}" lower="${-1.570796 - epsilon}" effort="100" velocity="100"/>
+    <limit upper="0.09" lower="${-1.570796 - epsilon}" effort="100" velocity="100"/>
   </joint>
   <joint name="l3l_to_l2l" type="revolute">
@@ -550,5 +550,5 @@
     <child link="l4l_1"/>
     <axis xyz="-0.0 -1.0 0.0"/>
-    <limit upper="${2.356194 + epsilon}" lower="${-epsilon}" effort="100" velocity="100"/>
+    <limit upper="${2.356194 + epsilon}" lower="-1.5" effort="100" velocity="100"/>
   </joint>
   <joint name="l5l_to_l4l" type="revolute">
@@ -571,5 +571,5 @@
     <child link="l2r_1"/>
     <axis xyz="1.0 0.0 0.0"/>
-    <limit upper="${epsilon}" lower="${-1.570796 -epsilon}" effort="100" velocity="100"/>
+    <limit upper="0.1" lower="${-1.570796 - 0.1}" effort="100" velocity="100"/>
   </joint>
   <joint name="l3r_to_l2r" type="revolute">

File: bender_description/urdf/ros2_control.xacro (robot description, xacro)
@@ -70,11 +70,49 @@
 		</joint>
 		<gpio name="motor_l2r">
-			<param name="type">dxl</param>
-			<param name="ID">11</param>
-			<command_interface name="Goal Position" />
-			<state_interface name="Present Position" />
-			<state_interface name="Present Velocity" />
-			<state_interface name="Present Load" />
-			<param name="[unit info]">Present Position, 0.001533981, rad, unsigned, -3.1001879291; Goal Position, 0.001533981, rad, unsigned, -3.1001879291</param>
+    		<param name="type">dxl</param>
+    		<param name="ID">4</param>
+    		<command_interface name="Goal Position" />
+    		<state_interface name="Present Position" />
+    		<state_interface name="Present Velocity" />
+    		<state_interface name="Present Load" />
+    		<param name="[unit info]">Present Position, 0.001047198, rad, unsigned, -1.6221098; Goal Position, 0.001047198, rad, unsigned, -1.6221098</param>
+    		<param name="CW Compliance Margin">1</param>
+    		<param name="CCW Compliance Margin">1</param>
+    		<param name="CW Compliance Slope">254</param>
+    		<param name="CCW Compliance Slope">254</param>
+    		<param name="Return Delay Time">25</param>
+		</gpio>
+		<joint name="l3r_to_l2r">
+			<command_interface name="position" />
+			<state_interface name="position" />
+			<state_interface name="velocity" />
+		</joint>
+		<gpio name="motor_l3r">
+			<param name="type">dxl</param>
+			<param name="ID">3</param>
+			<command_interface name="Goal Position" />
+			<state_interface name="Present Position" />
+			<state_interface name="Present Velocity" />
+			<state_interface name="Present Load" />
+			<param name="[unit info]">Present Position, 0.005061455, rad, unsigned, -2.04988725; Goal Position, 0.005061455, rad, unsigned, -2.04988725</param>
+			<param name="CW Compliance Margin">1</param>
+			<param name="CCW Compliance Margin">1</param>
+			<param name="CW Compliance Slope">254</param>
+			<param name="CCW Compliance Slope">254</param>
+			<param name="Return Delay Time">25</param>
+		</gpio>
+		<joint name="l4r_to_l3r">
+			<command_interface name="position" />
+			<state_interface name="position" />
+			<state_interface name="velocity" />
+		</joint>
+		<gpio name="motor_l4r">
+			<param name="type">dxl</param>
+			<param name="ID">13</param>
+			<command_interface name="Goal Position" />
+			<state_interface name="Present Position" />
+			<state_interface name="Present Velocity" />
+			<state_interface name="Present Load" />
+			<param name="[unit info]">Present Position, 0.001533981, rad, unsigned, -3.05262219; Goal Position, 0.001533981, rad, unsigned, -3.05262219</param>
 			<param name="P Gain">8</param>
 			<param name="I Gain">2</param>
@@ -82,10 +120,64 @@
 			<param name="Return Delay Time">25</param>
 		</gpio>
-		<joint name="l3r_to_l2r">
-			<command_interface name="position" />
-			<state_interface name="position" />
-			<state_interface name="velocity" />
-		</joint>
-		<gpio name="motor_l3r">
+		<joint name="l5r_to_l4r">
+			<command_interface name="position" />
+			<state_interface name="position" />
+			<state_interface name="velocity" />
+		</joint>
+		<gpio name="motor_l5r">
+			<param name="type">dxl</param>
+			<param name="ID">5</param>
+			<command_interface name="Goal Position" />
+			<state_interface name="Present Position" />
+			<state_interface name="Present Velocity" />
+			<state_interface name="Present Load" />
+			<param name="CW Compliance Margin">1</param>
+			<param name="CCW Compliance Margin">1</param>
+			<param name="CW Compliance Slope">254</param>
+			<param name="CCW Compliance Slope">254</param>
+			<param name="Return Delay Time">25</param>
+		</gpio>
+		<joint name="l6r_to_l5r">
+			<command_interface name="position" />
+			<state_interface name="position" />
+			<state_interface name="velocity" />
+		</joint>
+		<gpio name="motor_l6r">
+			<param name="type">dxl</param>
+			<param name="ID">15</param>
+			<command_interface name="Goal Position" />
+			<state_interface name="Present Position" />
+			<state_interface name="Present Velocity" />
+			<state_interface name="Present Load" />
+			<param name="[unit info]">Present Position, 0.005061455, rad, unsigned, -1.94866011; Goal Position, 0.005061455, rad, unsigned, -1.94866011</param>
+			<param name="CW Compliance Margin">1</param>
+			<param name="CCW Compliance Margin">1</param>
+			<param name="CW Compliance Slope">254</param>
+			<param name="CCW Compliance Slope">254</param>
+			<param name="Return Delay Time">25</param>
+		</gpio>
+		<joint name="l2l_to_l1l">
+			<command_interface name="position" />
+			<state_interface name="position" />
+			<state_interface name="velocity" />
+		</joint>
+		<gpio name="motor_l2l">
+    		<param name="type">dxl</param>
+    		<param name="ID">1</param>
+    		<command_interface name="Goal Position" />
+    		<state_interface name="Present Position" />
+    		<state_interface name="Present Velocity" />
+    		<state_interface name="Present Load" />
+    		<param name="P Gain">8</param>
+    		<param name="I Gain">2</param>
+    		<param name="D Gain">5</param>
+    		<param name="Return Delay Time">25</param>
+		</gpio>
+		<joint name="l3l_to_l2l">
+			<command_interface name="position" />
+			<state_interface name="position" />
+			<state_interface name="velocity" />
+		</joint>
+		<gpio name="motor_l3l">
 			<param name="type">dxl</param>
 			<param name="ID">12</param>
@@ -94,23 +186,24 @@
 			<state_interface name="Present Velocity" />
 			<state_interface name="Present Load" />
-			<param name="CW Compliance Margin">1</param>
-			<param name="CCW Compliance Margin">1</param>
-			<param name="CW Compliance Slope">254</param>
-			<param name="CCW Compliance Slope">254</param>
-			<param name="Return Delay Time">25</param>
-		</gpio>
-		<joint name="l4r_to_l3r">
-			<command_interface name="position" />
-			<state_interface name="position" />
-			<state_interface name="velocity" />
-		</joint>
-		<gpio name="motor_l4r">
-			<param name="type">dxl</param>
-			<param name="ID">13</param>
-			<command_interface name="Goal Position" />
-			<state_interface name="Present Position" />
-			<state_interface name="Present Velocity" />
-			<state_interface name="Present Load" />
-			<param name="[unit info]">Present Position, 0.001533981, rad, unsigned, -3.471399003; Goal Position, 0.001533981, rad, unsigned, -3.471399003</param>
+			<param name="[unit info]">Present Position, 0.005061455, rad, unsigned, -2.566157685; Goal Position, 0.005061455, rad, unsigned, -2.566157685</param>
+			<param name="CW Compliance Margin">1</param>
+			<param name="CCW Compliance Margin">1</param>
+			<param name="CW Compliance Slope">254</param>
+			<param name="CCW Compliance Slope">254</param>
+			<param name="Return Delay Time">25</param>
+		</gpio>
+		<joint name="l4l_to_l3l">
+			<command_interface name="position" />
+			<state_interface name="position" />
+			<state_interface name="velocity" />
+		</joint>
+		<gpio name="motor_l4l">
+			<param name="type">dxl</param>
+			<param name="ID">11</param>
+			<command_interface name="Goal Position" />
+			<state_interface name="Present Position" />
+			<state_interface name="Present Velocity" />
+			<state_interface name="Present Load" />
+			<param name="[unit info]">Present Position, 0.001533981, rad, unsigned, -3.040350342; Goal Position, 0.001533981, rad, unsigned, -3.040350342</param>
 			<param name="P Gain">8</param>
 			<param name="I Gain">2</param>
@@ -118,104 +211,12 @@
 			<param name="Return Delay Time">25</param>
 		</gpio>
-		<joint name="l5r_to_l4r">
-			<command_interface name="position" />
-			<state_interface name="position" />
-			<state_interface name="velocity" />
-		</joint>
-		<gpio name="motor_l5r">
+		<joint name="l5l_to_l4l">
+			<command_interface name="position" />
+			<state_interface name="position" />
+			<state_interface name="velocity" />
+		</joint>
+		<gpio name="motor_l5l">
 			<param name="type">dxl</param>
 			<param name="ID">14</param>
-			<command_interface name="Goal Position" />
-			<state_interface name="Present Position" />
-			<state_interface name="Present Velocity" />
-			<state_interface name="Present Load" />
-			<param name="CW Compliance Margin">1</param>
-			<param name="CCW Compliance Margin">1</param>
-			<param name="CW Compliance Slope">254</param>
-			<param name="CCW Compliance Slope">254</param>
-			<param name="Return Delay Time">25</param>
-		</gpio>
-		<joint name="l6r_to_l5r">
-			<command_interface name="position" />
-			<state_interface name="position" />
-			<state_interface name="velocity" />
-		</joint>
-		<gpio name="motor_l6r">
-			<param name="type">dxl</param>
-			<param name="ID">15</param>
-			<command_interface name="Goal Position" />
-			<state_interface name="Present Position" />
-			<state_interface name="Present Velocity" />
-			<state_interface name="Present Load" />
-			<param name="CW Compliance Margin">1</param>
-			<param name="CCW Compliance Margin">1</param>
-			<param name="CW Compliance Slope">254</param>
-			<param name="CCW Compliance Slope">254</param>
-			<param name="Return Delay Time">25</param>
-		</gpio>
-		<joint name="l2l_to_l1l">
-			<command_interface name="position" />
-			<state_interface name="position" />
-			<state_interface name="velocity" />
-		</joint>
-		<gpio name="motor_l2l">
-			<param name="type">dxl</param>
-			<param name="ID">4</param>
-			<command_interface name="Goal Position" />
-			<state_interface name="Present Position" />
-			<state_interface name="Present Velocity" />
-			<state_interface name="Present Load" />
-			<param name="[unit info]">Present Position, 0.001047198, rad, unsigned, -1.6221098; Goal Position, 0.001047198, rad, unsigned, -1.6221098</param>
-			<param name="CW Compliance Margin">1</param>
-			<param name="CCW Compliance Margin">1</param>
-			<param name="CW Compliance Slope">254</param>
-			<param name="CCW Compliance Slope">254</param>
-			<param name="Return Delay Time">25</param>
-		</gpio>
-		<joint name="l3l_to_l2l">
-			<command_interface name="position" />
-			<state_interface name="position" />
-			<state_interface name="velocity" />
-		</joint>
-		<gpio name="motor_l3l">
-			<param name="type">dxl</param>
-			<param name="ID">3</param>
-			<command_interface name="Goal Position" />
-			<state_interface name="Present Position" />
-			<state_interface name="Present Velocity" />
-			<state_interface name="Present Load" />
-			<param name="[unit info]">Present Position, 0.005061455, rad, unsigned, -2.070135026; Goal Position, 0.005061455, rad, unsigned, -2.070135026</param>
-			<param name="CW Compliance Margin">1</param>
-			<param name="CCW Compliance Margin">1</param>
-			<param name="CW Compliance Slope">254</param>
-			<param name="CCW Compliance Slope">254</param>
-			<param name="Return Delay Time">25</param>
-		</gpio>
-		<joint name="l4l_to_l3l">
-			<command_interface name="position" />
-			<state_interface name="position" />
-			<state_interface name="velocity" />
-		</joint>
-		<gpio name="motor_l4l">
-			<param name="type">dxl</param>
-			<param name="ID">1</param>
-			<command_interface name="Goal Position" />
-			<state_interface name="Present Position" />
-			<state_interface name="Present Velocity" />
-			<state_interface name="Present Load" />
-			<param name="[unit info]">Present Position, 0.001533981, rad, unsigned, -2.963651292; Goal Position, 0.001533981, rad, unsigned, -2.963651292</param>
-			<param name="P Gain">8</param>
-			<param name="I Gain">2</param>
-			<param name="D Gain">5</param>
-			<param name="Return Delay Time">25</param>
-		</gpio>
-		<joint name="l5l_to_l4l">
-			<command_interface name="position" />
-			<state_interface name="position" />
-			<state_interface name="velocity" />
-		</joint>
-		<gpio name="motor_l5l">
-			<param name="type">dxl</param>
-			<param name="ID">5</param>
 			<command_interface name="Goal Position" />
 			<state_interface name="Present Position" />
