Commit message: (FG): add new moveit config

File: bender_description/urdf/bender.xacro (robot description, xacro)
@@ -336,39 +336,57 @@
     </joint>
     <link name="gripper_l_base">
-      <visual>
-        <origin rpy="0 0 0" xyz="0 0 0"/>
-        <geometry>
-          <mesh filename="file://$(find bender_description)/meshes/base.stl" scale="0.001 0.001 0.001"/>
-        </geometry>
-      </visual>
-    </link>
-    <joint name="gripper_base_to_fijo" type="fixed">
-      <parent link="gripper_l_base"/>
-      <child link="fijo"/>
-      <origin xyz="0 0 0"/>
-    </joint>
-    <link name="fijo">
-      <visual>
-        <origin rpy="0 0 0" xyz="0 0 0"/>
-        <geometry>
-          <mesh filename="file://$(find bender_description)/meshes/fijo_v2.stl" scale="0.001 0.001 0.001"/>
-        </geometry>
-      </visual>
-    </link>
-    <joint name="gripper_base_to_movil" type="revolute">
-      <axis xyz="0 1 0"/>
-      <origin rpy="0 0 0" xyz="-0.01869 0 -0.01945"/>
-      <parent link="gripper_l_base"/>
-      <child link="movil"/>
-      <limit effort="1000.0" lower="0.0" upper="0.5" velocity="0.5"/>
-    </joint>
-    <link name="movil">
-      <visual>
-        <origin rpy="0 0 0" xyz="0 0 0"/>
-        <geometry>
-          <mesh filename="file://$(find bender_description)/meshes/movil2.stl" scale="0.001 0.001 0.001"/>
-        </geometry>
-      </visual>
-    </link>
+          <visual>
+            <origin rpy="0 0 0" xyz="0 0 0"/>
+            <geometry>
+              <mesh filename="file://$(find bender_description)/meshes/base.stl" scale="0.001 0.001 0.001"/>
+            </geometry>
+          </visual>
+          <collision>
+            <origin rpy="0 0 0" xyz="0 0 0"/>
+            <geometry>
+              <mesh filename="file://$(find bender_description)/meshes/base.stl" scale="0.001 0.001 0.001"/>
+            </geometry>
+          </collision>
+        </link>
+        <joint name="gripper_base_to_fijo" type="fixed">
+          <parent link="gripper_l_base"/>
+          <child link="fijo"/>
+          <origin xyz="0 0 0"/>
+        </joint>
+        <link name="fijo">
+          <visual>
+            <origin rpy="0 0 0" xyz="0 0 0"/>
+            <geometry>
+              <mesh filename="file://$(find bender_description)/meshes/fijo_v2.stl" scale="0.001 0.001 0.001"/>
+            </geometry>
+          </visual>
+          <collision>
+            <origin rpy="0 0 0" xyz="0 0 0"/>
+            <geometry>
+              <mesh filename="file://$(find bender_description)/meshes/fijo_v2.stl" scale="0.001 0.001 0.001"/>
+            </geometry>
+          </collision>
+        </link>
+        <joint name="gripper_base_to_movil" type="revolute">
+          <axis xyz="0 1 0"/>
+          <origin rpy="0 -1.0 0" xyz="-0.01869 0 -0.01945"/>
+          <parent link="gripper_l_base"/>
+          <child link="movil"/>
+          <limit effort="1000.0" lower="0.0" upper="0.5" velocity="0.5"/>
+        </joint>
+        <link name="movil">
+          <visual>
+            <origin rpy="0 0 0" xyz="0 0 0"/>
+            <geometry>
+              <mesh filename="file://$(find bender_description)/meshes/movil2.stl" scale="0.001 0.001 0.001"/>
+            </geometry>
+          </visual>
+          <collision>
+            <origin rpy="0 0 0" xyz="0 0 0"/>
+            <geometry>
+              <mesh filename="file://$(find bender_description)/meshes/movil2.stl" scale="0.001 0.001 0.001"/>
+            </geometry>
+          </collision>
+        </link>
   <link name="laser_1">
     <inertial>
@@ -536,5 +554,5 @@
     <child link="l2l_1"/>
     <axis xyz="-1.0 0.0 -0.0"/>
-    <limit upper="0.09" lower="${-1.570796 - epsilon}" effort="100" velocity="100"/>
+    <limit upper="0.09" lower="${-1.570796 - epsilon}" effort="100.0" velocity="100.0"/>
   </joint>
   <joint name="l3l_to_l2l" type="revolute">
@@ -543,5 +561,5 @@
     <child link="l3l_1"/>
     <axis xyz="0.0 -0.0 -1.0"/>
-    <limit upper="${1.134464 + epsilon}" lower="${-1.134464 - epsilon}" effort="100" velocity="100"/>
+    <limit upper="${1.134464 + epsilon}" lower="${-1.134464 - epsilon}" effort="100.0" velocity="100.0"/>
   </joint>
   <joint name="l4l_to_l3l" type="revolute">
@@ -550,5 +568,5 @@
     <child link="l4l_1"/>
     <axis xyz="-0.0 -1.0 0.0"/>
-    <limit upper="${2.356194 + epsilon}" lower="-1.5" effort="100" velocity="100"/>
+    <limit upper="${2.356194 + epsilon}" lower="-1.5" effort="100.0" velocity="100.0"/>
   </joint>
   <joint name="l5l_to_l4l" type="revolute">
@@ -557,5 +575,5 @@
     <child link="l5l_1"/>
     <axis xyz="0.0 -0.0 -1.0"/>
-    <limit upper="${1.047198 + epsilon}" lower="${-1.047198 -epsilon}" effort="100" velocity="100"/>
+    <limit upper="${1.047198 + epsilon}" lower="${-1.047198 -epsilon}" effort="100.0" velocity="100.0"/>
   </joint>
   <joint name="l6l_to_l5l" type="revolute">
@@ -564,5 +582,5 @@
     <child link="l6l_1"/>
     <axis xyz="0.0 1.0 0.0"/>
-    <limit upper="${1.570796 + epsilon}" lower="${-1.570796 -epsilon}" effort="100" velocity="100"/>
+    <limit upper="${1.570796 + epsilon}" lower="${-1.570796 -epsilon}" effort="100.0" velocity="100.0"/>
   </joint>
   <joint name="l2r_to_l1r" type="revolute">
@@ -571,5 +589,5 @@
     <child link="l2r_1"/>
     <axis xyz="1.0 0.0 0.0"/>
-    <limit upper="0.1" lower="${-1.570796 - 0.1}" effort="100" velocity="100"/>
+    <limit upper="0.1" lower="${-1.570796 - 0.1}" effort="100.0" velocity="100.0"/>
   </joint>
   <joint name="l3r_to_l2r" type="revolute">
@@ -578,5 +596,5 @@
     <child link="l3r_1"/>
     <axis xyz="0.0 0.0 1.0"/>
-    <limit upper="${1.134464 + epsilon}" lower="${-1.134464 -epsilon}" effort="100" velocity="100"/>
+    <limit upper="${1.134464 + epsilon}" lower="${-1.134464 -epsilon}" effort="100.0" velocity="100.0"/>
   </joint>
   <joint name="l4r_to_l3r" type="revolute">
@@ -585,5 +603,5 @@
     <child link="l4r_1"/>
     <axis xyz="-0.0 -1.0 0.0"/>
-    <limit upper="${2.356194 + epsilon}" lower="-3.14" effort="100" velocity="100"/>
+    <limit upper="${2.356194 + epsilon}" lower="-3.14" effort="100.0" velocity="100.0"/>
   </joint>
   <joint name="l5r_to_l4r" type="revolute">
@@ -592,5 +610,5 @@
     <child link="l5r_1"/>
     <axis xyz="-0.0 0.0 1.0"/>
-    <limit upper="${1.047198 + epsilon}" lower="${-1.047198 - epsilon}" effort="100" velocity="100"/>
+    <limit upper="${1.047198 + epsilon}" lower="${-1.047198 - epsilon}" effort="100.0" velocity="100.0"/>
   </joint>
   <joint name="l6r_to_l5r" type="revolute">
@@ -599,5 +617,5 @@
     <child link="l6r_1"/>
     <axis xyz="-0.0 -1.0 0.0"/>
-    <limit upper="${1.570796 + epsilon}" lower="${-1.570796 - epsilon}" effort="100" velocity="100"/>
+    <limit upper="${1.570796 + epsilon}" lower="${-1.570796 - epsilon}" effort="100.0" velocity="100.0"/>
   </joint>
   <!-- head pitch joint -->
@@ -627,5 +645,5 @@
     <child link="g2ra_1"/>
     <axis xyz="1.0 -0.0 -0.0"/>
-    <limit upper="${1.570796 + epsilon}" lower="${-epsilon}" effort="100" velocity="100"/>
+    <limit upper="${1.570796 + epsilon}" lower="${-epsilon}" effort="100.0" velocity="100.0"/>
   </joint>
   <joint name="g2rb_to_g1r" type="revolute">
@@ -634,5 +652,5 @@
     <child link="g2rb_1"/>
     <axis xyz="1.0 -0.0 -0.0"/>
-    <limit upper="${epsilon}" lower="${-1.570796 - epsilon}" effort="100" velocity="100"/>
+    <limit upper="${epsilon}" lower="${-1.570796 - epsilon}" effort="100.0" velocity="100.0"/>
   </joint>
   <!-- <joint name="g1l_to_l6l" type="fixed">
@@ -646,5 +664,5 @@
     <child link="g2lb_1"/>
     <axis xyz="-1.0 0.0 -0.0"/>
-    <limit upper="${epsilon}" lower="${-1.570796 - epsilon}" effort="100" velocity="100"/>
+    <limit upper="${epsilon}" lower="${-1.570796 - epsilon}" effort="100.0" velocity="100.0"/>
   </joint> -->
   <!-- <joint name="g2la_to_g1l" type="revolute">
@@ -653,5 +671,5 @@
     <child link="g2la_1"/>
     <axis xyz="-1.0 0.0 -0.0"/>
-    <limit upper="${1.570796 + epsilon}" lower="${-epsilon}" effort="100" velocity="100"/>
+    <limit upper="${1.570796 + epsilon}" lower="${-epsilon}" effort="100.0" velocity="100.0"/>
   </joint>
  -->
@@ -690,5 +708,5 @@
     <child link="l1r_1"/>
     <axis xyz="0.0 -1.0 0.0"/>
-    <limit upper="${2.356194 + epsilon}" lower="${-1.570796 - epsilon}" effort="100" velocity="100"/>
+    <limit upper="${2.356194 + epsilon}" lower="${-1.570796 - epsilon}" effort="100.0" velocity="100.0"/>
   </joint>
   <joint name="l1l_to_base_link" type="revolute">
@@ -697,5 +715,5 @@
     <child link="l1l_1"/>
     <axis xyz="0.0 -1.0 0.0"/>
-    <limit upper="${2.356194 + epsilon}" lower="${-1.570796 - epsilon}" effort="100" velocity="100"/>
+    <limit upper="${2.356194 + epsilon}" lower="${-1.570796 - epsilon}" effort="100.0" velocity="100.0"/>
   </joint>
   <joint name="l1h_to_base_link" type="revolute">
@@ -704,5 +722,5 @@
     <child link="l1h_1"/>
     <axis xyz="0.0 0.0 1.0"/>
-    <limit effort="50" lower="${-1.570796 - epsilon}" upper="${1.570796 + epsilon}" velocity="50"/>
+    <limit effort="50.0" lower="${-1.570796 - epsilon}" upper="${1.570796 + epsilon}" velocity="50.0"/>
   </joint>
   <link name="base_footprint"/>

File: bender_description/urdf/ros2_control.xacro (robot description, xacro)
@@ -58,6 +58,6 @@
 			<param name="baud_rate">1000000</param>
 			<param name="protocol_version">1.0</param>
-			<param name="number_of_joints">12</param>
-			<param name="number_of_transmissions">12</param>
+			<param name="number_of_joints">14</param>
+			<param name="number_of_transmissions">14</param>
 			<param name="dynamixel_model_folder">/param/dxl_model</param>
 			<param name="disable_torque_at_init">true</param>
@@ -283,5 +283,10 @@
 			<param name="Return Delay Time">25</param>
 		</gpio>
-		<!-- <gpio name="motor_g2r">
+        <joint name="gripper_base_to_movil">
+            <command_interface name="position"/>
+            <state_interface name="position"/>
+            <state_interface name="velocity"/>
+        </joint>
+        <gpio name="motor_g2r">
 			<param name="type">dxl</param>
 			<param name="ID">7</param>
@@ -295,6 +300,6 @@
 			<param name="CCW Compliance Slope">254</param>
 			<param name="Return Delay Time">25</param>
-		</gpio> -->
-		<!-- <joint name="l1h_to_base_link">
+		</gpio>
+		<joint name="l1h_to_base_link">
 			<command_interface name="position" />
 			<state_interface name="position" />
@@ -314,5 +319,5 @@
 			<param name="Return Delay Time">25</param>
 		</gpio>
-		<joint name="l2h_to_l1h">
+		<!-- <joint name="l2h_to_l1h">
 			<command_interface name="position" />
 			<state_interface name="position" />

File: bender_moveit_config/config/bender.ros2_control.xacro (robot description, xacro)
@@ -8,46 +8,4 @@
                 <plugin>mock_components/GenericSystem</plugin>
             </hardware>
-            <joint name="l1l_to_base_link">
-                <command_interface name="position"/>
-                <state_interface name="position">
-                  <param name="initial_value">${initial_positions['l1l_to_base_link']}</param>
-                </state_interface>
-                <state_interface name="velocity"/>
-            </joint>
-            <joint name="l2l_to_l1l">
-                <command_interface name="position"/>
-                <state_interface name="position">
-                  <param name="initial_value">${initial_positions['l2l_to_l1l']}</param>
-                </state_interface>
-                <state_interface name="velocity"/>
-            </joint>
-            <joint name="l3l_to_l2l">
-                <command_interface name="position"/>
-                <state_interface name="position">
-                  <param name="initial_value">${initial_positions['l3l_to_l2l']}</param>
-                </state_interface>
-                <state_interface name="velocity"/>
-            </joint>
-            <joint name="l4l_to_l3l">
-                <command_interface name="position"/>
-                <state_interface name="position">
-                  <param name="initial_value">${initial_positions['l4l_to_l3l']}</param>
-                </state_interface>
-                <state_interface name="velocity"/>
-            </joint>
-            <joint name="l5l_to_l4l">
-                <command_interface name="position"/>
-                <state_interface name="position">
-                  <param name="initial_value">${initial_positions['l5l_to_l4l']}</param>
-                </state_interface>
-                <state_interface name="velocity"/>
-            </joint>
-            <joint name="l6l_to_l5l">
-                <command_interface name="position"/>
-                <state_interface name="position">
-                  <param name="initial_value">${initial_positions['l6l_to_l5l']}</param>
-                </state_interface>
-                <state_interface name="velocity"/>
-            </joint>
             <joint name="l1r_to_base_link">
                 <command_interface name="position"/>
@@ -106,18 +64,4 @@
                 <state_interface name="velocity"/>
             </joint>
-            <joint name="g2la_to_g1l">
-                <command_interface name="position"/>
-                <state_interface name="position">
-                  <param name="initial_value">${initial_positions['g2la_to_g1l']}</param>
-                </state_interface>
-                <state_interface name="velocity"/>
-            </joint>
-            <joint name="g2lb_to_g1l">
-                <command_interface name="position"/>
-                <state_interface name="position">
-                  <param name="initial_value">${initial_positions['g2lb_to_g1l']}</param>
-                </state_interface>
-                <state_interface name="velocity"/>
-            </joint>
             <joint name="g2ra_to_g1r">
                 <command_interface name="position"/>
@@ -134,4 +78,53 @@
                 <state_interface name="velocity"/>
             </joint>
+            <joint name="l1l_to_base_link">
+                <command_interface name="position"/>
+                <state_interface name="position">
+                  <param name="initial_value">${initial_positions['l1l_to_base_link']}</param>
+                </state_interface>
+                <state_interface name="velocity"/>
+            </joint>
+            <joint name="l2l_to_l1l">
+                <command_interface name="position"/>
+                <state_interface name="position">
+                  <param name="initial_value">${initial_positions['l2l_to_l1l']}</param>
+                </state_interface>
+                <state_interface name="velocity"/>
+            </joint>
+            <joint name="l3l_to_l2l">
+                <command_interface name="position"/>
+                <state_interface name="position">
+                  <param name="initial_value">${initial_positions['l3l_to_l2l']}</param>
+                </state_interface>
+                <state_interface name="velocity"/>
+            </joint>
+            <joint name="l4l_to_l3l">
+                <command_interface name="position"/>
+                <state_interface name="position">
+                  <param name="initial_value">${initial_positions['l4l_to_l3l']}</param>
+                </state_interface>
+                <state_interface name="velocity"/>
+            </joint>
+            <joint name="l5l_to_l4l">
+                <command_interface name="position"/>
+                <state_interface name="position">
+                  <param name="initial_value">${initial_positions['l5l_to_l4l']}</param>
+                </state_interface>
+                <state_interface name="velocity"/>
+            </joint>
+            <joint name="l6l_to_l5l">
+                <command_interface name="position"/>
+                <state_interface name="position">
+                  <param name="initial_value">${initial_positions['l6l_to_l5l']}</param>
+                </state_interface>
+                <state_interface name="velocity"/>
+            </joint>
+            <joint name="gripper_base_to_movil">
+                <command_interface name="position"/>
+                <state_interface name="position">
+                  <param name="initial_value">${initial_positions['gripper_base_to_movil']}</param>
+                </state_interface>
+                <state_interface name="velocity"/>
+            </joint>
         </ros2_control>
     </xacro:macro>

File: bender_moveit_config/config/bender.urdf.xacro (robot description, xacro)
@@ -1,5 +1,9 @@
 <?xml version="1.0"?>
 <robot xmlns:xacro="http://www.ros.org/wiki/xacro" name="bender">
+    <xacro:arg name="initial_positions_file" default="initial_positions.yaml" />
     <!-- Import bender urdf file -->
     <xacro:include filename="$(find bender_description)/urdf/bender.xacro" />
+    <!-- Import control_xacro -->
+    <xacro:include filename="bender.ros2_control.xacro" />
+    <xacro:bender_ros2_control name="FakeSystem" initial_positions_file="$(arg initial_positions_file)"/>
 </robot>
