Commit message: (FG): change joint orientations

File: bender_description/urdf/bender.xacro (robot description, xacro)
@@ -553,6 +553,6 @@
     <parent link="l1l_1"/>
     <child link="l2l_1"/>
-    <axis xyz="-1.0 0.0 -0.0"/>
-    <limit upper="0.09" lower="${-1.570796 - epsilon}" effort="100.0" velocity="100.0"/>
+    <axis xyz="1.0 0.0 -0.0"/>
+    <limit upper="${1.570796 + epsilon}" lower="-0.09" effort="100.0" velocity="100.0"/>
   </joint>
   <joint name="l3l_to_l2l" type="revolute">
@@ -560,5 +560,5 @@
     <parent link="l2l_1"/>
     <child link="l3l_1"/>
-    <axis xyz="0.0 -0.0 -1.0"/>
+    <axis xyz="0.0 -0.0 1.0"/>
     <limit upper="${1.134464 + epsilon}" lower="${-1.134464 - epsilon}" effort="100.0" velocity="100.0"/>
   </joint>
@@ -595,5 +595,5 @@
     <parent link="l2r_1"/>
     <child link="l3r_1"/>
-    <axis xyz="0.0 0.0 1.0"/>
+    <axis xyz="0.0 0.0 -1.0"/>
     <limit upper="${1.134464 + epsilon}" lower="${-1.134464 -epsilon}" effort="100.0" velocity="100.0"/>
   </joint>
@@ -602,6 +602,6 @@
     <parent link="l3r_1"/>
     <child link="l4r_1"/>
-    <axis xyz="-0.0 -1.0 0.0"/>
-    <limit upper="${2.356194 + epsilon}" lower="-3.14" effort="100.0" velocity="100.0"/>
+    <axis xyz="-0.0 1.0 0.0"/>
+    <limit upper="1.5" lower="${-2.356194 - epsilon}" effort="100.0" velocity="100.0"/>
   </joint>
   <joint name="l5r_to_l4r" type="revolute">
@@ -609,5 +609,5 @@
     <parent link="l4r_1"/>
     <child link="l5r_1"/>
-    <axis xyz="-0.0 0.0 1.0"/>
+    <axis xyz="-0.0 0.0 -1.0"/>
     <limit upper="${1.047198 + epsilon}" lower="${-1.047198 - epsilon}" effort="100.0" velocity="100.0"/>
   </joint>
@@ -616,5 +616,5 @@
     <parent link="l5r_1"/>
     <child link="l6r_1"/>
-    <axis xyz="-0.0 -1.0 0.0"/>
+    <axis xyz="-0.0 1.0 0.0"/>
     <limit upper="${1.570796 + epsilon}" lower="${-1.570796 - epsilon}" effort="100.0" velocity="100.0"/>
   </joint>
@@ -654,24 +654,4 @@
     <limit upper="${epsilon}" lower="${-1.570796 - epsilon}" effort="100.0" velocity="100.0"/>
   </joint>
-  <!-- <joint name="g1l_to_l6l" type="fixed">
-    <origin xyz="0.0 -0.02225 -0.024015" rpy="0 0 0"/>
-    <parent link="l6l_1"/>
-    <child link="g1l_1"/>
-  </joint> -->
-  <!-- <joint name="g2lb_to_g1l" type="revolute">
-    <origin xyz="0.02195 0.0185 -0.0416" rpy="0 0 0"/>
-    <parent link="g1l_1"/>
-    <child link="g2lb_1"/>
-    <axis xyz="-1.0 0.0 -0.0"/>
-    <limit upper="${epsilon}" lower="${-1.570796 - epsilon}" effort="100.0" velocity="100.0"/>
-  </joint> -->
-  <!-- <joint name="g2la_to_g1l" type="revolute">
-    <origin xyz="0.02195 -0.0185 -0.0416" rpy="0 0 0"/>
-    <parent link="g1l_1"/>
-    <child link="g2la_1"/>
-    <axis xyz="-1.0 0.0 -0.0"/>
-    <limit upper="${1.570796 + epsilon}" lower="${-epsilon}" effort="100.0" velocity="100.0"/>
-  </joint>
- -->
   <joint name="laser_to_base_link" type="fixed">
     <origin xyz="0.188322 -0.007366 0.25882" rpy="0 0 0"/>

File: bender_description/urdf/ros2_control.xacro (robot description, xacro)
@@ -81,5 +81,5 @@
     		<param name="CW Compliance Slope">254</param>
     		<param name="CCW Compliance Slope">254</param>
-    		<param name="Return Delay Time">25</param>
+    		<param name="Return Delay Time">10</param>
 		</gpio>
 		<joint name="l3r_to_l2r">
@@ -100,5 +100,5 @@
 			<param name="CW Compliance Slope">254</param>
 			<param name="CCW Compliance Slope">254</param>
-			<param name="Return Delay Time">25</param>
+			<param name="Return Delay Time">10</param>
 		</gpio>
 		<joint name="l4r_to_l3r">
@@ -118,5 +118,5 @@
 			<param name="I Gain">2</param>
 			<param name="D Gain">5</param>
-			<param name="Return Delay Time">25</param>
+			<param name="Return Delay Time">10</param>
 		</gpio>
 		<joint name="l5r_to_l4r">
@@ -136,5 +136,5 @@
 			<param name="CW Compliance Slope">254</param>
 			<param name="CCW Compliance Slope">254</param>
-			<param name="Return Delay Time">25</param>
+			<param name="Return Delay Time">10</param>
 		</gpio>
 		<joint name="l6r_to_l5r">
@@ -155,5 +155,5 @@
 			<param name="CW Compliance Slope">254</param>
 			<param name="CCW Compliance Slope">254</param>
-			<param name="Return Delay Time">25</param>
+			<param name="Return Delay Time">10</param>
 		</gpio>
 		<joint name="l2l_to_l1l">
@@ -172,5 +172,5 @@
     		<param name="I Gain">2</param>
     		<param name="D Gain">5</param>
-    		<param name="Return Delay Time">25</param>
+    		<param name="Return Delay Time">10</param>
 		</gpio>
 		<joint name="l3l_to_l2l">
@@ -186,10 +186,10 @@
 			<state_interface name="Present Velocity" />
 			<state_interface name="Present Load" />
-			<param name="[unit info]">Present Position, 0.005061455, rad, unsigned, -2.566157685; Goal Position, 0.005061455, rad, unsigned, -2.566157685</param>
-			<param name="CW Compliance Margin">1</param>
-			<param name="CCW Compliance Margin">1</param>
-			<param name="CW Compliance Slope">254</param>
-			<param name="CCW Compliance Slope">254</param>
-			<param name="Return Delay Time">25</param>
+			<param name="[unit info]">Present Position, -0.005061455, rad, unsigned, 2.566157685; Goal Position, -0.005061455, rad, unsigned, 2.566157685</param>
+			<param name="CW Compliance Margin">1</param>
+			<param name="CCW Compliance Margin">1</param>
+			<param name="CW Compliance Slope">254</param>
+			<param name="CCW Compliance Slope">254</param>
+			<param name="Return Delay Time">10</param>
 		</gpio>
 		<joint name="l4l_to_l3l">
@@ -209,5 +209,5 @@
 			<param name="I Gain">2</param>
 			<param name="D Gain">5</param>
-			<param name="Return Delay Time">25</param>
+			<param name="Return Delay Time">10</param>
 		</gpio>
 		<joint name="l5l_to_l4l">
@@ -227,5 +227,5 @@
 			<param name="CW Compliance Slope">254</param>
 			<param name="CCW Compliance Slope">254</param>
-			<param name="Return Delay Time">25</param>
+			<param name="Return Delay Time">10</param>
 		</gpio>
 		<joint name="l6l_to_l5l">
@@ -245,5 +245,5 @@
 			<param name="CW Compliance Slope">254</param>
 			<param name="CCW Compliance Slope">254</param>
-			<param name="Return Delay Time">25</param>
+			<param name="Return Delay Time">10</param>
 		</gpio>
 		<joint name="g2ra_to_g1r">
@@ -263,5 +263,5 @@
 			<param name="CW Compliance Slope">254</param>
 			<param name="CCW Compliance Slope">254</param>
-			<param name="Return Delay Time">25</param>
+			<param name="Return Delay Time">10</param>
 		</gpio>
 		<joint name="g2rb_to_g1r">
@@ -281,5 +281,5 @@
 			<param name="CW Compliance Slope">254</param>
 			<param name="CCW Compliance Slope">254</param>
-			<param name="Return Delay Time">25</param>
+			<param name="Return Delay Time">10</param>
 		</gpio>
         <joint name="gripper_base_to_movil">
@@ -299,5 +299,5 @@
 			<param name="CW Compliance Slope">254</param>
 			<param name="CCW Compliance Slope">254</param>
-			<param name="Return Delay Time">25</param>
+			<param name="Return Delay Time">10</param>
 		</gpio>
 		<joint name="l1h_to_base_link">
@@ -317,5 +317,5 @@
 			<param name="CW Compliance Slope">254</param>
 			<param name="CCW Compliance Slope">254</param>
-			<param name="Return Delay Time">25</param>
+			<param name="Return Delay Time">10</param>
 		</gpio>
 		<!-- <joint name="l2h_to_l1h">
@@ -335,5 +335,5 @@
 			<param name="CW Compliance Slope">254</param>
 			<param name="CCW Compliance Slope">254</param>
-			<param name="Return Delay Time">25</param>
+			<param name="Return Delay Time">10</param>
 		</gpio>
 		<gpio name="motor_l2h_2">

Commit message: (FG): pid controller for shoulder joint

File: bender_description/urdf/bender.xacro (robot description, xacro)
@@ -370,8 +370,8 @@
         <joint name="gripper_base_to_movil" type="revolute">
           <axis xyz="0 1 0"/>
-          <origin rpy="0 -1.0 0" xyz="-0.01869 0 -0.01945"/>
+          <origin rpy="0 0 0" xyz="-0.01869 0 -0.01945"/>
           <parent link="gripper_l_base"/>
           <child link="movil"/>
-          <limit effort="1000.0" lower="0.0" upper="0.5" velocity="0.5"/>
+          <limit effort="1000.0" lower="-2.0" upper="0.3495" velocity="0.5"/>
         </joint>
         <link name="movil">
@@ -620,5 +620,5 @@
   </joint>
   <!-- head pitch joint -->
-  <joint name="l2h_to_l1h" type="revolute">
+  <joint name="l2h_to_l1h" type="fixed">
     <origin rpy="0 0 0" xyz="0.0 -0.03 0.07"/>
     <parent link="l1h_1"/>
@@ -641,17 +641,19 @@
   </joint>
   <joint name="g2ra_to_g1r" type="revolute">
-    <origin xyz="0.02195 0.0185 -0.0416" rpy="0 0 0"/>
-    <parent link="g1r_1"/>
-    <child link="g2ra_1"/>
-    <axis xyz="1.0 -0.0 -0.0"/>
-    <limit upper="${1.570796 + epsilon}" lower="${-epsilon}" effort="100.0" velocity="100.0"/>
-  </joint>
-  <joint name="g2rb_to_g1r" type="revolute">
-    <origin xyz="0.02195 -0.0185 -0.0416" rpy="0 0 0"/>
-    <parent link="g1r_1"/>
-    <child link="g2rb_1"/>
-    <axis xyz="1.0 -0.0 -0.0"/>
-    <limit upper="${epsilon}" lower="${-1.570796 - epsilon}" effort="100.0" velocity="100.0"/>
-  </joint>
+      <origin xyz="0.02195 0.0185 -0.0416" rpy="0 0 0"/>
+      <parent link="g1r_1"/>
+      <child link="g2ra_1"/>
+      <axis xyz="1.0 -0.0 -0.0"/>
+      <limit upper="${1.570796 + epsilon}" lower="${-epsilon}" effort="100.0" velocity="100.0"/>
+    </joint>
+    <joint name="g2rb_to_g1r" type="revolute">
+      <origin xyz="0.02195 -0.0185 -0.0416" rpy="0 0 0"/>
+      <parent link="g1r_1"/>
+      <child link="g2rb_1"/>
+      <axis xyz="1.0 -0.0 -0.0"/>
+      <limit upper="${epsilon}" lower="${-1.570796 - epsilon}" effort="100.0" velocity="100.0"/>
+      <!-- Agregamos la etiqueta mimic aquí -->
+      <mimic joint="g2ra_to_g1r" multiplier="-1.0" offset="0.0"/>
+    </joint>
   <joint name="laser_to_base_link" type="fixed">
     <origin xyz="0.188322 -0.007366 0.25882" rpy="0 0 0"/>
@@ -659,5 +661,5 @@
     <child link="laser_1"/>
   </joint>
-  <joint name="wfr_to_base_link" type="continuous">
+  <joint name="wfr_to_base_link" type="fixed">
     <origin rpy="0 0 0" xyz="0.135487 -0.164865 0.09982"/>
     <parent link="base_link"/>
@@ -665,5 +667,5 @@
     <axis xyz="0 1 0"/>
   </joint>
-  <joint name="wrr_to_base_link" type="continuous">
+  <joint name="wrr_to_base_link" type="fixed">
     <origin rpy="0 0 0" xyz="-0.114513 -0.164865 0.09982"/>
     <parent link="base_link"/>
@@ -671,5 +673,5 @@
     <axis xyz="0 1 0"/>
   </joint>
-  <joint name="wfl_to_base_link" type="continuous">
+  <joint name="wfl_to_base_link" type="fixed">
     <origin rpy="0 0 0" xyz="0.135487 0.150135 0.09982"/>
     <parent link="base_link"/>
@@ -677,5 +679,5 @@
     <axis xyz="0 1 0"/>
   </joint>
-  <joint name="wrl_to_base_link" type="continuous">
+  <joint name="wrl_to_base_link" type="fixed">
     <origin rpy="0 0 0" xyz="-0.114513 0.150135 0.09982"/>
     <parent link="base_link"/>

File: bender_description/urdf/ros2_control.xacro (robot description, xacro)
@@ -16,5 +16,5 @@
 				<param name="watchdog_timeout">1.0</param>
 				<param name="gear_ratio">${gear_ratio}</param>
-				<command_interface name="position" />
+				<!-- <command_interface name="position" /> -->
 				<command_interface name="velocity" />
 				<command_interface name="effort" />
@@ -266,5 +266,4 @@
 		</gpio>
 		<joint name="g2rb_to_g1r">
-			<command_interface name="position" />
 			<state_interface name="position" />
 			<state_interface name="velocity" />
@@ -289,16 +288,17 @@
         </joint>
         <gpio name="motor_g2r">
-			<param name="type">dxl</param>
-			<param name="ID">7</param>
-			<command_interface name="Goal Position" />
-			<state_interface name="Present Position" />
-			<state_interface name="Present Velocity" />
-			<state_interface name="Present Load" />
-			<param name="CW Compliance Margin">1</param>
-			<param name="CCW Compliance Margin">1</param>
-			<param name="CW Compliance Slope">254</param>
-			<param name="CCW Compliance Slope">254</param>
-			<param name="Return Delay Time">10</param>
-		</gpio>
+            <param name="type">dxl</param>
+            <param name="ID">7</param>
+            <command_interface name="Goal Position" />
+            <state_interface name="Present Position" />
+            <state_interface name="Present Velocity" />
+            <state_interface name="Present Load" />
+            <param name="[unit info]">Present Position, 0.005061455, rad, unsigned, -3.335673; Goal Position, 0.005061455, rad, unsigned, -3.335673</param>
+            <param name="CW Compliance Margin">1</param>
+            <param name="CCW Compliance Margin">1</param>
+            <param name="CW Compliance Slope">254</param>
+            <param name="CCW Compliance Slope">254</param>
+            <param name="Return Delay Time">10</param>
+        </gpio>
 		<joint name="l1h_to_base_link">
 			<command_interface name="position" />

Commit message: (FG): add head interface

File: bender_description/urdf/bender.xacro (robot description, xacro)
@@ -549,4 +549,11 @@
     </collision>
   </link>
+  <link name="l3h_1">
+    <inertial>
+      <origin xyz="0.0 0.0 0.0" rpy="0 0 0"/>
+      <mass value="0.001"/>
+      <inertia ixx="0.0001" iyy="0.0001" izz="0.0001" ixy="0.0" iyz="0.0" ixz="0.0"/>
+    </inertial>
+  </link>
   <joint name="l2l_to_l1l" type="revolute">
     <origin xyz="0.02775 0.0345 -0.018" rpy="0 0 0"/>
@@ -627,12 +634,11 @@
     <limit effort="50" lower="${-0.706858 - epsilon}" upper="${0.706858 + epsilon}" velocity="50"/>
   </joint>
-  <!-- head roll joint -->
-  <!-- <joint name="l3h_to_l2h" type="revolute">
+  <joint name="l3h_to_l1h" type="revolute">
     <origin rpy="0 0 0" xyz="0.0 -0.03 0.07"/>
-    <parent link="l2h_1"/>
+    <parent link="l1h_1"/>
     <child link="l3h_1"/>
-    <axis xyz="-0.0 -1.0 0.0"/>
+    <axis xyz="1.0 0.0 0.0"/>
     <limit effort="50" lower="${-0.706858 - epsilon}" upper="${0.706858 + epsilon}" velocity="50"/>
-  </joint> -->
+  </joint>
   <joint name="g1r_to_l6r" type="fixed">
     <origin xyz="0.0 0.02225 -0.024015" rpy="0 0 0"/>

File: bender_description/urdf/ros2_control.xacro (robot description, xacro)
@@ -53,15 +53,51 @@
 	</ros2_control>
 	<ros2_control name="DynamixelChainMain" type="system">
-		<hardware>
-			<plugin>dynamixel_hardware_interface/DynamixelHardware</plugin>
-			<param name="port_name">/dev/dynamixel</param>
-			<param name="baud_rate">1000000</param>
-			<param name="protocol_version">1.0</param>
-			<param name="number_of_joints">14</param>
-			<param name="number_of_transmissions">14</param>
-			<param name="dynamixel_model_folder">/param/dxl_model</param>
-			<param name="disable_torque_at_init">true</param>
-			<param name="torque_enable">0</param>
-		</hardware>
+        <hardware>
+            <plugin>dynamixel_hardware_interface/DynamixelHardware</plugin>
+            <param name="port_name">/dev/dynamixel</param>
+            <param name="baud_rate">1000000</param>
+            <param name="protocol_version">1.0</param>
+            <param name="number_of_joints">16</param>
+            <param name="number_of_transmissions">16</param>
+            <param name="dynamixel_model_folder">/param/dxl_model</param>
+            <param name="disable_torque_at_init">true</param>
+            <param name="torque_enable">0</param>
+            <param name="transmission_to_joint_matrix">
+                1, 0, 0, 0, 0, 0, 0, 0, 0, 0, 0, 0, 0, 0, 0, 0,
+                0, 1, 0, 0, 0, 0, 0, 0, 0, 0, 0, 0, 0, 0, 0, 0,
+                0, 0, 1, 0, 0, 0, 0, 0, 0, 0, 0, 0, 0, 0, 0, 0,
+                0, 0, 0, 1, 0, 0, 0, 0, 0, 0, 0, 0, 0, 0, 0, 0,
+                0, 0, 0, 0, 1, 0, 0, 0, 0, 0, 0, 0, 0, 0, 0, 0,
+                0, 0, 0, 0, 0, 1, 0, 0, 0, 0, 0, 0, 0, 0, 0, 0,
+                0, 0, 0, 0, 0, 0, 1, 0, 0, 0, 0, 0, 0, 0, 0, 0,
+                0, 0, 0, 0, 0, 0, 0, 1, 0, 0, 0, 0, 0, 0, 0, 0,
+                0, 0, 0, 0, 0, 0, 0, 0, 1, 0, 0, 0, 0, 0, 0, 0,
+                0, 0, 0, 0, 0, 0, 0, 0, 0, 1, 0, 0, 0, 0, 0, 0,
+                0, 0, 0, 0, 0, 0, 0, 0, 0, 0, 1, 0, 0, 0, 0, 0,
+                0, 0, 0, 0, 0, 0, 0, 0, 0, 0, 0, 1, 0, 0, 0, 0,
+                0, 0, 0, 0, 0, 0, 0, 0, 0, 0, 0, 0, 1, 0, 0, 0,
+                0, 0, 0, 0, 0, 0, 0, 0, 0, 0, 0, 0, 0, 1, 0, 0,
+                0, 0, 0, 0, 0, 0, 0, 0, 0, 0, 0, 0, 0, 0, 0.5, 0.5,
+                0, 0, 0, 0, 0, 0, 0, 0, 0, 0, 0, 0, 0, 0, -0.5, 0.5
+            </param>
+            <param name="joint_to_transmission_matrix">
+                1, 0, 0, 0, 0, 0, 0, 0, 0, 0, 0, 0, 0, 0, 0, 0,
+                0, 1, 0, 0, 0, 0, 0, 0, 0, 0, 0, 0, 0, 0, 0, 0,
+                0, 0, 1, 0, 0, 0, 0, 0, 0, 0, 0, 0, 0, 0, 0, 0,
+                0, 0, 0, 1, 0, 0, 0, 0, 0, 0, 0, 0, 0, 0, 0, 0,
+                0, 0, 0, 0, 1, 0, 0, 0, 0, 0, 0, 0, 0, 0, 0, 0,
+                0, 0, 0, 0, 0, 1, 0, 0, 0, 0, 0, 0, 0, 0, 0, 0,
+                0, 0, 0, 0, 0, 0, 1, 0, 0, 0, 0, 0, 0, 0, 0, 0,
+                0, 0, 0, 0, 0, 0, 0, 1, 0, 0, 0, 0, 0, 0, 0, 0,
+                0, 0, 0, 0, 0, 0, 0, 0, 1, 0, 0, 0, 0, 0, 0, 0,
+                0, 0, 0, 0, 0, 0, 0, 0, 0, 1, 0, 0, 0, 0, 0, 0,
+                0, 0, 0, 0, 0, 0, 0, 0, 0, 0, 1, 0, 0, 0, 0, 0,
+                0, 0, 0, 0, 0, 0, 0, 0, 0, 0, 0, 1, 0, 0, 0, 0,
+                0, 0, 0, 0, 0, 0, 0, 0, 0, 0, 0, 0, 1, 0, 0, 0,
+                0, 0, 0, 0, 0, 0, 0, 0, 0, 0, 0, 0, 0, 1, 0, 0,
+                0, 0, 0, 0, 0, 0, 0, 0, 0, 0, 0, 0, 0, 0, 1, -1,
+                0, 0, 0, 0, 0, 0, 0, 0, 0, 0, 0, 0, 0, 0, 1, 1
+            </param>
+        </hardware>
 		<joint name="l2r_to_l1r">
 			<command_interface name="position" />
@@ -319,5 +355,10 @@
 			<param name="Return Delay Time">25</param>
 		</gpio>
-		<!-- <joint name="l2h_to_l1h">
+		<joint name="l2h_to_l1h">
+			<command_interface name="position" />
+			<state_interface name="position" />
+			<state_interface name="velocity" />
+		</joint>
+		<joint name="l3h_to_l1h">
 			<command_interface name="position" />
 			<state_interface name="position" />
@@ -349,5 +390,5 @@
 			<param name="CCW Compliance Slope">254</param>
 			<param name="Return Delay Time">100</param>
-		</gpio> -->
+		</gpio>
 	</ros2_control>
 </robot>

Commit message: (FG): change gripper and head movement

File: bender_description/urdf/bender.xacro (robot description, xacro)
@@ -627,5 +627,5 @@
   </joint>
   <!-- head pitch joint -->
-  <joint name="l2h_to_l1h" type="fixed">
+  <joint name="l2h_to_l1h" type="revolute">
     <origin rpy="0 0 0" xyz="0.0 -0.03 0.07"/>
     <parent link="l1h_1"/>

File: bender_description/urdf/ros2_control.xacro (robot description, xacro)
@@ -74,6 +74,6 @@
                 0, 0, 0, 0, 0, 0, 0, 0, 1, 0, 0, 0, 0, 0, 0, 0,
                 0, 0, 0, 0, 0, 0, 0, 0, 0, 1, 0, 0, 0, 0, 0, 0,
-                0, 0, 0, 0, 0, 0, 0, 0, 0, 0, 1, 0, 0, 0, 0, 0,
-                0, 0, 0, 0, 0, 0, 0, 0, 0, 0, 0, 1, 0, 0, 0, 0,
+                0, 0, 0, 0, 0, 0, 0, 0, 0, 0, 0.5, -0.5, 0, 0, 0, 0,
+                0, 0, 0, 0, 0, 0, 0, 0, 0, 0, 0.5, 0.5, 0, 0, 0, 0,
                 0, 0, 0, 0, 0, 0, 0, 0, 0, 0, 0, 0, 1, 0, 0, 0,
                 0, 0, 0, 0, 0, 0, 0, 0, 0, 0, 0, 0, 0, 1, 0, 0,
@@ -92,6 +92,6 @@
                 0, 0, 0, 0, 0, 0, 0, 0, 1, 0, 0, 0, 0, 0, 0, 0,
                 0, 0, 0, 0, 0, 0, 0, 0, 0, 1, 0, 0, 0, 0, 0, 0,
-                0, 0, 0, 0, 0, 0, 0, 0, 0, 0, 1, 0, 0, 0, 0, 0,
-                0, 0, 0, 0, 0, 0, 0, 0, 0, 0, 0, 1, 0, 0, 0, 0,
+                0, 0, 0, 0, 0, 0, 0, 0, 0, 0, 1, 1, 0, 0, 0, 0,
+                0, 0, 0, 0, 0, 0, 0, 0, 0, 0, -1, 1, 0, 0, 0, 0,
                 0, 0, 0, 0, 0, 0, 0, 0, 0, 0, 0, 0, 1, 0, 0, 0,
                 0, 0, 0, 0, 0, 0, 0, 0, 0, 0, 0, 0, 0, 1, 0, 0,
@@ -288,4 +288,8 @@
 			<state_interface name="velocity" />
 		</joint>
+		<joint name="g2rb_to_g1r">
+            <state_interface name="position" />
+            <state_interface name="velocity" />
+        </joint>
 		<gpio name="motor_g2ra">
 			<param name="type">dxl</param>
@@ -301,8 +305,4 @@
 			<param name="Return Delay Time">10</param>
 		</gpio>
-		<joint name="g2rb_to_g1r">
-			<state_interface name="position" />
-			<state_interface name="velocity" />
-		</joint>
 		<gpio name="motor_g2rb">
 			<param name="type">dxl</param>
@@ -349,4 +349,5 @@
 			<state_interface name="Present Velocity" />
 			<state_interface name="Present Load" />
+			<param name="[unit info]">Present Position, 0.005061455, rad, unsigned, -3.22920829; Goal Position, 0.005061455, rad, unsigned, -3.22920829</param>
 			<param name="CW Compliance Margin">1</param>
 			<param name="CCW Compliance Margin">1</param>
@@ -372,4 +373,5 @@
 			<state_interface name="Present Velocity" />
 			<state_interface name="Present Load" />
+			<param name="[unit info]">Present Position, 0.005061455, rad, unsigned, -1.047721185; Goal Position, 0.005061455, rad, unsigned, -1.047721185</param>
 			<param name="CW Compliance Margin">1</param>
 			<param name="CCW Compliance Margin">1</param>
@@ -385,4 +387,5 @@
 			<state_interface name="Present Velocity" />
 			<state_interface name="Present Load" />
+			<param name="[unit info]">Present Position, 0.005061455, rad, unsigned, -3.993487995; Goal Position, 0.005061455, rad, unsigned, -3.993487995</param>
 			<param name="CW Compliance Margin">1</param>
 			<param name="CCW Compliance Margin">1</param>
