Commit message: (FG): add pioneer hardware interface

File: bender_description/urdf/bender.xacro (robot description, xacro)
@@ -667,11 +667,12 @@
     <child link="laser_1"/>
   </joint>
-  <joint name="wfr_to_base_link" type="fixed">
+  <joint name="wfr_to_base_link" type="continuous">
     <origin rpy="0 0 0" xyz="0.135487 -0.164865 0.09982"/>
     <parent link="base_link"/>
     <child link="wfr_1"/>
     <axis xyz="0 1 0"/>
-  </joint>
-  <joint name="wrr_to_base_link" type="fixed">
+    <mimic joint="wrr_to_base_link" multiplier="1.0" offset="0.0"/>
+  </joint>
+  <joint name="wrr_to_base_link" type="continuous">
     <origin rpy="0 0 0" xyz="-0.114513 -0.164865 0.09982"/>
     <parent link="base_link"/>
@@ -679,11 +680,12 @@
     <axis xyz="0 1 0"/>
   </joint>
-  <joint name="wfl_to_base_link" type="fixed">
+  <joint name="wfl_to_base_link" type="continuous">
     <origin rpy="0 0 0" xyz="0.135487 0.150135 0.09982"/>
     <parent link="base_link"/>
     <child link="wfl_1"/>
     <axis xyz="0 1 0"/>
-  </joint>
-  <joint name="wrl_to_base_link" type="fixed">
+    <mimic joint="wrl_to_base_link" multiplier="1.0" offset="0.0"/>
+  </joint>
+  <joint name="wrl_to_base_link" type="continuous">
     <origin rpy="0 0 0" xyz="-0.114513 0.150135 0.09982"/>
     <parent link="base_link"/>

File: bender_description/urdf/ros2_control.xacro (robot description, xacro)
@@ -2,5 +2,5 @@
 <robot
 	xmlns:xacro="http://www.ros.org/wiki/xacro">
-<xacro:macro name="odrive_ros2_control" params="name serial_number joint_name axis:=0 gear_ratio:=1.0">
+    <xacro:macro name="odrive_ros2_control" params="name serial_number joint_name axis:=0 gear_ratio:=1.0">
 		<ros2_control name="${name}" type="system">
 			<hardware>
@@ -24,16 +24,16 @@
 	</xacro:macro>
 	<xacro:odrive_ros2_control
-    name="OdriveLeft"
-    serial_number="3690387D3333"
-    joint_name="l1l_to_base_link"
-    axis="0"
-	gear_ratio="250"
+        name="OdriveLeft"
+        serial_number="3690387D3333"
+        joint_name="l1l_to_base_link"
+        axis="0"
+    	gear_ratio="250"
 	/>
 	<xacro:odrive_ros2_control
-    name="OdriveRight"
-    serial_number="336B33573235"
-    joint_name="l1r_to_base_link"
-    axis="0"
-	gear_ratio="250"
+        name="OdriveRight"
+        serial_number="336B33573235"
+        joint_name="l1r_to_base_link"
+        axis="0"
+    	gear_ratio="250"
 	/>
 	<ros2_control name="ShoulderJoint" type="sensor">
@@ -395,3 +395,33 @@
 		</gpio>
 	</ros2_control>
+	<ros2_control name="Pioneer" type="system">
+    	<hardware>
+            <plugin>mock_components/GenericSystem</plugin>
+            <param name="calculate_dynamics">false</param>
+            <param name="custom_interface_with_following_offset"></param>
+            <param name="disable_commands">false</param>
+            <param name="mock_gpio_commands">false</param>
+            <param name="mock_sensor_commands">false</param>
+            <param name="position_state_following_offset">0.0</param>
+        </hardware>
+        <joint name="joint1">
+            <command_interface name="position"/>
+            <command_interface name="velocity"/>
+            <state_interface name="position">
+            <param name="initial_value">3.45</param>
+            </state_interface>
+            <state_interface name="velocity"/>
+            <state_interface name="acceleration"/>
+        </joint>
+        <joint name="joint2">
+            <command_interface name="velocity"/>
+            <command_interface name="acceleration"/>
+            <state_interface name="position">
+            <param name="initial_value">2.78</param>
+            </state_interface>
+            <state_interface name="position"/>
+            <state_interface name="velocity"/>
+            <state_interface name="acceleration"/>
+        </joint>
+	</ros2_control>
 </robot>

Commit message: (LC): add tcp

File: bender_description/urdf/bender.xacro (robot description, xacro)
@@ -662,4 +662,10 @@
       <mimic joint="g2ra_to_g1r" multiplier="-1.0" offset="0.0"/>
     </joint>
+    <link name="TCP"/>
+    <joint name="g1r_to_TCP" type="fixed">
+      <origin xyz="0.0 0.0 -0.12" rpy="0 0 0"/>
+      <parent link="g1r_1"/>
+      <child link="TCP"/>
+    </joint>
   <joint name="laser_to_base_link" type="fixed">
     <origin xyz="0.188322 -0.007366 0.25882" rpy="0 0 0"/>

Commit message: add changes (WIP)

File: bender_description/urdf/bender.xacro (robot description, xacro)
@@ -9,5 +9,5 @@
       camera_name="camera"
       parent='l2h_1'
-      xyz_offset="0.0435 0.03 0.160"
+      xyz_offset="0.0435 0.03 0.180"
       rpy_offset="0 0 0"/>
   <link name="base_link">

File: bender_description/urdf/ros2_control.xacro (robot description, xacro)
@@ -2,5 +2,5 @@
 <robot
 	xmlns:xacro="http://www.ros.org/wiki/xacro">
-<xacro:macro name="odrive_ros2_control" params="name serial_number joint_name axis:=0 gear_ratio:=1.0">
+<xacro:macro name="odrive_ros2_control" params="name serial_number joint_name_left joint_name_right axis_left axis_right gear_ratio_left gear_ratio_right">
 		<ros2_control name="${name}" type="system">
 			<hardware>
@@ -37,6 +37,6 @@
     joint_name_left="l1l_to_base_link"
     joint_name_right="l1r_to_base_link"
-    axis_left="0"
-    axis_right="1"
+    axis_left="1"
+    axis_right="0"
 	gear_ratio_left="250"
 	gear_ratio_right="250"

Commit message: (FG): tf modification

File: bender_description/urdf/bender.xacro (robot description, xacro)
@@ -10,5 +10,5 @@
       parent='l2h_1'
       xyz_offset="0.0435 0.03 0.180"
-      rpy_offset="0 0 0"/>
+      rpy_offset="0 0.2 0"/>
   <link name="base_link">
     <visual>
@@ -631,5 +631,5 @@
     <parent link="l1h_1"/>
     <child link="l2h_1"/>
-    <axis xyz="-0.0 -1.0 0.0"/>
+    <axis xyz="-0.0 1.0 0.0"/>
     <limit effort="50" lower="${-0.706858 - epsilon}" upper="${0.706858 + epsilon}" velocity="50"/>
   </joint>

File: bender_description/urdf/ros2_control.xacro (robot description, xacro)
@@ -83,6 +83,6 @@
                 0, 0, 0, 0, 0, 0, 0, 0, 0, 0, 0, 0, 1, 0, 0, 0,
                 0, 0, 0, 0, 0, 0, 0, 0, 0, 0, 0, 0, 0, 1, 0, 0,
-                0, 0, 0, 0, 0, 0, 0, 0, 0, 0, 0, 0, 0, 0, 0.5, 0.5,
-                0, 0, 0, 0, 0, 0, 0, 0, 0, 0, 0, 0, 0, 0, -0.5, 0.5
+                0, 0, 0, 0, 0, 0, 0, 0, 0, 0, 0, 0, 0, 0, 0.5, -0.5,
+                0, 0, 0, 0, 0, 0, 0, 0, 0, 0, 0, 0, 0, 0, 0.5, 0.5
             </param>
             <param name="joint_to_transmission_matrix">
@@ -101,6 +101,6 @@
                 0, 0, 0, 0, 0, 0, 0, 0, 0, 0, 0, 0, 1, 0, 0, 0,
                 0, 0, 0, 0, 0, 0, 0, 0, 0, 0, 0, 0, 0, 1, 0, 0,
-                0, 0, 0, 0, 0, 0, 0, 0, 0, 0, 0, 0, 0, 0, 1, -1,
-                0, 0, 0, 0, 0, 0, 0, 0, 0, 0, 0, 0, 0, 0, 1, 1
+                0, 0, 0, 0, 0, 0, 0, 0, 0, 0, 0, 0, 0, 0, 1, 1,
+                0, 0, 0, 0, 0, 0, 0, 0, 0, 0, 0, 0, 0, 0, -1, 1
             </param>
         </hardware>
@@ -120,6 +120,6 @@
     		<param name="CW Compliance Margin">1</param>
     		<param name="CCW Compliance Margin">1</param>
-    		<param name="CW Compliance Slope">32</param>
-    		<param name="CCW Compliance Slope">32</param>
+    		<param name="CW Compliance Slope">254</param>
+    		<param name="CCW Compliance Slope">254</param>
     		<param name="Return Delay Time">10</param>
 		</gpio>
@@ -139,6 +139,6 @@
 			<param name="CW Compliance Margin">1</param>
 			<param name="CCW Compliance Margin">1</param>
-			<param name="CW Compliance Slope">32</param>
-			<param name="CCW Compliance Slope">32</param>
+			<param name="CW Compliance Slope">254</param>
+			<param name="CCW Compliance Slope">254</param>
 			<param name="Return Delay Time">10</param>
 		</gpio>
@@ -176,5 +176,5 @@
 			<param name="CCW Compliance Margin">1</param>
 			<param name="CW Compliance Slope">254</param>
-			<param name="CCW Compliance Slope">32</param>
+			<param name="CCW Compliance Slope">254</param>
 			<param name="Return Delay Time">10</param>
 		</gpio>
@@ -194,6 +194,6 @@
 			<param name="CW Compliance Margin">1</param>
 			<param name="CCW Compliance Margin">1</param>
-			<param name="CW Compliance Slope">32</param>
-			<param name="CCW Compliance Slope">32</param>
+			<param name="CW Compliance Slope">254</param>
+			<param name="CCW Compliance Slope">254</param>
 			<param name="Return Delay Time">10</param>
 		</gpio>
@@ -230,6 +230,6 @@
 			<param name="CW Compliance Margin">1</param>
 			<param name="CCW Compliance Margin">1</param>
-			<param name="CW Compliance Slope">32</param>
-			<param name="CCW Compliance Slope">32</param>
+			<param name="CW Compliance Slope">254</param>
+			<param name="CCW Compliance Slope">254</param>
 			<param name="Return Delay Time">10</param>
 		</gpio>
@@ -266,6 +266,6 @@
 			<param name="CW Compliance Margin">1</param>
 			<param name="CCW Compliance Margin">1</param>
-			<param name="CW Compliance Slope">32</param>
-			<param name="CCW Compliance Slope">32</param>
+			<param name="CW Compliance Slope">254</param>
+			<param name="CCW Compliance Slope">254</param>
 			<param name="Return Delay Time">10</param>
 		</gpio>
@@ -284,6 +284,6 @@
 			<param name="CW Compliance Margin">1</param>
 			<param name="CCW Compliance Margin">1</param>
-			<param name="CW Compliance Slope">32</param>
-			<param name="CCW Compliance Slope">32</param>
+			<param name="CW Compliance Slope">254</param>
+			<param name="CCW Compliance Slope">254</param>
 			<param name="Return Delay Time">10</param>
 		</gpio>
@@ -306,6 +306,6 @@
 			<param name="CW Compliance Margin">1</param>
 			<param name="CCW Compliance Margin">1</param>
-			<param name="CW Compliance Slope">32</param>
-			<param name="CCW Compliance Slope">32</param>
+			<param name="CW Compliance Slope">254</param>
+			<param name="CCW Compliance Slope">254</param>
 			<param name="Return Delay Time">10</param>
 		</gpio>
@@ -319,6 +319,6 @@
 			<param name="CW Compliance Margin">1</param>
 			<param name="CCW Compliance Margin">1</param>
-			<param name="CW Compliance Slope">32</param>
-			<param name="CCW Compliance Slope">32</param>
+			<param name="CW Compliance Slope">254</param>
+			<param name="CCW Compliance Slope">254</param>
 			<param name="Return Delay Time">10</param>
 		</gpio>
@@ -338,6 +338,6 @@
             <param name="CW Compliance Margin">1</param>
             <param name="CCW Compliance Margin">1</param>
-            <param name="CW Compliance Slope">32</param>
-            <param name="CCW Compliance Slope">32</param>
+            <param name="CW Compliance Slope">254</param>
+            <param name="CCW Compliance Slope">254</param>
             <param name="Return Delay Time">10</param>
         </gpio>
@@ -357,6 +357,6 @@
 			<param name="CW Compliance Margin">1</param>
 			<param name="CCW Compliance Margin">1</param>
-			<param name="CW Compliance Slope">32</param>
-			<param name="CCW Compliance Slope">32</param>
+			<param name="CW Compliance Slope">254</param>
+			<param name="CCW Compliance Slope">254</param>
 			<param name="Return Delay Time">10</param>
 		</gpio>
@@ -378,9 +378,9 @@
 			<state_interface name="Present Velocity" />
 			<state_interface name="Present Load" />
-			<param name="[unit info]">Present Position, 0.005061455, rad, unsigned, -1.047721185; Goal Position, 0.005061455, rad, unsigned, -1.047721185</param>
-			<param name="CW Compliance Margin">1</param>
-			<param name="CCW Compliance Margin">1</param>
-			<param name="CW Compliance Slope">32</param>
-			<param name="CCW Compliance Slope">32</param>
+			<param name="[unit info]">Present Position, 0.005061455, rad, unsigned, -1.012291; Goal Position, 0.005061455, rad, unsigned, -1.012291</param>
+			<param name="CW Compliance Margin">1</param>
+			<param name="CCW Compliance Margin">1</param>
+			<param name="CW Compliance Slope">254</param>
+			<param name="CCW Compliance Slope">254</param>
 			<param name="Return Delay Time">10</param>
 		</gpio>
@@ -392,9 +392,9 @@
 			<state_interface name="Present Velocity" />
 			<state_interface name="Present Load" />
-			<param name="[unit info]">Present Position, 0.005061455, rad, unsigned, -3.993487995; Goal Position, 0.005061455, rad, unsigned, -3.993487995</param>
-			<param name="CW Compliance Margin">1</param>
-			<param name="CCW Compliance Margin">1</param>
-			<param name="CW Compliance Slope">32</param>
-			<param name="CCW Compliance Slope">32</param>
+			<param name="[unit info]">Present Position, 0.005061455, rad, unsigned, -3.912504715; Goal Position, 0.005061455, rad, unsigned, -3.912504715</param>
+			<param name="CW Compliance Margin">1</param>
+			<param name="CCW Compliance Margin">1</param>
+			<param name="CW Compliance Slope">254</param>
+			<param name="CCW Compliance Slope">254</param>
 			<param name="Return Delay Time">100</param>
 		</gpio>

File: bender_moveit_config/config/bender.ros2_control.xacro (robot description, xacro)
@@ -64,15 +64,15 @@
                 <state_interface name="velocity"/>
             </joint>
+            <joint name="l3h_to_l1h">
+                <command_interface name="position"/>
+                <state_interface name="position">
+                  <param name="initial_value">${initial_positions['l3h_to_l1h']}</param>
+                </state_interface>
+                <state_interface name="velocity"/>
+            </joint>
             <joint name="g2ra_to_g1r">
                 <command_interface name="position"/>
                 <state_interface name="position">
                   <param name="initial_value">${initial_positions['g2ra_to_g1r']}</param>
-                </state_interface>
-                <state_interface name="velocity"/>
-            </joint>
-            <joint name="g2rb_to_g1r">
-                <command_interface name="position"/>
-                <state_interface name="position">
-                  <param name="initial_value">${initial_positions['g2rb_to_g1r']}</param>
                 </state_interface>
                 <state_interface name="velocity"/>

Commit message: manipulation WIP

File: bender_description/urdf/bender.xacro (robot description, xacro)
@@ -664,5 +664,5 @@
     <link name="TCP"/>
     <joint name="g1r_to_TCP" type="fixed">
-      <origin xyz="0.0 0.0 -0.12" rpy="0 0 0"/>
+      <origin xyz="0.0 0.0 -0.12" rpy="3.14159 0 1.5707963"/>
       <parent link="g1r_1"/>
       <child link="TCP"/>

File: bender_description/urdf/ros2_control.xacro (robot description, xacro)
@@ -139,6 +139,6 @@
 			<param name="CW Compliance Margin">1</param>
 			<param name="CCW Compliance Margin">1</param>
-			<param name="CW Compliance Slope">254</param>
-			<param name="CCW Compliance Slope">254</param>
+			<param name="CW Compliance Slope">128</param>
+			<param name="CCW Compliance Slope">128</param>
 			<param name="Return Delay Time">10</param>
 		</gpio>
@@ -175,6 +175,6 @@
 			<param name="CW Compliance Margin">1</param>
 			<param name="CCW Compliance Margin">1</param>
-			<param name="CW Compliance Slope">254</param>
-			<param name="CCW Compliance Slope">254</param>
+			<param name="CW Compliance Slope">128</param>
+			<param name="CCW Compliance Slope">128</param>
 			<param name="Return Delay Time">10</param>
 		</gpio>
@@ -230,6 +230,6 @@
 			<param name="CW Compliance Margin">1</param>
 			<param name="CCW Compliance Margin">1</param>
-			<param name="CW Compliance Slope">254</param>
-			<param name="CCW Compliance Slope">254</param>
+			<param name="CW Compliance Slope">127</param>
+			<param name="CCW Compliance Slope">127</param>
 			<param name="Return Delay Time">10</param>
 		</gpio>

Commit message: (FG): add missing config for gazebo simulation

File: bender_description/urdf/bender.xacro (robot description, xacro)
@@ -3,5 +3,10 @@
   <xacro:include filename="$(find bender_description)/urdf/materials.xacro" />
   <xacro:include filename="$(find bender_description)/urdf/rgbd_camera.xacro"/>
-  <xacro:include filename="$(find bender_description)/urdf/ros2_control.xacro" />
+  <xacro:arg name="hardware" default="real"/>
+  <xacro:property name="hardware" value="$(arg hardware)"/>
+  <xacro:if value="${hardware not in ['real', 'mock', 'sim']}">
+    ${xacro.fatal("hardware param must be 'real', 'mock' o 'sim', got: " + hardware)}
+  </xacro:if>
+  <xacro:include filename="$(find bender_description)/urdf/bender_${hardware}.xacro"/>
   <xacro:property name="epsilon" value="1e-4"/>
   <xacro:rgbd_camera

File: bender_description/urdf/bender_real.xacro (robot description, xacro)
@@ -417,10 +417,4 @@
 		</gpio>
 	</ros2_control>
-	<!-- DESHABILITADO temporalmente para probar todo menos la base Pioneer.
-	     Recordar sacar también wrl_to_base_link/wrr_to_base_link de la lista
-	     de joints de joint_state_broadcaster en controllers.yaml: si quedan
-	     ahí sin hardware detrás, controller_manager aborta el proceso completo
-	     al no encontrar esas interfaces. -->
-	<!--
 	<ros2_control name="Pioneer" type="system">
     	<hardware>
@@ -441,5 +435,3 @@
         </sensor>
 	</ros2_control>
-	-->
-	<!-- FIN bloque Pioneer -->
 </robot>

File: bender_description/urdf/bender_sim.xacro (robot description, xacro)
@@ -86,4 +86,10 @@
       <state_interface name="effort"/>
     </joint>
+    <joint name="l3h_to_l1h">
+      <command_interface name="position"/>
+      <state_interface name="position"/>
+      <state_interface name="velocity"/>
+      <state_interface name="effort"/>
+    </joint>
     <joint name="l1h_to_base_link">
       <command_interface name="position"/>
@@ -93,11 +99,6 @@
     </joint>
      <!-- Gripper Izquierdo -->
-    <joint name="g2la_to_g1l">
+    <joint name="gripper_base_to_movil">
       <command_interface name="position"/>
-      <state_interface name="position"/>
-      <state_interface name="velocity"/>
-      <state_interface name="effort"/>
-    </joint>
-    <joint name="g2lb_to_g1l">
       <state_interface name="position"/>
       <state_interface name="velocity"/>
@@ -127,11 +128,10 @@
       <state_interface name="position"/>
     </joint>
+    <!-- Delanteras: mimic de las traseras (definido en bender.xacro), por eso sin comando -->
     <joint name="wfl_to_base_link">
-      <command_interface name="velocity"/>
       <state_interface name="velocity"/>
       <state_interface name="position"/>
     </joint>
     <joint name="wfr_to_base_link">
-      <command_interface name="velocity"/>
       <state_interface name="velocity"/>
       <state_interface name="position"/>

File: bender_moveit_config/config/bender.urdf.xacro (robot description, xacro)
@@ -1,9 +1,6 @@
 <?xml version="1.0"?>
 <robot xmlns:xacro="http://www.ros.org/wiki/xacro" name="bender">
-    <xacro:arg name="initial_positions_file" default="initial_positions.yaml" />
-    <!-- Import bender urdf file -->
+    <!-- Se declara antes del include para que este default le gane al de bender.xacro (real). -->
+    <xacro:arg name="hardware" default="mock" />
     <xacro:include filename="$(find bender_description)/urdf/bender.xacro" />
-    <!-- Import control_xacro -->
-    <xacro:include filename="bender.ros2_control.xacro" />
-    <xacro:bender_ros2_control name="FakeSystem" initial_positions_file="$(arg initial_positions_file)"/>
 </robot>
