Commit message: (FG): add configuration for gazebo

File: bender_description/urdf/bender.xacro (robot description, xacro)
@@ -10,4 +10,8 @@
   <xacro:include filename="$(find bender_description)/urdf/bender_${hardware}.xacro"/>
   <xacro:property name="epsilon" value="1e-4"/>
+  <!-- TODO: change mass -->
+  <xacro:property name="gripper_l_base_mass" value="0.0733"/>   <!-- 118.2 cm3 -->
+  <xacro:property name="gripper_l_fijo_mass" value="0.0233"/>   <!-- 37.6 cm3 -->
+  <xacro:property name="gripper_l_movil_mass" value="0.0420"/>  <!-- 67.8 cm3 -->
   <xacro:rgbd_camera
       prefix=""
@@ -341,4 +345,10 @@
     </joint>
     <link name="gripper_l_base">
+          <inertial>
+            <origin xyz="-0.002432 0.002273 -0.032502" rpy="0 0 0"/>
+            <mass value="${gripper_l_base_mass}"/>
+            <inertia ixx="${gripper_l_base_mass * 4.79885e-4}" iyy="${gripper_l_base_mass * 5.64127e-4}" izz="${gripper_l_base_mass * 3.73860e-4}"
+                     ixy="${gripper_l_base_mass * -2.978e-6}" ixz="${gripper_l_base_mass * 1.7268e-5}" iyz="${gripper_l_base_mass * -1.48e-7}"/>
+          </inertial>
           <visual>
             <origin rpy="0 0 0" xyz="0 0 0"/>
@@ -360,4 +370,10 @@
         </joint>
         <link name="fijo">
+          <inertial>
+            <origin xyz="0.038899 0.002262 0.018539" rpy="0 0 0"/>
+            <mass value="${gripper_l_fijo_mass}"/>
+            <inertia ixx="${gripper_l_fijo_mass * 1.404186e-3}" iyy="${gripper_l_fijo_mass * 1.246171e-3}" izz="${gripper_l_fijo_mass * 1.92308e-4}"
+                     ixy="${gripper_l_fijo_mass * 0.0}" ixz="${gripper_l_fijo_mass * -4.8706e-5}" iyz="${gripper_l_fijo_mass * 0.0}"/>
+          </inertial>
           <visual>
             <origin rpy="0 0 0" xyz="0 0 0"/>
@@ -381,4 +397,10 @@
         </joint>
         <link name="movil">
+          <inertial>
+            <origin xyz="-0.003199 0.002041 0.044445" rpy="0 0 0"/>
+            <mass value="${gripper_l_movil_mass}"/>
+            <inertia ixx="${gripper_l_movil_mass * 1.909822e-3}" iyy="${gripper_l_movil_mass * 1.526318e-3}" izz="${gripper_l_movil_mass * 5.58397e-4}"
+                     ixy="${gripper_l_movil_mass * 1.487e-6}" ixz="${gripper_l_movil_mass * -4.0392e-5}" iyz="${gripper_l_movil_mass * 3.214e-6}"/>
+          </inertial>
           <visual>
             <origin rpy="0 0 0" xyz="0 0 0"/>

File: bender_description/urdf/bender_sim.xacro (robot description, xacro)
@@ -1,140 +1,63 @@
 <?xml version="1.0"?>
 <robot name="bender" xmlns:xacro="http://www.ros.org/wiki/xacro">
-  <ros2_control name="RobotSystem" type="system">
-    <hardware>
-          <plugin>gz_ros2_control/GazeboSimSystem</plugin>
-    </hardware>
-    <!-- Brazo Izquierdo -->
-    <joint name="l1l_to_base_link">
+  <xacro:macro name="sim_position_joint" params="name">
+    <joint name="${name}">
       <command_interface name="position"/>
+      <state_interface name="position"/>
+      <state_interface name="velocity"/>
+    </joint>
+  </xacro:macro>
+  <xacro:macro name="sim_shoulder_joint" params="name">
+    <joint name="${name}">
+      <command_interface name="velocity"/>
+      <command_interface name="effort"/>
       <state_interface name="position"/>
       <state_interface name="velocity"/>
       <state_interface name="effort"/>
     </joint>
-    <joint name="l2l_to_l1l">
-      <command_interface name="position"/>
+  </xacro:macro>
+  <xacro:macro name="sim_mimic_joint" params="name">
+    <joint name="${name}">
       <state_interface name="position"/>
       <state_interface name="velocity"/>
-      <state_interface name="effort"/>
     </joint>
-    <joint name="l3l_to_l2l">
-      <command_interface name="position"/>
-      <state_interface name="position"/>
-      <state_interface name="velocity"/>
-      <state_interface name="effort"/>
-    </joint>
-    <joint name="l4l_to_l3l">
-      <command_interface name="position"/>
-      <state_interface name="position"/>
-      <state_interface name="velocity"/>
-      <state_interface name="effort"/>
-    </joint>
-    <joint name="l5l_to_l4l">
-      <command_interface name="position"/>
-      <state_interface name="position"/>
-      <state_interface name="velocity"/>
-      <state_interface name="effort"/>
-    </joint>
-    <joint name="l6l_to_l5l">
-      <command_interface name="position"/>
-      <state_interface name="position"/>
-      <state_interface name="velocity"/>
-      <state_interface name="effort"/>
-    </joint>
-    <!-- Brazo Derecho -->
-    <joint name="l1r_to_base_link">
-      <command_interface name="position"/>
-      <state_interface name="position"/>
-      <state_interface name="velocity"/>
-      <state_interface name="effort"/>
-    </joint>
-    <joint name="l2r_to_l1r">
-      <command_interface name="position"/>
-      <state_interface name="position"/>
-      <state_interface name="velocity"/>
-      <state_interface name="effort"/>
-    </joint>
-    <joint name="l3r_to_l2r">
-      <command_interface name="position"/>
-      <state_interface name="position"/>
-      <state_interface name="velocity"/>
-      <state_interface name="effort"/>
-    </joint>
-    <joint name="l4r_to_l3r">
-      <command_interface name="position"/>
-      <state_interface name="position"/>
-      <state_interface name="velocity"/>
-      <state_interface name="effort"/>
-    </joint>
-    <joint name="l5r_to_l4r">
-      <command_interface name="position"/>
-      <state_interface name="position"/>
-      <state_interface name="velocity"/>
-      <state_interface name="effort"/>
-    </joint>
-    <joint name="l6r_to_l5r">
-      <command_interface name="position"/>
-      <state_interface name="position"/>
-      <state_interface name="velocity"/>
-      <state_interface name="effort"/>
-    </joint>
-    <!-- Cuello -->
-    <joint name="l2h_to_l1h">
-      <command_interface name="position"/>
-      <state_interface name="position"/>
-      <state_interface name="velocity"/>
-      <state_interface name="effort"/>
-    </joint>
-    <joint name="l3h_to_l1h">
-      <command_interface name="position"/>
-      <state_interface name="position"/>
-      <state_interface name="velocity"/>
-      <state_interface name="effort"/>
-    </joint>
-    <joint name="l1h_to_base_link">
-      <command_interface name="position"/>
-      <state_interface name="position"/>
-      <state_interface name="velocity"/>
-      <state_interface name="effort"/>
-    </joint>
-     <!-- Gripper Izquierdo -->
-    <joint name="gripper_base_to_movil">
-      <command_interface name="position"/>
-      <state_interface name="position"/>
-      <state_interface name="velocity"/>
-      <state_interface name="effort"/>
-    </joint>
-    <!-- Gripper Derecho -->
-    <joint name="g2ra_to_g1r">
-      <command_interface name="position"/>
-      <state_interface name="position"/>
-      <state_interface name="velocity"/>
-      <state_interface name="effort"/>
-    </joint>
-    <joint name="g2rb_to_g1r">
-      <state_interface name="position"/>
-      <state_interface name="velocity"/>
-      <state_interface name="effort"/>
-    </joint>
-    <!-- RUEDAS BASE -->
-    <joint name="wrl_to_base_link">
+  </xacro:macro>
+  <xacro:macro name="sim_wheel_joint" params="name">
+    <joint name="${name}">
       <command_interface name="velocity"/>
       <state_interface name="velocity"/>
       <state_interface name="position"/>
     </joint>
-    <joint name="wrr_to_base_link">
-      <command_interface name="velocity"/>
-      <state_interface name="velocity"/>
-      <state_interface name="position"/>
-    </joint>
-    <!-- Delanteras: mimic de las traseras (definido en bender.xacro), por eso sin comando -->
-    <joint name="wfl_to_base_link">
-      <state_interface name="velocity"/>
-      <state_interface name="position"/>
-    </joint>
-    <joint name="wfr_to_base_link">
-      <state_interface name="velocity"/>
-      <state_interface name="position"/>
-    </joint>
+  </xacro:macro>
+  <ros2_control name="RobotSystem" type="system">
+    <hardware>
+      <plugin>gz_ros2_control/GazeboSimSystem</plugin>
+    </hardware>
+    <!-- left arms -->
+    <xacro:sim_shoulder_joint name="l1l_to_base_link"/>
+    <xacro:sim_position_joint name="l2l_to_l1l"/>
+    <xacro:sim_position_joint name="l3l_to_l2l"/>
+    <xacro:sim_position_joint name="l4l_to_l3l"/>
+    <xacro:sim_position_joint name="l5l_to_l4l"/>
+    <xacro:sim_position_joint name="l6l_to_l5l"/>
+    <!-- right arms -->
+    <xacro:sim_shoulder_joint name="l1r_to_base_link"/>
+    <xacro:sim_position_joint name="l2r_to_l1r"/>
+    <xacro:sim_position_joint name="l3r_to_l2r"/>
+    <xacro:sim_position_joint name="l4r_to_l3r"/>
+    <xacro:sim_position_joint name="l5r_to_l4r"/>
+    <xacro:sim_position_joint name="l6r_to_l5r"/>
+    <!-- Head -->
+    <xacro:sim_position_joint name="l1h_to_base_link"/>
+    <xacro:sim_position_joint name="l2h_to_l1h"/>
+    <xacro:sim_position_joint name="l3h_to_l1h"/>
+    <!-- Grippers -->
+    <xacro:sim_position_joint name="gripper_base_to_movil"/>
+    <xacro:sim_position_joint name="g2ra_to_g1r"/>
+    <xacro:sim_mimic_joint name="g2rb_to_g1r"/>
+    <xacro:sim_wheel_joint name="wrl_to_base_link"/>
+    <xacro:sim_wheel_joint name="wrr_to_base_link"/>
+    <xacro:sim_mimic_joint name="wfl_to_base_link"/>
+    <xacro:sim_mimic_joint name="wfr_to_base_link"/>
   </ros2_control>
   <gazebo>

Commit message: (FG): change joint limits

File: bender_description/urdf/bender.xacro (robot description, xacro)
@@ -396,5 +396,5 @@
           <parent link="gripper_l_base"/>
           <child link="movil"/>
-          <limit effort="1000.0" lower="-2.0" upper="0.3495" velocity="0.5"/>
+          <limit effort="1000.0" lower="-2.100" upper="0.359" velocity="0.5"/>
         </joint>
         <link name="movil">
@@ -590,5 +590,5 @@
     <child link="l2l_1"/>
     <axis xyz="1.0 0.0 -0.0"/>
-    <limit upper="${1.570796 + epsilon}" lower="-0.09" effort="100.0" velocity="100.0"/>
+    <limit upper="1.794" lower="-0.193" effort="100.0" velocity="100.0"/>
   </joint>
   <joint name="l3l_to_l2l" type="revolute">
@@ -597,5 +597,5 @@
     <child link="l3l_1"/>
     <axis xyz="0.0 -0.0 1.0"/>
-    <limit upper="${1.134464 + epsilon}" lower="${-1.134464 - epsilon}" effort="100.0" velocity="100.0"/>
+    <limit upper="1.148" lower="-1.027" effort="100.0" velocity="100.0"/>
   </joint>
   <joint name="l4l_to_l3l" type="revolute">
@@ -604,5 +604,5 @@
     <child link="l4l_1"/>
     <axis xyz="-0.0 -1.0 0.0"/>
-    <limit upper="${2.356194 + epsilon}" lower="-1.5" effort="100.0" velocity="100.0"/>
+    <limit upper="2.011" lower="-2.127" effort="100.0" velocity="100.0"/>
   </joint>
   <joint name="l5l_to_l4l" type="revolute">
@@ -611,5 +611,5 @@
     <child link="l5l_1"/>
     <axis xyz="0.0 -0.0 -1.0"/>
-    <limit upper="${1.047198 + epsilon}" lower="${-1.047198 -epsilon}" effort="100.0" velocity="100.0"/>
+    <limit upper="1.308" lower="-1.262" effort="100.0" velocity="100.0"/>
   </joint>
   <joint name="l6l_to_l5l" type="revolute">
@@ -618,5 +618,5 @@
     <child link="l6l_1"/>
     <axis xyz="0.0 1.0 0.0"/>
-    <limit upper="${1.570796 + epsilon}" lower="${-1.570796 -epsilon}" effort="100.0" velocity="100.0"/>
+    <limit upper="1.508" lower="-1.209" effort="100.0" velocity="100.0"/>
   </joint>
   <joint name="l2r_to_l1r" type="revolute">
@@ -625,5 +625,5 @@
     <child link="l2r_1"/>
     <axis xyz="1.0 0.0 0.0"/>
-    <limit upper="0.1" lower="${-1.570796 - 0.1}" effort="100.0" velocity="100.0"/>
+    <limit upper="0.181" lower="-1.668" effort="100.0" velocity="100.0"/>
   </joint>
   <joint name="l3r_to_l2r" type="revolute">
@@ -632,5 +632,5 @@
     <child link="l3r_1"/>
     <axis xyz="0.0 0.0 -1.0"/>
-    <limit upper="${1.134464 + epsilon}" lower="${-1.134464 -epsilon}" effort="100.0" velocity="100.0"/>
+    <limit upper="1.138" lower="-1.240" effort="100.0" velocity="100.0"/>
   </joint>
   <joint name="l4r_to_l3r" type="revolute">
@@ -639,5 +639,5 @@
     <child link="l4r_1"/>
     <axis xyz="-0.0 1.0 0.0"/>
-    <limit upper="1.5" lower="${-2.356194 - epsilon}" effort="100.0" velocity="100.0"/>
+    <limit upper="1.974" lower="-2.100" effort="100.0" velocity="100.0"/>
   </joint>
   <joint name="l5r_to_l4r" type="revolute">
@@ -646,5 +646,5 @@
     <child link="l5r_1"/>
     <axis xyz="-0.0 0.0 -1.0"/>
-    <limit upper="${1.047198 + epsilon}" lower="${-1.047198 - epsilon}" effort="100.0" velocity="100.0"/>
+    <limit upper="1.314" lower="-1.150" effort="100.0" velocity="100.0"/>
   </joint>
   <joint name="l6r_to_l5r" type="revolute">
@@ -653,5 +653,5 @@
     <child link="l6r_1"/>
     <axis xyz="-0.0 1.0 0.0"/>
-    <limit upper="${1.570796 + epsilon}" lower="${-1.570796 - epsilon}" effort="100.0" velocity="100.0"/>
+    <limit upper="1.867" lower="-1.948" effort="100.0" velocity="100.0"/>
   </joint>
   <!-- head pitch joint -->
@@ -747,5 +747,5 @@
     <child link="l1h_1"/>
     <axis xyz="0.0 0.0 1.0"/>
-    <limit effort="50.0" lower="${-1.570796 - epsilon}" upper="${1.570796 + epsilon}" velocity="50.0"/>
+    <limit effort="50.0" lower="-3.229" upper="1.948" velocity="50.0"/>
   </joint>
   <link name="base_footprint"/>

File: bender_description/urdf/bender_real.xacro (robot description, xacro)
@@ -32,9 +32,8 @@
 		</ros2_control>
 	</xacro:macro>
-	<!-- use_arms: hombros (ODrive + encoders) y cadenas Dynamixel (brazos, grippers y cabeza) -->
 	<xacro:if value="$(arg use_arms)">
 	<xacro:odrive_ros2_control
     name="Odrive"
-    serial_number="3690387D3333"
+    serial_number="336B33573235"
     joint_name_left="l1l_to_base_link"
     joint_name_right="l1r_to_base_link"
@@ -96,14 +95,13 @@
 		<gpio name="motor_l2r">
     		<param name="type">dxl</param>
-    		<param name="ID">4</param>
+    		<param name="ID">1</param>
     		<command_interface name="Goal Position" />
     		<state_interface name="Present Position" />
     		<state_interface name="Present Velocity" />
     		<state_interface name="Present Load" />
-    		<param name="[unit info]">Present Position, 0.001047198, rad, unsigned, -1.6221098; Goal Position, 0.001047198, rad, unsigned, -1.6221098</param>
-    		<param name="CW Compliance Margin">1</param>
-    		<param name="CCW Compliance Margin">1</param>
-    		<param name="CW Compliance Slope">50</param>
-    		<param name="CCW Compliance Slope">50</param>
+    		<param name="[unit info]">Present Position, -0.001533981, rad, unsigned, 3.113981; Goal Position, -0.001533981, rad, unsigned, 3.113981</param>
+    		<param name="P Gain">8</param>
+    		<param name="I Gain">2</param>
+    		<param name="D Gain">5</param>
     		<param name="Return Delay Time">5</param>
 		</gpio>
@@ -134,10 +132,10 @@
 		<gpio name="motor_l4r">
 			<param name="type">dxl</param>
-			<param name="ID">13</param>
-			<command_interface name="Goal Position" />
-			<state_interface name="Present Position" />
-			<state_interface name="Present Velocity" />
-			<state_interface name="Present Load" />
-			<param name="[unit info]">Present Position, 0.001533981, rad, unsigned, -3.05262219; Goal Position, 0.001533981, rad, unsigned, -3.05262219</param>
+			<param name="ID">11</param>
+			<command_interface name="Goal Position" />
+			<state_interface name="Present Position" />
+			<state_interface name="Present Velocity" />
+			<state_interface name="Present Load" />
+			<param name="[unit info]">Present Position, -0.001533981, rad, unsigned, 3.983749; Goal Position, -0.001533981, rad, unsigned, 3.983749</param>
 			<param name="P Gain">50</param>
 			<param name="I Gain">32</param>
@@ -193,9 +191,10 @@
 		<gpio name="motor_g2ra">
 			<param name="type">dxl</param>
-			<param name="ID">16</param>
-			<command_interface name="Goal Position" />
-			<state_interface name="Present Position" />
-			<state_interface name="Present Velocity" />
-			<state_interface name="Present Load" />
+			<param name="ID">6</param>
+			<command_interface name="Goal Position" />
+			<state_interface name="Present Position" />
+			<state_interface name="Present Velocity" />
+			<state_interface name="Present Load" />
+			<param name="[unit info]">Present Position, 0.005061455, rad, unsigned, -2.647141; Goal Position, 0.005061455, rad, unsigned, -2.647141</param>
 			<param name="CW Compliance Margin">1</param>
 			<param name="CCW Compliance Margin">1</param>
@@ -264,7 +263,9 @@
     		<state_interface name="Present Velocity" />
     		<state_interface name="Present Load" />
-    		<param name="P Gain">8</param>
-    		<param name="I Gain">2</param>
-    		<param name="D Gain">5</param>
+    		<param name="[unit info]">Present Position, -0.001047198, rad, unsigned, 3.878821; Goal Position, -0.001047198, rad, unsigned, 3.878821</param>
+    		<param name="CW Compliance Margin">1</param>
+    		<param name="CCW Compliance Margin">1</param>
+    		<param name="CW Compliance Slope">50</param>
+    		<param name="CCW Compliance Slope">50</param>
     		<param name="Return Delay Time">5</param>
 		</gpio>
@@ -295,10 +296,10 @@
 		<gpio name="motor_l4l">
 			<param name="type">dxl</param>
-			<param name="ID">11</param>
-			<command_interface name="Goal Position" />
-			<state_interface name="Present Position" />
-			<state_interface name="Present Velocity" />
-			<state_interface name="Present Load" />
-			<param name="[unit info]">Present Position, 0.001533981, rad, unsigned, -3.040350342; Goal Position, 0.001533981, rad, unsigned, -3.040350342</param>
+			<param name="ID">13</param>
+			<command_interface name="Goal Position" />
+			<state_interface name="Present Position" />
+			<state_interface name="Present Velocity" />
+			<state_interface name="Present Load" />
+			<param name="[unit info]">Present Position, 0.001533981, rad, unsigned, -2.127632; Goal Position, 0.001533981, rad, unsigned, -2.127632</param>
 			<param name="P Gain">8</param>
 			<param name="I Gain">2</param>
@@ -331,9 +332,10 @@
 		<gpio name="motor_l6l">
 			<param name="type">dxl</param>
-			<param name="ID">6</param>
-			<command_interface name="Goal Position" />
-			<state_interface name="Present Position" />
-			<state_interface name="Present Velocity" />
-			<state_interface name="Present Load" />
+			<param name="ID">16</param>
+			<command_interface name="Goal Position" />
+			<state_interface name="Present Position" />
+			<state_interface name="Present Velocity" />
+			<state_interface name="Present Load" />
+			<param name="[unit info]">Present Position, 0.005061455, rad, unsigned, -2.672448; Goal Position, 0.005061455, rad, unsigned, -2.672448</param>
 			<param name="CW Compliance Margin">1</param>
 			<param name="CCW Compliance Margin">1</param>
@@ -420,5 +422,4 @@
 	</ros2_control>
 	</xacro:if>
-	<!-- use_base: base Pioneer y parada de emergencia -->
 	<xacro:if value="$(arg use_base)">
 	<ros2_control name="Pioneer" type="system">
@@ -428,5 +429,4 @@
             <param name="baud_rate">9600</param>
             <param name="wheel_separation">0.397</param>
-            <!-- Igual que wheel_radius de pioneer_base_controller (controllers.yaml) -->
             <param name="wheel_radius">0.1</param>
         </hardware>

Commit message: (FG): change limits

File: bender_description/urdf/bender.xacro (robot description, xacro)
@@ -661,5 +661,5 @@
     <child link="l2h_1"/>
     <axis xyz="-0.0 1.0 0.0"/>
-    <limit effort="50" lower="${-0.706858 - epsilon}" upper="${0.706858 + epsilon}" velocity="50"/>
+    <limit effort="50" lower="-0.726" upper="0.625" velocity="50"/>
   </joint>
   <joint name="l3h_to_l1h" type="revolute">
@@ -668,5 +668,5 @@
     <child link="l3h_1"/>
     <axis xyz="1.0 0.0 0.0"/>
-    <limit effort="50" lower="${-0.706858 - epsilon}" upper="${0.706858 + epsilon}" velocity="50"/>
+    <limit effort="50" lower="-0.405" upper="0.458" velocity="50"/>
   </joint>
   <joint name="g1r_to_l6r" type="fixed">

File: bender_description/urdf/bender_real.xacro (robot description, xacro)
@@ -401,9 +401,9 @@
 			<state_interface name="Present Velocity" />
 			<state_interface name="Present Load" />
-			<param name="[unit info]">Present Position, 0.005061455, rad, unsigned, -1.012291; Goal Position, 0.005061455, rad, unsigned, -1.012291</param>
-			<param name="CW Compliance Margin">1</param>
-			<param name="CCW Compliance Margin">1</param>
-			<param name="CW Compliance Slope">254</param>
-			<param name="CCW Compliance Slope">254</param>
+			<param name="[unit info]">Present Position, 0.005061455, rad, unsigned, -1.098335735; Goal Position, 0.005061455, rad, unsigned, -1.098335735</param>
+			<param name="CW Compliance Margin">1</param>
+			<param name="CCW Compliance Margin">1</param>
+			<param name="CW Compliance Slope">32</param>
+			<param name="CCW Compliance Slope">32</param>
 			<param name="Return Delay Time">5</param>
 		</gpio>
@@ -415,9 +415,9 @@
 			<state_interface name="Present Velocity" />
 			<state_interface name="Present Load" />
-			<param name="[unit info]">Present Position, 0.005061455, rad, unsigned, -3.912504715; Goal Position, 0.005061455, rad, unsigned, -3.912504715</param>
-			<param name="CW Compliance Margin">1</param>
-			<param name="CCW Compliance Margin">1</param>
-			<param name="CW Compliance Slope">254</param>
-			<param name="CCW Compliance Slope">254</param>
+			<param name="[unit info]">Present Position, 0.005061455, rad, unsigned, -3.831521435; Goal Position, 0.005061455, rad, unsigned, -3.831521435</param>
+			<param name="CW Compliance Margin">1</param>
+			<param name="CCW Compliance Margin">1</param>
+			<param name="CW Compliance Slope">32</param>
+			<param name="CCW Compliance Slope">32</param>
 			<param name="Return Delay Time">5</param>
 		</gpio>
