Commit message: (FG): add new parameters

File: bender_description/urdf/ros2_control.xacro (robot description, xacro)
@@ -1,361 +1,347 @@
 <?xml version="1.0" ?>
-<robot xmlns:xacro="http://www.ros.org/wiki/xacro">
-<!-- <xacro:macro name="odrive_ros2_control" params="name serial_number joint_name axis:=0">
-    <ros2_control name="${name}" type="system">
-      <hardware>
-        <plugin>odrive_hardware_interface/ODriveHardwareInterface</plugin>
-      </hardware>
-      <sensor name="${name}_dev0">
-        <param name="serial_number">${serial_number}</param>
-      </sensor>
-      <joint name="${joint_name}">
-        <param name="serial_number">${serial_number}</param>
-        <param name="axis">${axis}</param>
-        <param name="enable_watchdog">1</param>
-        <param name="watchdog_timeout">1.0</param>
-        <command_interface name="position" />
-        <command_interface name="velocity" />
-        <command_interface name="effort" />
-        <state_interface name="position" />
-        <state_interface name="velocity" />
-        <state_interface name="effort" />
-      </joint>
-    </ros2_control>
-  </xacro:macro>
-  <xacro:odrive_ros2_control
+<robot
+	xmlns:xacro="http://www.ros.org/wiki/xacro">
+<xacro:macro name="odrive_ros2_control" params="name serial_number joint_name axis:=0 gear_ratio:=1.0">
+		<ros2_control name="${name}" type="system">
+			<hardware>
+				<plugin>odrive_hardware_interface/ODriveHardwareInterface</plugin>
+			</hardware>
+			<sensor name="${name}_dev0">
+				<param name="serial_number">${serial_number}</param>
+			</sensor>
+			<joint name="${joint_name}">
+				<param name="serial_number">${serial_number}</param>
+				<param name="axis">${axis}</param>
+				<param name="enable_watchdog">0</param>
+				<param name="watchdog_timeout">1.0</param>
+				<param name="gear_ratio">${gear_ratio}</param>
+				<command_interface name="position" />
+				<command_interface name="velocity" />
+				<command_interface name="effort" />
+				<state_interface name="effort" />
+			</joint>
+		</ros2_control>
+	</xacro:macro>
+	<xacro:odrive_ros2_control
     name="OdriveLeft"
+    serial_number="3690387D3333"
+    joint_name="l1l_to_base_link"
+    axis="0"
+	gear_ratio="250"
+	/>
+	<xacro:odrive_ros2_control
+    name="OdriveRight"
     serial_number="336B33573235"
-    joint_name="l1l_to_base_link"
-    axis="0"/>
-  <xacro:odrive_ros2_control
-    name="OdriveRight"
-    serial_number="CAMBIA EL NUMERO DE SERIE LUCHO"
     joint_name="l1r_to_base_link"
-    axis="0"/>
-  <transmission name="trans_l1l_to_base_link">
-    <plugin>transmission_interface/SimpleTransmission</plugin>
-    <actuator name="motor_l1l_to_base_link" role="actuator1"/>
-    <joint name="l1l_to_base_link" role="joint1">
-      <mechanicalReduction>10.0</mechanicalReduction>
-    </joint>
-  </transmission>
-  <transmission name="trans_l1r_to_base_link">
-    <plugin>transmission_interface/SimpleTransmission</plugin>
-    <actuator name="motor_l1r_to_base_link" role="actuator1"/>
-    <joint name="l1r_to_base_link" role="joint1">
-      <mechanicalReduction>10.0</mechanicalReduction>
-    </joint>
-  </transmission>
-       <ros2_control name="ShoulderJoint" type="sensor">
-           <hardware>
-             <plugin>bender_hardware_interfaces/EncoderInterface</plugin>
-             <param name="serial_device">/dev/encoders</param>
-             <param name="baud_rate">115200</param>
-           </hardware>
-           <sensor name="base_link_to_l1l">
-             <state_interface name="position" />
-             <state_interface name="velocity" />
-           </sensor>
-           <sensor name="base_link_to_l1r">
-             <state_interface name="position" />
-             <state_interface name="velocity" />
-           </sensor>
-         </ros2_control> -->
-         <ros2_control name="DynamixelChainMain" type="system">
-             <hardware>
-               <plugin>dynamixel_hardware_interface/DynamixelHardware</plugin>
-               <param name="port_name">/dev/dynamixel</param>
-               <param name="baud_rate">1000000</param>
-               <param name="protocol_version">1.0</param>
-               <param name="number_of_joints">14</param>
-               <param name="number_of_transmissions">14</param>
-               <param name="dynamixel_model_folder">/param/dxl_model</param>
-               <param name="disable_torque_at_init">true</param>
-               <param name="torque_enable">0</param>
-             </hardware>
-             <joint name="l2r_to_l1r">
-                <command_interface name="position" />
-                <state_interface name="position" />
-                <state_interface name="velocity" />
-             </joint>
-             <joint name="l3r_to_l2r">
-                <command_interface name="position" />
-                <state_interface name="position" />
-                <state_interface name="velocity" />
-             </joint>
-             <joint name="l4r_to_l3r">
-                <command_interface name="position" />
-                <state_interface name="position" />
-                <state_interface name="velocity" />
-             </joint>
-             <joint name="l5r_to_l4r">
-                <command_interface name="position" />
-                <state_interface name="position" />
-                <state_interface name="velocity" />
-             </joint>
-             <joint name="l6r_to_l5r">
-                <command_interface name="position" />
-                <state_interface name="position" />
-                <state_interface name="velocity" />
-             </joint>
-             <joint name="l2l_to_l1l">
-                <command_interface name="position" />
-                <state_interface name="position" />
-                <state_interface name="velocity" />
-             </joint>
-             <joint name="l3l_to_l2l">
-                <command_interface name="position" />
-                <state_interface name="position" />
-                <state_interface name="velocity" />
-             </joint>
-             <joint name="l5l_to_l4l">
-                <command_interface name="position" />
-                <state_interface name="position" />
-                <state_interface name="velocity" />
-             </joint>
-             <joint name="l6l_to_l5l">
-                <command_interface name="position" />
-                <state_interface name="position" />
-                <state_interface name="velocity" />
-             </joint>
-             <joint name="g2ra_to_g1r">
-                <command_interface name="position" />
-                <state_interface name="position" />
-                <state_interface name="velocity" />
-             </joint>
-             <joint name="g2rb_to_g1r">
-                <command_interface name="position" />
-                <state_interface name="position" />
-                <state_interface name="velocity" />
-             </joint>
-             <!-- <joint name="g2r_to_g1r"><command_interface name="position" /><state_interface name="position" /><state_interface name="velocity" /></joint> -->
-             <joint name="l1h_to_base_link">
-                <command_interface name="position" />
-                <state_interface name="position" />
-                <state_interface name="velocity" />
-             </joint>
-             <joint name="l2h_to_l1h">
-                <command_interface name="position" />
-                <state_interface name="position" />
-                <state_interface name="velocity" />
-             </joint>
-             <!-- <joint name="l2h_to_l1h_coupled"><command_interface name="position" /><state_interface name="position" /><state_interface name="velocity" /></joint> -->
-             <gpio name="motor_l2r">
-                <param name="type">dxl</param>
-                <param name="ID">11</param>
-                <command_interface name="Goal Position" />
-                <state_interface name="Present Position" />
-                <state_interface name="Present Velocity" />
-                <state_interface name="Present Load" />
-                <!-- software re-center -->
-                <param name="[unit info]">Present Position, 0.001533981, rad, unsigned, -3.1001879291; Goal Position, 0.001533981, rad, unsigned, -3.1001879291</param>
-                <param name="P Gain">8</param>
-                <param name="I Gain">2</param>
-                <param name="D Gain">5</param>
-                <param name="Return Delay Time">25</param>
-            </gpio>
-             <gpio name="motor_l3r">
-                <param name="type">dxl</param>
-                <param name="ID">12</param>
-                <command_interface name="Goal Position" />
-                <state_interface name="Present Position" />
-                <state_interface name="Present Velocity" />
-                <state_interface name="Present Load" />
-                <!-- doesn't need recentering -->
-                <param name="CW Compliance Margin">1</param>
-                <param name="CCW Compliance Margin">1</param>
-                <param name="CW Compliance Slope">254</param>
-                <param name="CCW Compliance Slope">254</param>
-                <param name="Return Delay Time">25</param>
-             </gpio>
-             <gpio name="motor_l4r">
-                <param name="type">dxl</param>
-                <param name="ID">13</param>
-                <command_interface name="Goal Position" />
-                <state_interface name="Present Position" />
-                <state_interface name="Present Velocity" />
-                <state_interface name="Present Load" />
-                <param name="[unit info]">Present Position, 0.001533981, rad, unsigned, -3.471399003; Goal Position, 0.001533981, rad, unsigned, -3.471399003</param>
-                <param name="P Gain">8</param>
-                <param name="I Gain">2</param>
-                <param name="D Gain">5</param>
-                <param name="Return Delay Time">25</param>
-             </gpio>
-             <gpio name="motor_l5r">
-                <param name="type">dxl</param>
-                <param name="ID">14</param>
-                <command_interface name="Goal Position" />
-                <state_interface name="Present Position" />
-                <state_interface name="Present Velocity" />
-                <state_interface name="Present Load" />
-                <param name="CW Compliance Margin">1</param>
-                <param name="CCW Compliance Margin">1</param>
-                <param name="CW Compliance Slope">254</param>
-                <param name="CCW Compliance Slope">254</param>
-                <param name="Return Delay Time">25</param>
-             </gpio>
-             <gpio name="motor_l6r">
-                <param name="type">dxl</param>
-                <param name="ID">15</param>
-                <command_interface name="Goal Position" />
-                <state_interface name="Present Position" />
-                <state_interface name="Present Velocity" />
-                <state_interface name="Present Load" />
-                <param name="CW Compliance Margin">1</param>
-                <param name="CCW Compliance Margin">1</param>
-                <param name="CW Compliance Slope">254</param>
-                <param name="CCW Compliance Slope">254</param>
-                <param name="Return Delay Time">25</param>
-             </gpio>
-             <gpio name="motor_l2l">
-                <param name="type">dxl</param>
-                <param name="ID">4</param>
-                <command_interface name="Goal Position" />
-                <state_interface name="Present Position" />
-                <state_interface name="Present Velocity" />
-                <state_interface name="Present Load" />
-                <param name="[unit info]">Present Position, 0.001047198, rad, unsigned, -1.6221098; Goal Position, 0.001047198, rad, unsigned, -1.6221098</param>
-                <param name="CW Compliance Margin">1</param>
-                <param name="CCW Compliance Margin">1</param>
-                <param name="CW Compliance Slope">254</param>
-                <param name="CCW Compliance Slope">254</param>
-                <param name="Return Delay Time">25</param>
-             </gpio>
-             <gpio name="motor_l3l">
-                <param name="type">dxl</param>
-                <param name="ID">3</param>
-                <command_interface name="Goal Position" />
-                <state_interface name="Present Position" />
-                <state_interface name="Present Velocity" />
-                <state_interface name="Present Load" />
-                <param name="[unit info]">Present Position, 0.005061455, rad, unsigned, -2.070135026; Goal Position, 0.005061455, rad, unsigned, -2.070135026</param>
-                <param name="CW Compliance Margin">1</param>
-                <param name="CCW Compliance Margin">1</param>
-                <param name="CW Compliance Slope">254</param>
-                <param name="CCW Compliance Slope">254</param>
-                <param name="Return Delay Time">25</param>
-             </gpio>
-             <gpio name="motor_l5l">
-                <param name="type">dxl</param>
-                <param name="ID">5</param>
-                <command_interface name="Goal Position" />
-                <state_interface name="Present Position" />
-                <state_interface name="Present Velocity" />
-                <state_interface name="Present Load" />
-                <param name="CW Compliance Margin">1</param>
-                <param name="CCW Compliance Margin">1</param>
-                <param name="CW Compliance Slope">254</param>
-                <param name="CCW Compliance Slope">254</param>
-                <param name="Return Delay Time">25</param>
-             </gpio>
-             <gpio name="motor_l6l">
-                <param name="type">dxl</param>
-                <param name="ID">6</param>
-                <command_interface name="Goal Position" />
-                <state_interface name="Present Position" />
-                <state_interface name="Present Velocity" />
-                <state_interface name="Present Load" />
-                <param name="CW Compliance Margin">1</param>
-                <param name="CCW Compliance Margin">1</param>
-                <param name="CW Compliance Slope">254</param>
-                <param name="CCW Compliance Slope">254</param>
-                <param name="Return Delay Time">25</param>
-             </gpio>
-             <gpio name="motor_g2ra">
-                <param name="type">dxl</param>
-                <param name="ID">16</param>
-                <command_interface name="Goal Position" />
-                <state_interface name="Present Position" />
-                <state_interface name="Present Velocity" />
-                <state_interface name="Present Load" />
-                <param name="CW Compliance Margin">1</param>
-                <param name="CCW Compliance Margin">1</param>
-                <param name="CW Compliance Slope">254</param>
-                <param name="CCW Compliance Slope">254</param>
-                <param name="Return Delay Time">25</param>
-             </gpio>
-             <gpio name="motor_g2rb">
-                <param name="type">dxl</param>
-                <param name="ID">17</param>
-                <command_interface name="Goal Position" />
-                <state_interface name="Present Position" />
-                <state_interface name="Present Velocity" />
-                <state_interface name="Present Load" />
-                <param name="CW Compliance Margin">1</param>
-                <param name="CCW Compliance Margin">1</param>
-                <param name="CW Compliance Slope">254</param>
-                <param name="CCW Compliance Slope">254</param>
-                <param name="Return Delay Time">25</param>
-             </gpio>
-             <gpio name="motor_g2r">
-                <param name="type">dxl</param>
-                <param name="ID">7</param>
-                <command_interface name="Goal Position" />
-                <state_interface name="Present Position" />
-                <state_interface name="Present Velocity" />
-                <state_interface name="Present Load" />
-                <param name="CW Compliance Margin">1</param>
-                <param name="CCW Compliance Margin">1</param>
-                <param name="CW Compliance Slope">254</param>
-                <param name="CCW Compliance Slope">254</param>
-                <param name="Return Delay Time">25</param>
-             </gpio>
-             <gpio name="motor_l1h">
-                <param name="type">dxl</param>
-                <param name="ID">19</param>
-                <command_interface name="Goal Position" />
-                <state_interface name="Present Position" />
-                <state_interface name="Present Velocity" />
-                <state_interface name="Present Load" />
-                <param name="CW Compliance Margin">1</param>
-                <param name="CCW Compliance Margin">1</param>
-                <param name="CW Compliance Slope">254</param>
-                <param name="CCW Compliance Slope">254</param>
-                <param name="Return Delay Time">25</param>
-             </gpio>
-             <joint name="l4l_to_l3l">
-               <command_interface name="position" />
-               <state_interface name="position" />
-               <state_interface name="velocity" />
-             </joint>
-             <gpio name="motor_l4l">
-               <param name="type">dxl</param>
-               <param name="ID">1</param>
-               <command_interface name="Goal Position" />
-               <state_interface name="Present Position" />
-               <state_interface name="Present Velocity" />
-               <state_interface name="Present Load" />
-               <param name="[unit info]">Present Position, 0.001533981, rad, unsigned, -2.963651292; Goal Position, 0.001533981, rad, unsigned, -2.963651292</param>
-               <param name="P Gain">8</param>
-               <param name="I Gain">2</param>
-               <param name="D Gain">5</param>
-               <param name="Return Delay Time">25</param>
-             </gpio>
-             <!-- <gpio name="motor_l2h_1">
-                <param name="type">dxl</param>
-                <param name="ID">20</param>
-                <command_interface name="Goal Position" />
-                <state_interface name="Present Position" />
-                <state_interface name="Present Velocity" />
-                <state_interface name="Present Load" />
-                <param name="CW Compliance Margin">1</param>
-                <param name="CCW Compliance Margin">1</param>
-                <param name="CW Compliance Slope">254</param>
-                <param name="CCW Compliance Slope">254</param>
-                <param name="Return Delay Time">25</param>
-             </gpio>
-             <gpio name="motor_l2h_2">
-                <param name="type">dxl</param>
-                <param name="ID">21</param>
-                <command_interface name="Goal Position" />
-                <state_interface name="Present Position" />
-                <state_interface name="Present Velocity" />
-                <state_interface name="Present Load" />
-                <param name="CW Compliance Margin">1</param>
-                <param name="CCW Compliance Margin">1</param>
-                <param name="CW Compliance Slope">254</param>
-                <param name="CCW Compliance Slope">254</param>
-                <param name="Return Delay Time">100</param>
-             </gpio> -->
-           </ros2_control>
+    axis="0"
+	gear_ratio="250"
+	/>
+	<ros2_control name="ShoulderJoint" type="sensor">
+		<hardware>
+			<plugin>bender_hardware_interfaces/EncoderInterface</plugin>
+			<param name="serial_device">/dev/encoders</param>
+			<param name="baud_rate">115200</param>
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
Commit message: (FG): modify odrive ros2 control xacro

File: bender_description/urdf/ros2_control.xacro (robot description, xacro)
@@ -10,11 +10,20 @@
 				<param name="serial_number">${serial_number}</param>
 			</sensor>
-			<joint name="${joint_name}">
+			<joint name="${joint_name_left}">
 				<param name="serial_number">${serial_number}</param>
-				<param name="axis">${axis}</param>
+				<param name="axis">${axis_left}</param>
 				<param name="enable_watchdog">0</param>
 				<param name="watchdog_timeout">1.0</param>
-				<param name="gear_ratio">${gear_ratio}</param>
-				<!-- <command_interface name="position" /> -->
+				<param name="gear_ratio">${gear_ratio_left}</param>
+				<command_interface name="velocity" />
+				<command_interface name="effort" />
+				<state_interface name="effort" />
+			</joint>
+			<joint name="${joint_name_right}">
+				<param name="serial_number">${serial_number}</param>
+				<param name="axis">${axis_right}</param>
+				<param name="enable_watchdog">0</param>
+				<param name="watchdog_timeout">1.0</param>
+				<param name="gear_ratio">${gear_ratio_right}</param>
 				<command_interface name="velocity" />
 				<command_interface name="effort" />
@@ -24,16 +33,12 @@
 	</xacro:macro>
 	<xacro:odrive_ros2_control
-    name="OdriveLeft"
+    name="Odrive"
     serial_number="3690387D3333"
-    joint_name="l1l_to_base_link"
-    axis="0"
-	gear_ratio="250"
-	/>
-	<xacro:odrive_ros2_control
-    name="OdriveRight"
-    serial_number="336B33573235"
-    joint_name="l1r_to_base_link"
-    axis="0"
-	gear_ratio="250"
+    joint_name_left="l1l_to_base_link"
+    joint_name_right="l1r_to_base_link"
+    axis_left="0"
+    axis_right="1"
+	gear_ratio_left="250"
+	gear_ratio_right="250"
 	/>
 	<ros2_control name="ShoulderJoint" type="sensor">
