Commit message: (FG): tuned controllers

File: bender_description/urdf/ros2_control.xacro (robot description, xacro)
@@ -120,7 +120,7 @@
     		<param name="CW Compliance Margin">1</param>
     		<param name="CCW Compliance Margin">1</param>
-    		<param name="CW Compliance Slope">254</param>
-    		<param name="CCW Compliance Slope">254</param>
-    		<param name="Return Delay Time">10</param>
+    		<param name="CW Compliance Slope">50</param>
+    		<param name="CCW Compliance Slope">50</param>
+    		<param name="Return Delay Time">5</param>
 		</gpio>
 		<joint name="l3r_to_l2r">
@@ -137,64 +137,64 @@
 			<state_interface name="Present Load" />
 			<param name="[unit info]">Present Position, 0.005061455, rad, unsigned, -2.04988725; Goal Position, 0.005061455, rad, unsigned, -2.04988725</param>
+			<param name="CW Compliance Margin">1</param>
+			<param name="CCW Compliance Margin">1</param>
+			<param name="CW Compliance Slope">16</param>
+			<param name="CCW Compliance Slope">16</param>
+			<param name="Return Delay Time">5</param>
+		</gpio>
+		<joint name="l4r_to_l3r">
+			<command_interface name="position" />
+			<state_interface name="position" />
+			<state_interface name="velocity" />
+		</joint>
+		<gpio name="motor_l4r">
+			<param name="type">dxl</param>
+			<param name="ID">13</param>
+			<command_interface name="Goal Position" />
+			<state_interface name="Present Position" />
+			<state_interface name="Present Velocity" />
+			<state_interface name="Present Load" />
+			<param name="[unit info]">Present Position, 0.001533981, rad, unsigned, -3.05262219; Goal Position, 0.001533981, rad, unsigned, -3.05262219</param>
+			<param name="P Gain">50</param>
+			<param name="I Gain">32</param>
+			<param name="D Gain">22</param>
+			<param name="Return Delay Time">5</param>
+		</gpio>
+		<joint name="l5r_to_l4r">
+			<command_interface name="position" />
+			<state_interface name="position" />
+			<state_interface name="velocity" />
+		</joint>
+		<gpio name="motor_l5r">
+			<param name="type">dxl</param>
+			<param name="ID">5</param>
+			<command_interface name="Goal Position" />
+			<state_interface name="Present Position" />
+			<state_interface name="Present Velocity" />
+			<state_interface name="Present Load" />
+			<param name="CW Compliance Margin">1</param>
+			<param name="CCW Compliance Margin">1</param>
+			<param name="CW Compliance Slope">64</param>
+			<param name="CCW Compliance Slope">64</param>
+			<param name="Return Delay Time">5</param>
+		</gpio>
+		<joint name="l6r_to_l5r">
+			<command_interface name="position" />
+			<state_interface name="position" />
+			<state_interface name="velocity" />
+		</joint>
+		<gpio name="motor_l6r">
+			<param name="type">dxl</param>
+			<param name="ID">15</param>
+			<command_interface name="Goal Position" />
+			<state_interface name="Present Position" />
+			<state_interface name="Present Velocity" />
+			<state_interface name="Present Load" />
+			<param name="[unit info]">Present Position, 0.005061455, rad, unsigned, -1.94866011; Goal Position, 0.005061455, rad, unsigned, -1.94866011</param>
 			<param name="CW Compliance Margin">1</param>
 			<param name="CCW Compliance Margin">1</param>
 			<param name="CW Compliance Slope">128</param>
 			<param name="CCW Compliance Slope">128</param>
-			<param name="Return Delay Time">10</param>
-		</gpio>
-		<joint name="l4r_to_l3r">
-			<command_interface name="position" />
-			<state_interface name="position" />
-			<state_interface name="velocity" />
-		</joint>
-		<gpio name="motor_l4r">
-			<param name="type">dxl</param>
-			<param name="ID">13</param>
-			<command_interface name="Goal Position" />
-			<state_interface name="Present Position" />
-			<state_interface name="Present Velocity" />
-			<state_interface name="Present Load" />
-			<param name="[unit info]">Present Position, 0.001533981, rad, unsigned, -3.05262219; Goal Position, 0.001533981, rad, unsigned, -3.05262219</param>
-			<param name="P Gain">8</param>
-			<param name="I Gain">2</param>
-			<param name="D Gain">5</param>
-			<param name="Return Delay Time">10</param>
-		</gpio>
-		<joint name="l5r_to_l4r">
-			<command_interface name="position" />
-			<state_interface name="position" />
-			<state_interface name="velocity" />
-		</joint>
-		<gpio name="motor_l5r">
-			<param name="type">dxl</param>
-			<param name="ID">5</param>
-			<command_interface name="Goal Position" />
-			<state_interface name="Present Position" />
-			<state_interface name="Present Velocity" />
-			<state_interface name="Present Load" />
-			<param name="CW Compliance Margin">1</param>
-			<param name="CCW Compliance Margin">1</param>
-			<param name="CW Compliance Slope">128</param>
-			<param name="CCW Compliance Slope">128</param>
-			<param name="Return Delay Time">10</param>
-		</gpio>
-		<joint name="l6r_to_l5r">
-			<command_interface name="position" />
-			<state_interface name="position" />
-			<state_interface name="velocity" />
-		</joint>
-		<gpio name="motor_l6r">
-			<param name="type">dxl</param>
-			<param name="ID">15</param>
-			<command_interface name="Goal Position" />
-			<state_interface name="Present Position" />
-			<state_interface name="Present Velocity" />
-			<state_interface name="Present Load" />
-			<param name="[unit info]">Present Position, 0.005061455, rad, unsigned, -1.94866011; Goal Position, 0.005061455, rad, unsigned, -1.94866011</param>
-			<param name="CW Compliance Margin">1</param>
-			<param name="CCW Compliance Margin">1</param>
-			<param name="CW Compliance Slope">254</param>
-			<param name="CCW Compliance Slope">254</param>
-			<param name="Return Delay Time">10</param>
+			<param name="Return Delay Time">5</param>
 		</gpio>
 		<joint name="l2l_to_l1l">
@@ -213,5 +213,5 @@
     		<param name="I Gain">2</param>
     		<param name="D Gain">5</param>
-    		<param name="Return Delay Time">10</param>
+    		<param name="Return Delay Time">5</param>
 		</gpio>
 		<joint name="l3l_to_l2l">
@@ -232,5 +232,5 @@
 			<param name="CW Compliance Slope">127</param>
 			<param name="CCW Compliance Slope">127</param>
-			<param name="Return Delay Time">10</param>
+			<param name="Return Delay Time">5</param>
 		</gpio>
 		<joint name="l4l_to_l3l">
@@ -250,5 +250,5 @@
 			<param name="I Gain">2</param>
 			<param name="D Gain">5</param>
-			<param name="Return Delay Time">10</param>
+			<param name="Return Delay Time">5</param>
 		</gpio>
 		<joint name="l5l_to_l4l">
@@ -268,5 +268,5 @@
 			<param name="CW Compliance Slope">254</param>
 			<param name="CCW Compliance Slope">254</param>
-			<param name="Return Delay Time">10</param>
+			<param name="Return Delay Time">5</param>
 		</gpio>
 		<joint name="l6l_to_l5l">
@@ -286,5 +286,5 @@
 			<param name="CW Compliance Slope">254</param>
 			<param name="CCW Compliance Slope">254</param>
-			<param name="Return Delay Time">10</param>
+			<param name="Return Delay Time">5</param>
 		</gpio>
 		<joint name="g2ra_to_g1r">
@@ -308,5 +308,5 @@
 			<param name="CW Compliance Slope">32</param>
 			<param name="CCW Compliance Slope">32</param>
-			<param name="Return Delay Time">10</param>
+			<param name="Return Delay Time">5</param>
 		</gpio>
 		<gpio name="motor_g2rb">
@@ -321,5 +321,5 @@
 			<param name="CW Compliance Slope">32</param>
 			<param name="CCW Compliance Slope">32</param>
-			<param name="Return Delay Time">10</param>
+			<param name="Return Delay Time">5</param>
 		</gpio>
         <joint name="gripper_base_to_movil">
@@ -340,5 +340,5 @@
             <param name="CW Compliance Slope">254</param>
             <param name="CCW Compliance Slope">254</param>
-            <param name="Return Delay Time">10</param>
+            <param name="Return Delay Time">5</param>
         </gpio>
 		<joint name="l1h_to_base_link">
@@ -359,5 +359,5 @@
 			<param name="CW Compliance Slope">254</param>
 			<param name="CCW Compliance Slope">254</param>
-			<param name="Return Delay Time">10</param>
+			<param name="Return Delay Time">5</param>
 		</gpio>
 		<joint name="l2h_to_l1h">
@@ -383,5 +383,5 @@
 			<param name="CW Compliance Slope">254</param>
 			<param name="CCW Compliance Slope">254</param>
-			<param name="Return Delay Time">10</param>
+			<param name="Return Delay Time">5</param>
 		</gpio>
 		<gpio name="motor_l2h_2">
@@ -397,5 +397,5 @@
 			<param name="CW Compliance Slope">254</param>
 			<param name="CCW Compliance Slope">254</param>
-			<param name="Return Delay Time">100</param>
+			<param name="Return Delay Time">5</param>
 		</gpio>
 	</ros2_control>

Commit message: (FG): rename joints

File: bender_description/urdf/ros2_control.xacro (robot description, xacro)
@@ -410,10 +410,10 @@
             <param name="wheel_separation">0.397</param>
         </hardware>
-        <joint name="joint1">
+        <joint name="wrl_to_base_link">
             <!-- TODO: check if more state interfaces are available in ARIACODA -->
             <command_interface name="velocity"/>
             <state_interface name="velocity"/>
         </joint>
-        <joint name="joint2">
+        <joint name="wrr_to_base_link">
             <!-- TODO: check if more state interfaces are available in ARIACODA -->
             <command_interface name="velocity"/>

Commit message: (FG): separate arm communication

File: bender_description/urdf/ros2_control.xacro (robot description, xacro)
@@ -57,50 +57,32 @@
 		</sensor>
 	</ros2_control>
-	<ros2_control name="DynamixelChainMain" type="system">
+	<ros2_control name="DynamixelChainRight" type="system">
         <hardware>
             <plugin>dynamixel_hardware_interface/DynamixelHardware</plugin>
-            <param name="port_name">/dev/dynamixel</param>
+            <param name="port_name">/dev/dynamixel_right</param>
             <param name="baud_rate">1000000</param>
             <param name="protocol_version">1.0</param>
-            <param name="number_of_joints">16</param>
-            <param name="number_of_transmissions">16</param>
+            <param name="number_of_joints">7</param>
+            <param name="number_of_transmissions">7</param>
             <param name="dynamixel_model_folder">/param/dxl_model</param>
             <param name="disable_torque_at_init">true</param>
             <param name="torque_enable">0</param>
             <param name="transmission_to_joint_matrix">
-                1, 0, 0, 0, 0, 0, 0, 0, 0, 0, 0, 0, 0, 0, 0, 0,
-                0, 1, 0, 0, 0, 0, 0, 0, 0, 0, 0, 0, 0, 0, 0, 0,
-                0, 0, 1, 0, 0, 0, 0, 0, 0, 0, 0, 0, 0, 0, 0, 0,
-                0, 0, 0, 1, 0, 0, 0, 0, 0, 0, 0, 0, 0, 0, 0, 0,
-                0, 0, 0, 0, 1, 0, 0, 0, 0, 0, 0, 0, 0, 0, 0, 0,
-                0, 0, 0, 0, 0, 1, 0, 0, 0, 0, 0, 0, 0, 0, 0, 0,
-                0, 0, 0, 0, 0, 0, 1, 0, 0, 0, 0, 0, 0, 0, 0, 0,
-                0, 0, 0, 0, 0, 0, 0, 1, 0, 0, 0, 0, 0, 0, 0, 0,
-                0, 0, 0, 0, 0, 0, 0, 0, 1, 0, 0, 0, 0, 0, 0, 0,
-                0, 0, 0, 0, 0, 0, 0, 0, 0, 1, 0, 0, 0, 0, 0, 0,
-                0, 0, 0, 0, 0, 0, 0, 0, 0, 0, 0.5, -0.5, 0, 0, 0, 0,
-                0, 0, 0, 0, 0, 0, 0, 0, 0, 0, 0.5, 0.5, 0, 0, 0, 0,
-                0, 0, 0, 0, 0, 0, 0, 0, 0, 0, 0, 0, 1, 0, 0, 0,
-                0, 0, 0, 0, 0, 0, 0, 0, 0, 0, 0, 0, 0, 1, 0, 0,
-                0, 0, 0, 0, 0, 0, 0, 0, 0, 0, 0, 0, 0, 0, 0.5, -0.5,
-                0, 0, 0, 0, 0, 0, 0, 0, 0, 0, 0, 0, 0, 0, 0.5, 0.5
+                1, 0, 0, 0, 0, 0, 0,
+                0, 1, 0, 0, 0, 0, 0,
+                0, 0, 1, 0, 0, 0, 0,
+                0, 0, 0, 1, 0, 0, 0,
+                0, 0, 0, 0, 1, 0, 0,
+                0, 0, 0, 0, 0, 0.5, -0.5,
+                0, 0, 0, 0, 0, 0.5, 0.5
             </param>
             <param name="joint_to_transmission_matrix">
-                1, 0, 0, 0, 0, 0, 0, 0, 0, 0, 0, 0, 0, 0, 0, 0,
-                0, 1, 0, 0, 0, 0, 0, 0, 0, 0, 0, 0, 0, 0, 0, 0,
-                0, 0, 1, 0, 0, 0, 0, 0, 0, 0, 0, 0, 0, 0, 0, 0,
-                0, 0, 0, 1, 0, 0, 0, 0, 0, 0, 0, 0, 0, 0, 0, 0,
-                0, 0, 0, 0, 1, 0, 0, 0, 0, 0, 0, 0, 0, 0, 0, 0,
-                0, 0, 0, 0, 0, 1, 0, 0, 0, 0, 0, 0, 0, 0, 0, 0,
-                0, 0, 0, 0, 0, 0, 1, 0, 0, 0, 0, 0, 0, 0, 0, 0,
-                0, 0, 0, 0, 0, 0, 0, 1, 0, 0, 0, 0, 0, 0, 0, 0,
-                0, 0, 0, 0, 0, 0, 0, 0, 1, 0, 0, 0, 0, 0, 0, 0,
-                0, 0, 0, 0, 0, 0, 0, 0, 0, 1, 0, 0, 0, 0, 0, 0,
-                0, 0, 0, 0, 0, 0, 0, 0, 0, 0, 1, 1, 0, 0, 0, 0,
-                0, 0, 0, 0, 0, 0, 0, 0, 0, 0, -1, 1, 0, 0, 0, 0,
-                0, 0, 0, 0, 0, 0, 0, 0, 0, 0, 0, 0, 1, 0, 0, 0,
-                0, 0, 0, 0, 0, 0, 0, 0, 0, 0, 0, 0, 0, 1, 0, 0,
-                0, 0, 0, 0, 0, 0, 0, 0, 0, 0, 0, 0, 0, 0, 1, 1,
-                0, 0, 0, 0, 0, 0, 0, 0, 0, 0, 0, 0, 0, 0, -1, 1
+                1, 0, 0, 0, 0, 0, 0,
+                0, 1, 0, 0, 0, 0, 0,
+                0, 0, 1, 0, 0, 0, 0,
+                0, 0, 0, 1, 0, 0, 0,
+                0, 0, 0, 0, 1, 0, 0,
+                0, 0, 0, 0, 0, 1, 1,
+                0, 0, 0, 0, 0, -1, 1
             </param>
         </hardware>
@@ -198,4 +180,74 @@
 			<param name="Return Delay Time">5</param>
 		</gpio>
+		<joint name="g2ra_to_g1r">
+			<command_interface name="position" />
+			<state_interface name="position" />
+			<state_interface name="velocity" />
+		</joint>
+		<joint name="g2rb_to_g1r">
+            <state_interface name="position" />
+            <state_interface name="velocity" />
+        </joint>
+		<gpio name="motor_g2ra">
+			<param name="type">dxl</param>
+			<param name="ID">16</param>
+			<command_interface name="Goal Position" />
+			<state_interface name="Present Position" />
+			<state_interface name="Present Velocity" />
+			<state_interface name="Present Load" />
+			<param name="CW Compliance Margin">1</param>
+			<param name="CCW Compliance Margin">1</param>
+			<param name="CW Compliance Slope">32</param>
+			<param name="CCW Compliance Slope">32</param>
+			<param name="Return Delay Time">5</param>
+		</gpio>
+		<gpio name="motor_g2rb">
+			<param name="type">dxl</param>
+			<param name="ID">17</param>
+			<command_interface name="Goal Position" />
+			<state_interface name="Present Position" />
+			<state_interface name="Present Velocity" />
+			<state_interface name="Present Load" />
+			<param name="CW Compliance Margin">1</param>
+			<param name="CCW Compliance Margin">1</param>
+			<param name="CW Compliance Slope">32</param>
+			<param name="CCW Compliance Slope">32</param>
+			<param name="Return Delay Time">5</param>
+		</gpio>
+	</ros2_control>
+	<ros2_control name="DynamixelChainLeft" type="system">
+        <hardware>
+            <plugin>dynamixel_hardware_interface/DynamixelHardware</plugin>
+            <param name="port_name">/dev/dynamixel_left</param>
+            <param name="baud_rate">1000000</param>
+            <param name="protocol_version">1.0</param>
+            <param name="number_of_joints">9</param>
+            <param name="number_of_transmissions">9</param>
+            <param name="dynamixel_model_folder">/param/dxl_model</param>
+            <param name="disable_torque_at_init">true</param>
+            <param name="torque_enable">0</param>
+            <param name="transmission_to_joint_matrix">
+                1, 0, 0, 0, 0, 0, 0, 0, 0,
+                0, 1, 0, 0, 0, 0, 0, 0, 0,
+                0, 0, 1, 0, 0, 0, 0, 0, 0,
+                0, 0, 0, 1, 0, 0, 0, 0, 0,
+                0, 0, 0, 0, 1, 0, 0, 0, 0,
+                0, 0, 0, 0, 0, 1, 0, 0, 0,
+                0, 0, 0, 0, 0, 0, 1, 0, 0,
+                0, 0, 0, 0, 0, 0, 0, 0.5, -0.5,
+                0, 0, 0, 0, 0, 0, 0, 0.5, 0.5
+            </param>
+            <param name="joint_to_transmission_matrix">
+                1, 0, 0, 0, 0, 0, 0, 0, 0,
+                0, 1, 0, 0, 0, 0, 0, 0, 0,
+                0, 0, 1, 0, 0, 0, 0, 0, 0,
+                0, 0, 0, 1, 0, 0, 0, 0, 0,
+                0, 0, 0, 0, 1, 0, 0, 0, 0,
+                0, 0, 0, 0, 0, 1, 0, 0, 0,
+                0, 0, 0, 0, 0, 0, 1, 0, 0,
+                0, 0, 0, 0, 0, 0, 0, 1, 1,
+                0, 0, 0, 0, 0, 0, 0, -1, 1
+            </param>
+        </hardware>
 		<joint name="l2l_to_l1l">
 			<command_interface name="position" />
@@ -286,39 +338,4 @@
 			<param name="CW Compliance Slope">254</param>
 			<param name="CCW Compliance Slope">254</param>
-			<param name="Return Delay Time">5</param>
-		</gpio>
-		<joint name="g2ra_to_g1r">
-			<command_interface name="position" />
-			<state_interface name="position" />
-			<state_interface name="velocity" />
-		</joint>
-		<joint name="g2rb_to_g1r">
-            <state_interface name="position" />
-            <state_interface name="velocity" />
-        </joint>
-		<gpio name="motor_g2ra">
-			<param name="type">dxl</param>
-			<param name="ID">16</param>
-			<command_interface name="Goal Position" />
-			<state_interface name="Present Position" />
-			<state_interface name="Present Velocity" />
-			<state_interface name="Present Load" />
-			<param name="CW Compliance Margin">1</param>
-			<param name="CCW Compliance Margin">1</param>
-			<param name="CW Compliance Slope">32</param>
-			<param name="CCW Compliance Slope">32</param>
-			<param name="Return Delay Time">5</param>
-		</gpio>
-		<gpio name="motor_g2rb">
-			<param name="type">dxl</param>
-			<param name="ID">17</param>
-			<command_interface name="Goal Position" />
-			<state_interface name="Present Position" />
-			<state_interface name="Present Velocity" />
-			<state_interface name="Present Load" />
-			<param name="CW Compliance Margin">1</param>
-			<param name="CCW Compliance Margin">1</param>
-			<param name="CW Compliance Slope">32</param>
-			<param name="CCW Compliance Slope">32</param>
 			<param name="Return Delay Time">5</param>
 		</gpio>
@@ -400,4 +417,10 @@
 		</gpio>
 	</ros2_control>
+	<!-- DESHABILITADO temporalmente para probar todo menos la base Pioneer.
+	     Recordar sacar también wrl_to_base_link/wrr_to_base_link de la lista
+	     de joints de joint_state_broadcaster en controllers.yaml: si quedan
+	     ahí sin hardware detrás, controller_manager aborta el proceso completo
+	     al no encontrar esas interfaces. -->
+	<!--
 	<ros2_control name="Pioneer" type="system">
     	<hardware>
@@ -418,3 +441,5 @@
         </sensor>
 	</ros2_control>
+	-->
+	<!-- FIN bloque Pioneer -->
 </robot>
